File: hard/hw/Basic_pcb/SAM3N.sch (KiCad schematic (older format))
At the start: 33 parts, among them P1 CONN_02X02, U11 ZLDO1117G33TA, X401 12MHz

Commit message: version0.0
Parts:
- removed C396, C397, C398, C399, C400, C401, C404, C405, C408, C409, C410: 0.1uF, opendous:SM0603, symbol C
- removed C402, C403: 20pF, opendous:SM0603, symbol C
- removed C406, C411: 1uF, opendous:SM0603, symbol C
- removed C407, C412: 4.7uF, opendous:SM1206, symbol C
- removed C74, C76: 33uF, opendous:SM1206, symbol C
- removed C75: 100n, opendous:SM0603, symbol C
- removed D8, D9: LED, opendous:SM0603, symbol LED
- removed DP3: DIODE, opendous:SM0603_Opendous, symbol DIODE
- removed JMS2: USB-MINI, Connect:USB_Mini-B, symbol USB-MINI
- removed P1: CONN_02X02, hackrf:GSG-HEADER-2x2, symbol CONN_02X02
- removed PSA1: CONN_02X14, Socket_Strips:Socket_Strip_Straight_2x14, symbol CONN_02X14
- removed R33, R5: 1k, opendous:SM0603, symbol R
- removed RUF1, RUF2: 27, opendous:SM0603, symbol R
- removed U11: ZLDO1117G33TA, SMD_Packages:SOT-223, symbol LT1117CST
- removed US1: ATSAM3S2CA-AU, Housings_QFP:LQFP-100_14x14mm_Pitch0.5mm, symbol ATSAM3N2
- removed X401: 12MHz, resonator:ABM8G, symbol ABM8G
Connections:
- net labels removed: +1.8V, +3.3VP, AD0, AD1, AD11, AD2, AD3, AD4, AD5, AD8, AD9, AS0, AS1, AS10, AS11, AS12, AS13, AS2, AS3, AS4, AS5, AS6, AS7, AS8, AS9, AS[0..13], CLK_F, CLK_FPGA, DS0, DS1, DS2, DS3, DS4, DS5, DS6, DS7, DS[0..7], Erase, GND, JNRST, JTCK, JTDI, JTDO, JTMS, LED, PA1, PA2, PA27, PA28, PA29, PA3, PA30, PA4, PC10, PC14, PC16, PC9, PWMH0, PWMH1, PWMH2, PWMH3, PWML2, PWML3, RXD0, SAM_RX, SAM_TX, SNCS, SNRD, SNWAIT, SNWE, TIOA2, TXD0, URXD0, UTXD0, VDD5V
- wire segments 227 -> 0
- no-connect marks 2 -> 0
Other:
- note removed: "LEDS"
