File: hard/hw/Basic_pcb/i.MX283_Board.kicad_pcb (KiCad board)
At the start: 4 copper layers, 73 x 73 mm, 151 parts, among them P1 CONN_02X02, U11 ZLDO1117G33TA, X401 12MHz

Commit message: version0.0
Parts:
- removed C396, C397, C398, C399, C400, C401, C404, C405, C408, C409, C410: 0.1uF, SM0603
- removed C402, C403: 20pF, SM0603
- removed C406, C411: 1uF, SM0603
- removed C407, C412: 4.7uF, SM1206
- removed C74, C76: 33uF, SM1206
- removed C75: 100n, SM0603
- removed D8, D9: LED, SM0603
- removed DP3: DIODE, opendous:SM0603_Opendous
- removed JMS2: USB-MINI, Connect:USB_Mini-B
- removed PSA1: CONN_02X14, Socket_Strips:Socket_Strip_Straight_2x14
- removed R33, R5: 1k, SM0603
- removed RUF1, RUF2: 27, SM0603
- removed U11: ZLDO1117G33TA, LT1117
- removed US1: ATSAM3S2CA-AU, Housings_QFP:LQFP-100_14x14mm_Pitch0.5mm
- removed X401: 12MHz, ABM8G
- added IC1: MT48LC4M16A2P, opendous:TSOPII54_SDRAM_MT48, F.Cu at (98.0, 105.3)
- added J1: HDMI_A, HDMI:FCI_10029449-11[13]RLF, F.Cu at (90.9, 58.3)
- added P1: CONN_02X15, hackrf:GSG-HEADER-2x2, F.Cu at (84.1, 130.3)
- added Pl1: CONN_02X15, Pin_Headers:Pin_Header_Straight_2x15_Pitch2.00mm, F.Cu at (116.8, 86.8)
- added X1: OSCILLATORS-1, opendous:OSCILLATOR_7x5mm, F.Cu at (115.1, 56.8)
- P1: value CONN_02X02 -> CONN_02X15
- PFIO1: value CONN_02X18 -> CONN_02X15; footprint Socket_Strips:Socket_Strip_Straight_2x18 -> Socket_Strips:Socket_Strip_Straight_2x15_Pitch2.54mm
- PFIO2: value CONN_02X13 -> CONN_02X15; footprint Socket_Strips:Socket_Strip_Straight_2x12 -> Socket_Strips:Socket_Strip_Straight_2x15_Pitch2.54mm
- moved TH21 164.3 mm to (185.1, 86.9), turned to 90 degrees
- moved TH39 161.5 mm to (185.1, 84.4), turned to 90 degrees
- moved TH22 158.7 mm to (185.1, 81.8), turned to 90 degrees
- moved TH24 156.0 mm to (185.1, 79.3), turned to 90 degrees
- moved TH31 155.4 mm to (175.0, 102.3)
- moved TH32 155.4 mm to (175.0, 107.4)
- moved TH35 155.4 mm to (175.0, 112.5)
- moved TH36 155.4 mm to (175.0, 109.9)
- moved TH37 155.4 mm to (175.0, 104.9)
- moved TH27 153.3 mm to (185.1, 76.7), turned to 90 degrees
- moved TH29 150.6 mm to (185.1, 74.2), turned to 90 degrees
- moved TH1 149.9 mm to (171.2, 139.1)
- moved TH12 149.9 mm to (173.7, 139.1)
- moved TH15 149.9 mm to (176.3, 139.1)
- moved TH38 148.0 mm to (185.1, 71.7), turned to 90 degrees
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Connections:
- net /spartan6/F_TDO renamed /F_TDO
- net VDD5V renamed +5V
- FT1 pad 20: /SAM3M/JNRST -> /serial_interface/nTRST
- FT1 pad 23: /SAM3M/JTDI -> /serial_interface/TDI
- FT1 pad 40: /SAM3M/SAM_RX -> /serial_interface/TXD
- P1 pad 1: GND -> +3.3VDAC
- P1 pad 2: GND -> +3.3VDAC
- P1 pad 3: GND -> +3.3VDAC
- PFIO1 pad 1: /spartan6/IO72 -> /spartan6/IO70
- PFIO1 pad 10: /spartan6/IO65 -> Net-(PFIO1-Pad10)
- PFIO1 pad 11: /spartan6/IO62 -> /spartan6/IO60
- PFIO1 pad 12: /spartan6/IO63 -> /spartan6/IO61
- PFIO1 pad 13: /spartan6/IO60 -> GND
- PFIO1 pad 14: /spartan6/IO61 -> /spartan6/IO31
- PFIO1 pad 15: /spartan6/IO58 -> /spartan6/IO30
- PFIO1 pad 16: /spartan6/IO59 -> /spartan6/IO29
- PFIO1 pad 17: /spartan6/IO56 -> /spartan6/IO28
- PFIO1 pad 18: /spartan6/IO57 -> /spartan6/IO27
- PFIO1 pad 19: GND -> /spartan6/IO26
- PFIO1 pad 2: /spartan6/IO73 -> /spartan6/IO71
- PFIO1 pad 20: /spartan6/IO31 -> /spartan6/IO25
- PFIO1 pad 21: /spartan6/IO30 -> /spartan6/IO24
- PFIO1 pad 22: /spartan6/IO29 -> /spartan6/IO23
- PFIO1 pad 23: /spartan6/IO28 -> /spartan6/IO22
- PFIO1 pad 24: /spartan6/IO27 -> /spartan6/IO21
- PFIO1 pad 25: /spartan6/IO26 -> /spartan6/IO20
- PFIO1 pad 26: /spartan6/IO25 -> /spartan6/IO19
- PFIO1 pad 27: /spartan6/IO24 -> /spartan6/IO18
- PFIO1 pad 28: /spartan6/IO23 -> /spartan6/IO17
- PFIO1 pad 29: /spartan6/IO22 -> GND
- PFIO1 pad 3: /spartan6/IO70 -> /spartan6/IO68
- PFIO1 pad 30: /spartan6/IO21 -> +3.3VDAC
- PFIO1 pad 4: /spartan6/IO71 -> /spartan6/IO69
- PFIO1 pad 5: /spartan6/IO68 -> /spartan6/IO66
- PFIO1 pad 6: /spartan6/IO69 -> /spartan6/IO67
- PFIO1 pad 7: /spartan6/IO66 -> /spartan6/IO64
- PFIO1 pad 8: /spartan6/IO67 -> /spartan6/IO65
- PFIO1 pad 9: /spartan6/IO64 -> Net-(PFIO1-Pad9)
- RF3 pad 1: /spartan6/F_TDI -> /P_TDO
- UF1 pad 1: /SAM3M/AS10 -> /spartan6/CS
- UF1 pad 10: /spartan6/IO6 -> /spartan6/DQ1
- UF1 pad 11: /SAM3M/SNWAIT -> /spartan6/DQ2
- UF1 pad 12: /spartan6/IO7 -> /spartan6/DQ3
- UF1 pad 137: /SAM3M/DS1 -> /spartan6/A3
- UF1 pad 138: /SAM3M/DS2 -> /spartan6/A2
- UF1 pad 139: /SAM3M/DS3 -> /spartan6/A1
- UF1 pad 14: /spartan6/IO8 -> /spartan6/DQ4
- UF1 pad 140: /SAM3M/DS4 -> /spartan6/A0
- UF1 pad 141: /SAM3M/DS5 -> /spartan6/A10
- UF1 pad 142: /SAM3M/DS6 -> /spartan6/BA1
- UF1 pad 143: /SAM3M/DS7 -> /spartan6/BA0
- UF1 pad 15: /SAM3M/SNWE -> /spartan6/DQ5
- UF1 pad 16: /SAM3M/AS9 -> /spartan6/DQ6
- UF1 pad 17: /SAM3M/CLK_F -> /spartan6/DQMH
- UF1 pad 2: /spartan6/IO2 -> /spartan6/RAS
- UF1 pad 21: /SAM3M/AS8 -> /spartan6/DQ8
- UF1 pad 22: /spartan6/IO10 -> /spartan6/DQ9
- UF1 pad 23: /SAM3M/SNRD -> /spartan6/DQ10
- UF1 pad 24: /SAM3M/AS13 -> /spartan6/DQ11
- UF1 pad 26: /spartan6/IO11 -> /spartan6/DQ12
- UF1 pad 27: /SAM3M/AS12 -> /spartan6/DQ13
- UF1 pad 29: /SAM3M/AS11 -> /spartan6/DQ14
- UF1 pad 30: /spartan6/IO12 -> /spartan6/DQ15
- UF1 pad 32: /spartan6/IO13 -> /spartan6/CLK
- UF1 pad 33: /spartan6/IO14 -> /spartan6/CKE
- UF1 pad 35: /spartan6/IO16 -> /spartan6/A11
- UF1 pad 39: /SAM3M/AS7 -> /spartan6/AS7
- UF1 pad 40: /SAM3M/AS6 -> /spartan6/A9
- UF1 pad 41: /SAM3M/AS5 -> /spartan6/A8
- UF1 pad 43: /SAM3M/AS4 -> /spartan6/A7
- UF1 pad 44: /SAM3M/AS3 -> /spartan6/A6
- UF1 pad 45: /SAM3M/AS2 -> /spartan6/A5
- UF1 pad 46: /SAM3M/AS1 -> /spartan6/A4
- UF1 pad 47: /SAM3M/AS0 -> /spartan6/AS0
- UF1 pad 5: /spartan6/IO3 -> /spartan6/CAS
- UF1 pad 6: /spartan6/IO4 -> /spartan6/WE
- UF1 pad 7: /SAM3M/DS0 -> /spartan6/DQML
- UF1 pad 8: /spartan6/IO5 -> /spartan6/DQ7
- UF1 pad 9: /SAM3M/SNCS -> /spartan6/DQ0
- UF1 pad 94: /spartan6/IO46 -> /spartan6/FPGA_CLK
Routing:
- net (no net): track 0.00 -> 3280.1 mm, vias 0 -> 172
- net GND: track 347.6 -> 0.00 mm, vias 61 -> 0
- net +3.3VDAC: track 222.4 -> 8.70 mm, vias 22 -> 0
- net +5V: track 129.1 -> 0.00 mm, vias 3 -> 0
- net +3.3VP: track 121.2 -> 0.00 mm, vias 10 -> 0
- net +1V2: track 119.8 -> 0.00 mm, vias 9 -> 0
- net /spartan6/F_TCK: track 88.4 -> 0.00 mm, vias 4 -> 0
- net /spartan6/F_TMS: track 87.8 -> 0.00 mm, vias 3 -> 0
- net /SAM3M/JTDI: track 74.3 -> 0.00 mm, vias 2 -> 0
- net /SAM3M/JNRST: track 70.4 -> 0.00 mm, vias 6 -> 0
- net +1.8V: track 67.4 -> 0.00 mm, vias 8 -> 0
- net /spartan6/F_TDI: track 61.5 -> 0.00 mm, vias 3 -> 0
- net /serial_interface/RXD: track 56.2 -> 0.00 mm, vias 4 -> 0
- net /SAM3M/SAM_RX: track 54.1 -> 0.00 mm, vias 4 -> 0
- net /SAM3M/AD1: track 50.8 -> 0.00 mm, vias 2 -> 0
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Other:
- board size 73 x 73 mm -> 53.3 x 85.1 mm
