File: hard/hw/Basic_pcb/spartan6.sch (KiCad schematic (older format))
At the start: 48 parts

Commit message: version0.0
Parts:
- removed PFIO1: CONN_02X18, Socket_Strips:Socket_Strip_Straight_2x18, symbol CONN_02X18
- removed PFIO2: CONN_02X13, Socket_Strips:Socket_Strip_Straight_2x13, symbol CONN_02X13
- added IC1: MT48LC4M16A2P, opendous:TSOPII54_SDRAM_MT48, symbol MT48LC4M16A2P
- added J1: HDMI_A, HDMI:FCI_10029449-11[13]RLF, symbol HDMI_A
- added PFIO1, PFIO2: CONN_02X15, Socket_Strips:Socket_Strip_Straight_2x15_Pitch2.54mm, symbol CONN_02X15
- added Pl1: CONN_02X15, Pin_Headers:Pin_Header_Straight_2x15_Pitch2.00mm, symbol CONN_02X15
- added X1: OSCILLATORS-1, opendous:OSCILLATOR_7x5mm, symbol OSCILLATORS-1
- DF1: symbol LED -> LED-RESCUE-i.MX283_Board
Connections:
- net labels added: A0, A1, A10, A11, A2, A3, A4, A5, A6, A7, A8, A9, BA0, BA1, CAS, CKE, CLK, CS, DQ0, DQ1, DQ10, DQ11, DQ12, DQ13, DQ14, DQ15, DQ2, DQ3, DQ4, DQ5, DQ6, DQ7, DQ8, DQ9, DQMH, DQML, FPGA_CLK, RAS, WE
- net labels removed: AS1, AS10, AS11, AS12, AS13, AS2, AS3, AS4, AS5, AS6, AS8, AS9, AS[0..13], CLK_FPGA, DS0, DS1, DS2, DS3, DS4, DS5, DS6, DS7, DS[0..7], IO10, IO11, IO12, IO13, IO14, IO16, IO2, IO3, IO4, IO5, IO6, IO8, SNCS, SNRD, SNWAIT, SNWE
- wire segments 348 -> 421
Other:
- note added: "Ruben: Se eliminaron 1072, 1073, 1062, \n1063, 1058, 1059, 1056, 1057 por \nconector HDMI"
- moved on the sheet: CF30, CF31, CF32, CF33, CF34, CF35, RF5, UF2, UF3
