File: hard/hw/Basic_pcb/spartan6.sch (KiCad schematic (older format))
At the start: 52 parts, among them IC1 MT48LC4M16A2P, J1 HDMI_A, X1 OSCILLATORS-1

Commit message: Actualización Raiz
by Rubén
Parts:
- removed CF1, CF10, CF11, CF12, CF13, CF16, CF17, CF18, CF19, CF2, CF20, CF23, CF24, CF25, CF26, CF27, CF3, CF4, CF5, CF6, CF7, CF8, CF9: 0.1uF, opendous:SM0603, symbol C
- removed CF14, CF21, CF28: 1uF, opendous:SM0603, symbol C
- removed CF15, CF22, CF29: 4.7uF, opendous:SM1206_Opendous, symbol C
- X1: value OSCILLATORS-1 -> ASV-32.000MHZ-E-T; DIGIKEY REF (none) -> 535-10082-2-ND
Connections:
- net labels removed: AS0, AS7, IO15, IO17, IO24, IO29, IO30, IO31, IO32, IO33, IO34, IO35, IO36, IO37, IO38, IO39, IO40, IO41, IO42, IO43, IO44, IO45, IO46, IO47, IO48, IO49, IO50, IO51, IO53, IO54, IO60, IO61, IO64, IO65, IO66, IO67, IO68, IO69, IO70, IO71
- wire segments 383 -> 231
Other:
- note removed: "Check polarity for M0 and M1\ninit program"
- note removed: "Ruben: Se eliminaron 1072, 1073, 1062, \n1063, 1058, 1059, 1056, 1057 por \nconector HDMI.\nRubén: Se eliminaron IO18, IO19, \nIO20, IO21, IO22, IO23, IO25, IO26, \nIO27, IO28 por conector LVDS."
- note removed: "Ruben: Se eliminaron IO55 Y IO52 \npara USB RX y TX"
- moved on the sheet: DF1, IC1, PFIO1, PFIO2, Pl1, RF1, RF2, RF3, RF4, RF5, RF6, RF7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

Commit message: Actualizacion ref. DigitKey
by Rubén
Parts:
- IC1: value MT48LC4M16A2P -> W9812G6KH; DIGIKEY REF (none) -> W9812G6KH-6 TR-ND
- J1: DIGIKEY REF (none) -> 10029449-113RLF-ND
- UF1: DIGIKEY REF (none) -> 122-1745-ND
Changed lines of the file:
@@
 F 1 "XC6SLX9-2TQG144C" H 5550 4950 60  0000 C CNN
 F 2 "Housings_QFP:LQFP-144_20x20mm_Pitch0.5mm" H 4500 4250 60  0001 C CNN
-F 3 "" H 4500 4250 60  0000 C CNN
+F 3 "https://www.xilinx.com/support/documentation/data_sheets/ds162.pdf" H 4500 4250 60  0001 C CNN
+F 4 "122-1745-ND" H 5500 4900 60  0001 C CNN "DIGIKEY REF"
 	1    5500 4900
 	1    0    0    -1
@@
 P 8750 9400
 F 0 "IC1" H 8150 10600 50  0000 C CNN
-F 1 "MT48LC4M16A2P" H 9400 8200 50  0000 C CNN
+F 1 "W9812G6KH" H 9400 8200 50  0000 C CNN
 F 2 "opendous:TSOPII54_SDRAM_MT48" H 8750 9400 50  0000 C CIN
-F 3 "" H 8750 9150 50  0000 C CNN
+F 3 "http://www.winbond.com/resource-files/da00-w9812g6khc1.pdf" H 8750 9150 50  0001 C CNN
+F 4 "W9812G6KH-6 TR-ND" H 8750 9400 60  0001 C CNN "DIGIKEY REF"
 	1    8750 9400
 	1    0    0    -1
@@
 F 1 "HDMI_A" H 13800 1600 60  0000 C CNN
 F 2 "HDMI:FCI_10029449-11[13]RLF" H 12950 2350 60  0001 C CNN
-F 3 "" H 12950 2350 60  0000 C CNN
+F 3 "http://www.datasheets360.com/pdf/-1410121183821781271" H 12950 2350 60  0001 C CNN
+F 4 "10029449-113RLF-ND" H 13450 2850 60  0001 C CNN "DIGIKEY REF"
 	1    13450 2850
 	-1   0    0    1

Commit message: todas las huellas
by Ruben
Parts:
- added SW1: SWITCH_PUSHBUTTON, symbol SWITCH_PUSHBUTTON
Connections:
- net labels added: F_~SD, REBOOT
- wire segments 231 -> 233
Other:
- moved on the sheet: RF1, RF2, RF3, RF4, RF6, RF7, UF1, X1

Commit message: Organizando PIN OUT vr.:0.1
by Ruben
Parts:
- removed PFIO1, PFIO2: CONN_02X15, Socket_Strips:Socket_Strip_Straight_2x15_Pitch2.54mm, symbol CONN_02X15
- added PIO1: CONN_02X20, Socket_Strips:Socket_Strip_Straight_2x20_Pitch2.54mm, symbol CONN_02X20
- SW1: value SWITCH_PUSHBUTTON -> B3SL-1002P; footprint (none) -> Buttons_Switches_SMD:SW_SPST_B3SL-1002P; REF DIGIKEY (none) -> SW1064CT-ND
- renumbered Pl1 to LVDS1
Connections:
- net labels added: +5V, IO01, IO02, IO03, IO04, IO05, IO06, IO07, IO08, IO09, IO10, IO11, IO12, IO13, IO14, IO15, IO16, IO17, IO18, IO19, IO20, IO21, IO22, IO23, IO24, IO25, IO26, IO27, IO28, IO29, IO30, IO31, IO32, IO33, IO34, IO35, IO36, IO37, IO_LED
- net labels removed: IO7
- wire segments 233 -> 313
- no-connect marks 12 -> 15

Commit message: Terminado Shield
by Ruben
Parts:
- added DF2: LED, opendous:SM0603, symbol LED-RESCUE-i.MX283_Board
- added RF8: 1k, opendous:SM0603, symbol R
Connections:
- wire segments 313 -> 318
Other:
- moved on the sheet: DF1, RF5
Changed lines of the file:
@@
 L GND #PWR031
 U 1 1 54E73BD5
-P 6100 9650
-F 0 "#PWR031" H 6100 9650 30  0001 C CNN
-F 1 "GND" H 6100 9580 30  0001 C CNN
-F 2 "" H 6100 9650 60  0001 C CNN
-F 3 "" H 6100 9650 60  0001 C CNN
-	1    6100 9650
+P 5550 9200
+F 0 "#PWR031" H 5550 9200 30  0001 C CNN
+F 1 "GND" H 5550 9130 30  0001 C CNN
+F 2 "" H 5550 9200 60  0001 C CNN
+F 3 "" H 5550 9200 60  0001 C CNN
+	1    5550 9200
 	0    -1   1    0
 $EndComp
@@
 L LED-RESCUE-i.MX283_Board DF1
 U 1 1 54E73BDB
-P 5700 9350
+P 5150 8900
 AR Path="/54E73BDB" Ref="DF1"  Part="1"
 AR Path="/54B6445D/54E73BDB" Ref="DF1"  Part="1"
-F 0 "DF1" H 5700 9450 50  0000 C CNN
-F 1 "LED" H 5700 9250 50  0000 C CNN
-F 2 "opendous:SM0603" H 5700 9350 60  0001 C CNN
-F 3 "" H 5700 9350 60  0001 C CNN
-	1    5700 9350
+F 0 "DF1" H 5150 9000 50  0000 C CNN
+F 1 "LED" H 5150 8800 50  0000 C CNN
+F 2 "opendous:SM0603" H 5150 8900 60  0001 C CNN
+F 3 "" H 5150 8900 60  0001 C CNN
+	1    5150 8900
 	-1   0    0    1
 $EndComp
@@
 L R RF5
 U 1 1 54E73BE2
-P 5700 9650
-F 0 "RF5" V 5780 9650 50  0000 C CNN
-F 1 "1k" V 5700 9650 50  0000 C CNN
-F 2 "opendous:SM0603" H 5700 9650 60  0001 C CNN
-F 3 "" H 5700 9650 60  0001 C CNN
-	1    5700 9650
+P 5150 9200
+F 0 "RF5" V 5230 9200 50  0000 C CNN
+F 1 "1k" V 5150 9200 50  0000 C CNN
+F 2 "opendous:SM0603" H 5150 9200 60  0001 C CNN
+F 3 "" H 5150 9200 60  0001 C CNN
+	1    5150 9200
 	0    1    1    0
 $EndComp
@@
 	0    1    1    0
 $EndComp
-Text Label 5900 9350 0    60   ~ 0
+Text Label 5350 8900 0    60   ~ 0
 IO_LED
 $Comp
@@
 	7650 1800 7650 2150
 Wire Wire Line
-	5900 9350 6200 9350
-Wire Wire Line
-	5850 9650 6100 9650
-Wire Wire Line
-	5350 9650 5550 9650
-Wire Wire Line
-	5350 9650 5350 9350
-Wire Wire Line
-	5350 9350 5500 9350
+	5350 8900 5650 8900
+Wire Wire Line
+	5300 9200 5550 9200
+Wire Wire Line
+	4800 9200 5000 9200
+Wire Wire Line
+	4800 9200 4800 8900
+Wire Wire Line
+	4800 8900 4950 8900
 Wire Wire Line
 	7750 1900 8050 1900
@@
 Wire Wire Line
 	11700 5850 12050 5850
+$Comp
+L GND #PWR059
+U 1 1 58A75988
+P 3750 9250
+F 0 "#PWR059" H 3750 9250 30  0001 C CNN
+F 1 "GND" H 3750 9180 30  0001 C CNN
+F 2 "" H 3750 9250 60  0001 C CNN
+F 3 "" H 3750 9250 60  0001 C CNN
+	1    3750 9250
+	0    -1   1    0
+$EndComp
+$Comp
+L LED-RESCUE-i.MX283_Board DF2
+U 1 1 58A7598E
+P 3350 8950
+F 0 "DF2" H 3350 9050 50  0000 C CNN
+F 1 "LED" H 3350 8850 50  0000 C CNN
+F 2 "opendous:SM0603" H 3350 8950 60  0001 C CNN
+F 3 "" H 3350 8950 60  0001 C CNN
+	1    3350 8950
+	-1   0    0    1
+$EndComp
+$Comp
+L R RF8
+U 1 1 58A75994
+P 3350 9250
+F 0 "RF8" V 3430 9250 50  0000 C CNN
+F 1 "1k" V 3350 9250 50  0000 C CNN
+F 2 "opendous:SM0603" H 3350 9250 60  0001 C CNN
+F 3 "" H 3350 9250 60  0001 C CNN
+	1    3350 9250
+	0    1    1    0
+$EndComp
+Wire Wire Line
+	3550 8950 3850 8950
+Wire Wire Line
+	3500 9250 3750 9250
+Wire Wire Line
+	3000 9250 3200 9250
+Wire Wire Line
+	3000 9250 3000 8950
+Wire Wire Line
+	3000 8950 3150 8950
 $EndSCHEMATC

Commit message: shield 2.0
Parts:
- removed PIO1: CONN_02X20, Socket_Strips:Socket_Strip_Straight_2x20_Pitch2.54mm, symbol CONN_02X20
Connections:
- net labels removed: +5V, IO01, IO02, IO03, IO30, IO31, IO32, IO33, IO34, IO35, IO36, IO37
- wire segments 318 -> 265
Other:
- note added: ">>> F A L T A ! ! !\nAsignar a la FPGA"
- moved on the sheet: DF1, DF2, RF5, RF8

Commit message: Alimentacion Pantalla
Parts:
- R10, R11, R4, R5, R6, R7, R8, R9: footprint Resistors_SMD:R_0805 -> Resistors_SMD:R_0402
Connections:
- net labels removed: IO04, IO05, IO06, IO07, IO08, IO09, IO10, IO11, IO12, IO13, IO14, IO15, IO16, IO17, IO18, IO19, IO20, IO21, IO22, IO23, IO24, IO25, IO26, IO27, IO28, IO29, IO_LED
- wire segments 265 -> 238
- no-connect marks 15 -> 22
Changed lines of the file:
@@
 	0    1    1    0
 $EndComp
-Text Label 5250 8800 0    60   ~ 0
-IO_LED
 $Comp
 L GND #PWR032
@@
 TMDS_D0_P
 $Comp
-L R R4
-U 1 1 589C9D5F
-P 15100 2550
-F 0 "R4" V 15180 2550 50  0000 C CNN
-F 1 "51" V 15100 2550 50  0000 C CNN
-F 2 "Resistors_SMD:R_0805" V 15030 2550 50  0001 C CNN
-F 3 "" H 15100 2550 50  0000 C CNN
-	1    15100 2550
-	0    -1   -1   0
-$EndComp
-$Comp
-L R R5
-U 1 1 589CB340
-P 15100 2750
-F 0 "R5" V 15180 2750 50  0000 C CNN
-F 1 "51" V 15100 2750 50  0000 C CNN
-F 2 "Resistors_SMD:R_0805" V 15030 2750 50  0001 C CNN
-F 3 "" H 15100 2750 50  0000 C CNN
-	1    15100 2750
-	0    -1   -1   0
-$EndComp
-$Comp
-L R R6
-U 1 1 589CB476
-P 15100 2950
-F 0 "R6" V 15180 2950 50  0000 C CNN
-F 1 "51" V 15100 2950 50  0000 C CNN
-F 2 "Resistors_SMD:R_0805" V 15030 2950 50  0001 C CNN
-F 3 "" H 15100 2950 50  0000 C CNN
-	1    15100 2950
-	0    -1   -1   0
-$EndComp
-$Comp
 L HDMI_A J1
 U 1 1 58900C58
@@
 	1    13450 2850
 	-1   0    0    1
-$EndComp
-$Comp
-L R R7
-U 1 1 589D4314
-P 15100 3150
-F 0 "R7" V 15180 3150 50  0000 C CNN
-F 1 "51" V 15100 3150 50  0000 C CNN
-F 2 "Resistors_SMD:R_0805" V 15030 3150 50  0001 C CNN
-F 3 "" H 15100 3150 50  0000 C CNN
-	1    15100 3150
-	0    -1   -1   0
-$EndComp
-$Comp
-L R R8
-U 1 1 589D4454
-P 15100 3350
-F 0 "R8" V 15180 3350 50  0000 C CNN
-F 1 "51" V 15100 3350 50  0000 C CNN
-F 2 "Resistors_SMD:R_0805" V 15030 3350 50  0001 C CNN
-F 3 "" H 15100 3350 50  0000 C CNN
-	1    15100 3350
-	0    -1   -1   0
-$EndComp
-$Comp
-L R R9
-U 1 1 589D4596
-P 15100 3550
-F 0 "R9" V 15180 3550 50  0000 C CNN
-F 1 "51" V 15100 3550 50  0000 C CNN
-F 2 "Resistors_SMD:R_0805" V 15030 3550 50  0001 C CNN
-F 3 "" H 15100 3550 50  0000 C CNN
-	1    15100 3550
-	0    -1   -1   0
-$EndComp
-$Comp
-L R R10
-U 1 1 589D4676
-P 15100 3750
-F 0 "R10" V 15180 3750 50  0000 C CNN
-F 1 "51" V 15100 3750 50  0000 C CNN
-F 2 "Resistors_SMD:R_0805" V 15030 3750 50  0001 C CNN
-F 3 "" H 15100 3750 50  0000 C CNN
-	1    15100 3750
-	0    -1   -1   0
-$EndComp
-$Comp
-L R R11
-U 1 1 589D48FC
-P 15100 3950
-F 0 "R11" V 15180 3950 50  0000 C CNN
-F 1 "51" V 15100 3950 50  0000 C CNN
-F 2 "Resistors_SMD:R_0805" V 15030 3950 50  0001 C CNN
-F 3 "" H 15100 3950 50  0000 C CNN
-	1    15100 3950
-	0    -1   -1   0
 $EndComp
 $Comp
@@
 	0    1    1    0
 $EndComp
-Text Label 8950 4150 0    60   ~ 0
-IO_LED
-Text Label 8950 3550 0    60   ~ 0
-IO04
-Text Label 8950 3450 0    60   ~ 0
-IO05
 NoConn ~ 8900 3050
 NoConn ~ 8900 3150
-Text Label 9050 3250 0    60   ~ 0
-IO06
-Text Label 6000 2050 1    60   ~ 0
-IO07
-Text Label 5900 2050 1    60   ~ 0
-IO08
-Text Label 5800 2050 1    60   ~ 0
-IO09
-Text Label 5700 2050 1    60   ~ 0
-IO10
-Text Label 5600 2050 1    60   ~ 0
-IO11
-Text Label 5500 2050 1    60   ~ 0
-IO12
-Text Label 5400 2050 1    60   ~ 0
-IO13
-Text Label 5300 2050 1    60   ~ 0
-IO14
-Text Label 5100 2050 1    60   ~ 0
-IO16
-Text Label 5000 2050 1    60   ~ 0
-IO17
-Text Label 4900 2050 1    60   ~ 0
-IO18
-Text Label 4800 2050 1    60   ~ 0
-IO19
-Text Label 4700 2050 1    60   ~ 0
-IO20
-Text Label 5200 2050 1    60   ~ 0
-IO15
-Text Label 4500 2050 1    60   ~ 0
-IO21
-Text Label 4400 2050 1    60   ~ 0
-IO22
-Text Label 4300 2050 1    60   ~ 0
-IO23
-Text Label 4200 2050 1    60   ~ 0
-IO24
-Text Label 4100 2050 1    60   ~ 0
-IO25
-Text Label 3900 2050 1    60   ~ 0
-IO26
-Text Label 3800 2050 1    60   ~ 0
-IO27
-Text Label 2000 3200 0    60   ~ 0
-IO28
-Text Label 2000 3300 0    60   ~ 0
-IO29
 NoConn ~ 7550 2150
 $Comp
-L GND #PWR059
+L GND #PWR056
 U 1 1 58A75988
 P 3700 9100
-F 0 "#PWR059" H 3700 9100 30  0001 C CNN
+F 0 "#PWR056" H 3700 9100 30  0001 C CNN
 F 1 "GND" H 3700 9030 30  0001 C CNN
 F 2 "" H 3700 9100 60  0001 C CNN
@@
 	0    1    1    0
 $EndComp
+Text Notes 3850 9550 0    60   ~ 0
+>>> F A L T A ! ! !\nAsignar a la FPGA
 Wire Wire Line
 	14100 9200 14100 9300
@@
 Wire Wire Line
 	15350 2400 15350 3950
-Connection ~ 15350 3150
-Wire Wire Line
-	15350 3150 15250 3150
 Wire Wire Line
 	14450 5750 14450 5650
@@
 	14200 2650 14150 2650
 Wire Wire Line
-	14150 2550 14950 2550
-Wire Wire Line
-	14150 2750 14950 2750
-Wire Wire Line
-	14150 2950 14950 2950
-Wire Wire Line
-	14950 3150 14150 3150
-Wire Wire Line
-	14950 3350 14150 3350
-Wire Wire Line
-	14150 3550 14950 3550
-Wire Wire Line
-	14950 3750 14150 3750
-Wire Wire Line
-	14950 3950 14150 3950
-Wire Wire Line
-	15350 3950 15250 3950
-Wire Wire Line
-	15350 3750 15250 3750
-Connection ~ 15350 3750
-Wire Wire Line
-	15350 3550 15250 3550
-Connection ~ 15350 3550
-Wire Wire Line
-	15250 3350 15350 3350
-Connection ~ 15350 3350
-Wire Wire Line
-	15250 2950 15350 2950
-Connection ~ 15350 2950
-Wire Wire Line
-	15250 2750 15350 2750
-Connection ~ 15350 2750
-Wire Wire Line
-	15250 2550 15350 2550
-Connection ~ 15350 2550
-Wire Wire Line
 	1900 5550 1900 5600
-Wire Wire Line
-	9250 4150 8900 4150
-Wire Wire Line
-	9250 3550 8900 3550
-Wire Wire Line
-	9250 3450 8900 3450
-Wire Wire Line
-	9250 3250 8900 3250
-Wire Wire Line
-	6000 1800 6000 2150
-Wire Wire Line
-	5900 1800 5900 2150
-Wire Wire Line
-	5800 1800 5800 2150
-Wire Wire Line
-	5700 1800 5700 2150
-Wire Wire Line
-	5600 1800 5600 2150
-Wire Wire Line
-	5500 1800 5500 2150
-Wire Wire Line
-	5400 1800 5400 2150
-Wire Wire Line
-	5300 1800 5300 2150
-Wire Wire Line
-	5200 1800 5200 2150
-Wire Wire Line
-	5100 1800 5100 2150
-Wire Wire Line
-	5000 1800 5000 2150
-Wire Wire Line
-	4900 1800 4900 2150
-Wire Wire Line
-	4800 1800 4800 2150
-Wire Wire Line
-	4700 1800 4700 2150
-Wire Wire Line
-	4500 1800 4500 2150
-Wire Wire Line
-	4400 1800 4400 2150
-Wire Wire Line
-	4300 1800 4300 2150
-Wire Wire Line
-	4200 1800 4200 2150
-Wire Wire Line
-	4100 1800 4100 2150
-Wire Wire Line
-	3900 1800 3900 2150
-Wire Wire Line
-	3800 1800 3800 2150
-Wire Wire Line
-	1950 3200 2300 3200
-Wire Wire Line
-	1950 3300 2300 3300
 Wire Wire Line
 	3500 8800 3800 8800
@@
 Wire Notes Line
 	2400 9900 2400 8200
-Text Notes 3850 9550 0    60   ~ 0
->>> F A L T A ! ! !\nAsignar a la FPGA
+Wire Wire Line
+	14150 2750 14950 2750
+Wire Wire Line
+	14950 3150 14150 3150
+Wire Wire Line
+	14150 3550 14950 3550
+Wire Wire Line
+	14950 3950 14150 3950
+Wire Wire Line
+	14150 2550 14950 2550
+Wire Wire Line
+	14150 2950 14950 2950
+Wire Wire Line
+	14950 3350 14150 3350
+Wire Wire Line
+	14950 3750 14150 3750
+Wire Wire Line
+	15350 3950 15250 3950
+Wire Wire Line
+	15350 3750 15250 3750
+Connection ~ 15350 3750
+Wire Wire Line
+	15350 3550 15250 3550
+Connection ~ 15350 3550
+Wire Wire Line
+	15250 3350 15350 3350
+Connection ~ 15350 3350
+Wire Wire Line
+	15350 3150 15250 3150
+Connection ~ 15350 3150
+Wire Wire Line
+	15250 2950 15350 2950
+Connection ~ 15350 2950
+Wire Wire Line
+	15250 2750 15350 2750
+Connection ~ 15350 2750
+Wire Wire Line
+	15250 2550 15350 2550
+Connection ~ 15350 2550
+$Comp
+L R R11
+U 1 1 589D48FC
+P 15100 3950
+F 0 "R11" V 15180 3950 50  0000 C CNN
+F 1 "51" V 15100 3950 50  0000 C CNN
+F 2 "Resistors_SMD:R_0402" V 15030 3950 50  0001 C CNN
+F 3 "" H 15100 3950 50  0000 C CNN
+	1    15100 3950
+	0    -1   -1   0
+$EndComp
+$Comp
+L R R10
+U 1 1 589D4676
+P 15100 3750
+F 0 "R10" V 15180 3750 50  0000 C CNN
+F 1 "51" V 15100 3750 50  0000 C CNN
+F 2 "Resistors_SMD:R_0402" V 15030 3750 50  0001 C CNN
+F 3 "" H 15100 3750 50  0000 C CNN
+	1    15100 3750
+	0    -1   -1   0
+$EndComp
+$Comp
+L R R9
+U 1 1 589D4596
+P 15100 3550
+F 0 "R9" V 15180 3550 50  0000 C CNN
+F 1 "51" V 15100 3550 50  0000 C CNN
+F 2 "Resistors_SMD:R_0402" V 15030 3550 50  0001 C CNN
+F 3 "" H 15100 3550 50  0000 C CNN
+	1    15100 3550
+	0    -1   -1   0
+$EndComp
+$Comp
+L R R8
+U 1 1 589D4454
+P 15100 3350
+F 0 "R8" V 15180 3350 50  0000 C CNN
+F 1 "51" V 15100 3350 50  0000 C CNN
+F 2 "Resistors_SMD:R_0402" V 15030 3350 50  0001 C CNN
+F 3 "" H 15100 3350 50  0000 C CNN
+	1    15100 3350
+	0    -1   -1   0
+$EndComp
+$Comp
+L R R7
+U 1 1 589D4314
+P 15100 3150
+F 0 "R7" V 15180 3150 50  0000 C CNN
+F 1 "51" V 15100 3150 50  0000 C CNN
+F 2 "Resistors_SMD:R_0402" V 15030 3150 50  0001 C CNN
+F 3 "" H 15100 3150 50  0000 C CNN
+	1    15100 3150
+	0    -1   -1   0
+$EndComp
+$Comp
+L R R6
+U 1 1 589CB476
+P 15100 2950
+F 0 "R6" V 15180 2950 50  0000 C CNN
+F 1 "51" V 15100 2950 50  0000 C CNN
+F 2 "Resistors_SMD:R_0402" V 15030 2950 50  0001 C CNN
+F 3 "" H 15100 2950 50  0000 C CNN
+	1    15100 2950
+	0    -1   -1   0
+$EndComp
+$Comp
+L R R5
+U 1 1 589CB340
+P 15100 2750
+F 0 "R5" V 15180 2750 50  0000 C CNN
+F 1 "51" V 15100 2750 50  0000 C CNN
+F 2 "Resistors_SMD:R_0402" V 15030 2750 50  0001 C CNN
+F 3 "" H 15100 2750 50  0000 C CNN
+	1    15100 2750
+	0    -1   -1   0
+$EndComp
+$Comp
+L R R4
+U 1 1 589C9D5F
+P 15100 2550
+F 0 "R4" V 15180 2550 50  0000 C CNN
+F 1 "51" V 15100 2550 50  0000 C CNN
+F 2 "Resistors_SMD:R_0402" V 15030 2550 50  0001 C CNN
+F 3 "" H 15100 2550 50  0000 C CNN
+	1    15100 2550
+	0    -1   -1   0
+$EndComp
+NoConn ~ 14150 1750
+NoConn ~ 14150 1850
+NoConn ~ 14150 1950
+NoConn ~ 14150 2050
+NoConn ~ 14150 2150
+NoConn ~ 14150 2250
+NoConn ~ 14150 2350
 $EndSCHEMATC

Commit message: update
Parts:
- added PIO1, PIO2: CONN_02X10, Socket_Strips:Socket_Strip_Straight_2x10_Pitch2.54mm, symbol CONN_02X10
Connections:
- net labels added: +5V
- wire segments 238 -> 243
Changed lines of the file:
@@
 NoConn ~ 14150 2250
 NoConn ~ 14150 2350
+$Comp
+L CONN_02X10 PIO1
+U 1 1 58B73C30
+P 11400 4350
+F 0 "PIO1" H 11400 4900 50  0000 C CNN
+F 1 "CONN_02X10" V 11400 4350 50  0000 C CNN
+F 2 "Socket_Strips:Socket_Strip_Straight_2x10_Pitch2.54mm" H 11400 3150 50  0001 C CNN
+F 3 "" H 11400 3150 50  0000 C CNN
+	1    11400 4350
+	1    0    0    -1
+$EndComp
+$Comp
+L CONN_02X10 PIO2
+U 1 1 58B740F2
+P 11400 5800
+F 0 "PIO2" H 11400 6350 50  0000 C CNN
+F 1 "CONN_02X10" V 11400 5800 50  0000 C CNN
+F 2 "Socket_Strips:Socket_Strip_Straight_2x10_Pitch2.54mm" H 11400 4600 50  0001 C CNN
+F 3 "" H 11400 4600 50  0000 C CNN
+	1    11400 5800
+	1    0    0    -1
+$EndComp
+$Comp
+L +3V3 #PWR057
+U 1 1 58B745E8
+P 11750 5300
+F 0 "#PWR057" H 11750 5150 50  0001 C CNN
+F 1 "+3V3" H 11750 5440 50  0000 C CNN
+F 2 "" H 11750 5300 50  0000 C CNN
+F 3 "" H 11750 5300 50  0000 C CNN
+	1    11750 5300
+	1    0    0    -1
+$EndComp
+$Comp
+L GND #PWR058
+U 1 1 58B74641
+P 11750 5450
+F 0 "#PWR058" H 11750 5450 30  0001 C CNN
+F 1 "GND" H 11750 5380 30  0001 C CNN
+F 2 "" H 11750 5450 60  0001 C CNN
+F 3 "" H 11750 5450 60  0001 C CNN
+	1    11750 5450
+	0    -1   -1   0
+$EndComp
+$Comp
+L +5V #PWR059
+U 1 1 58B75DC4
+P 11050 5300
+F 0 "#PWR059" H 11050 5150 50  0001 C CNN
+F 1 "+5V" H 11050 5440 50  0000 C CNN
+F 2 "" H 11050 5300 50  0000 C CNN
+F 3 "" H 11050 5300 50  0000 C CNN
+	1    11050 5300
+	1    0    0    -1
+$EndComp
+Wire Wire Line
+	11750 5300 11750 5350
+Wire Wire Line
+	11750 5350 11650 5350
+Wire Wire Line
+	11750 5450 11650 5450
+Wire Wire Line
+	11150 5350 11050 5350
+Wire Wire Line
+	11050 5350 11050 5300
 $EndSCHEMATC
