File: hard/hw/Basic_pcb/Audio.sch (KiCad schematic (older format))
At the start: 14 parts, among them P1 CONN_01X05, P2 CONN_01X02, U1 PAM8302A

Commit message: Actualización Raiz
by Rubén
Parts:
- removed P1: CONN_01X05, symbol CONN_01X05
- added P1, P5: CONN_01X03, Socket_Strips:Socket_Strip_Straight_1x03_Pitch2.54mm, symbol CONN_01X03
Other:
- moved on the sheet: C1, R1
Changed lines of the file:
@@
 L C C1
 U 1 1 5898CF7F
-P 3050 5200
-F 0 "C1" H 2950 5300 50  0000 L CNN
-F 1 "10uF" H 2850 5100 50  0000 L CNN
-F 2 "Capacitors_SMD:C_0805" H 3600 5200 50  0001 C CNN
-F 3 "" H 3050 5200 50  0000 C CNN
-	1    3050 5200
+P 4700 5250
+F 0 "C1" H 4600 5350 50  0000 L CNN
+F 1 "10uF" H 4500 5150 50  0000 L CNN
+F 2 "Capacitors_SMD:C_0805" H 5250 5250 50  0001 C CNN
+F 3 "" H 4700 5250 50  0000 C CNN
+	1    4700 5250
 	-1   0    0    -1
 $EndComp
@@
 	1    0    0    -1
 $EndComp
-Text Label 2950 3500 0    60   ~ 0
+Text Label 2600 3300 0    60   ~ 0
 AIN+
-Text Label 2950 3600 0    60   ~ 0
+Text Label 2600 3400 0    60   ~ 0
 AIN-
-Text Label 2950 3700 0    60   ~ 0
+Text Label 2600 4350 0    60   ~ 0
 ~SD
 $Comp
-L GND #PWR026
+L GND #PWR022
 U 1 1 5898CF87
-P 3250 3900
-F 0 "#PWR026" H 3250 3650 50  0001 C CNN
-F 1 "GND" H 3250 3750 50  0000 C CNN
-F 2 "" H 3250 3900 50  0000 C CNN
-F 3 "" H 3250 3900 50  0000 C CNN
-	1    3250 3900
-	1    0    0    -1
-$EndComp
-$Comp
-L +5V #PWR027
+P 2750 4450
+F 0 "#PWR022" H 2750 4200 50  0001 C CNN
+F 1 "GND" H 2750 4300 50  0000 C CNN
+F 2 "" H 2750 4450 50  0000 C CNN
+F 3 "" H 2750 4450 50  0000 C CNN
+	1    2750 4450
+	1    0    0    -1
+$EndComp
+$Comp
+L +5V #PWR023
 U 1 1 5898CF88
-P 3250 3750
-F 0 "#PWR027" H 3250 3600 50  0001 C CNN
-F 1 "+5V" H 3250 3890 50  0000 C CNN
-F 2 "" H 3250 3750 50  0000 C CNN
-F 3 "" H 3250 3750 50  0000 C CNN
-	1    3250 3750
-	1    0    0    -1
-$EndComp
-$Comp
-L GND #PWR028
+P 2750 4250
+F 0 "#PWR023" H 2750 4100 50  0001 C CNN
+F 1 "+5V" H 2750 4390 50  0000 C CNN
+F 2 "" H 2750 4250 50  0000 C CNN
+F 3 "" H 2750 4250 50  0000 C CNN
+	1    2750 4250
+	1    0    0    -1
+$EndComp
+$Comp
+L GND #PWR024
 U 1 1 5898CF89
 P 7300 3600
-F 0 "#PWR028" H 7300 3350 50  0001 C CNN
+F 0 "#PWR024" H 7300 3350 50  0001 C CNN
 F 1 "GND" H 7300 3450 50  0000 C CNN
 F 2 "" H 7300 3600 50  0000 C CNN
@@
 $EndComp
 $Comp
-L +5V #PWR029
+L +5V #PWR025
 U 1 1 5898CF8A
 P 7150 3700
-F 0 "#PWR029" H 7150 3550 50  0001 C CNN
+F 0 "#PWR025" H 7150 3550 50  0001 C CNN
 F 1 "+5V" H 7150 3840 50  0000 C CNN
 F 2 "" H 7150 3700 50  0000 C CNN
@@
 $EndComp
 $Comp
-L GND #PWR030
+L GND #PWR026
 U 1 1 5898CF90
 P 8200 3700
-F 0 "#PWR030" H 8200 3450 50  0001 C CNN
+F 0 "#PWR026" H 8200 3450 50  0001 C CNN
 F 1 "GND" H 8200 3550 50  0000 C CNN
 F 2 "" H 8200 3700 50  0000 C CNN
@@
 $EndComp
 $Comp
-L GND #PWR031
+L GND #PWR027
 U 1 1 5898CF92
 P 8200 4500
-F 0 "#PWR031" H 8200 4250 50  0001 C CNN
+F 0 "#PWR027" H 8200 4250 50  0001 C CNN
 F 1 "GND" H 8200 4350 50  0000 C CNN
 F 2 "" H 8200 4500 50  0000 C CNN
@@
 Text Label 5950 3500 0    60   ~ 0
 ~SD
-Text Label 3800 4950 2    60   ~ 0
+Text Label 5450 5000 2    60   ~ 0
 ~SD
 $Comp
-L +5V #PWR032
+L +5V #PWR028
 U 1 1 589F6407
-P 3050 4850
-F 0 "#PWR032" H 3050 4700 50  0001 C CNN
-F 1 "+5V" H 3050 4990 50  0000 C CNN
-F 2 "" H 3050 4850 50  0000 C CNN
-F 3 "" H 3050 4850 50  0000 C CNN
-	1    3050 4850
-	1    0    0    -1
-$EndComp
-$Comp
-L GND #PWR033
+P 4700 4900
+F 0 "#PWR028" H 4700 4750 50  0001 C CNN
+F 1 "+5V" H 4700 5040 50  0000 C CNN
+F 2 "" H 4700 4900 50  0000 C CNN
+F 3 "" H 4700 4900 50  0000 C CNN
+	1    4700 4900
+	1    0    0    -1
+$EndComp
+$Comp
+L GND #PWR029
 U 1 1 589F6490
-P 3050 5500
-F 0 "#PWR033" H 3050 5250 50  0001 C CNN
-F 1 "GND" H 3050 5350 50  0000 C CNN
-F 2 "" H 3050 5500 50  0000 C CNN
-F 3 "" H 3050 5500 50  0000 C CNN
-	1    3050 5500
-	1    0    0    -1
-$EndComp
-$Comp
-L CONN_01X05 P1
-U 1 1 58A0B165
-P 2700 3700
-F 0 "P1" H 2700 4000 50  0000 C CNN
-F 1 "CONN_01X05" V 2800 3700 50  0000 C CNN
-F 2 "" H 2700 3700 50  0001 C CNN
-F 3 "" H 2700 3700 50  0000 C CNN
-	1    2700 3700
-	-1   0    0    1
-$EndComp
-Wire Wire Line
-	3050 5350 3050 5500
+P 4700 5550
+F 0 "#PWR029" H 4700 5300 50  0001 C CNN
+F 1 "GND" H 4700 5400 50  0000 C CNN
+F 2 "" H 4700 5550 50  0000 C CNN
+F 3 "" H 4700 5550 50  0000 C CNN
+	1    4700 5550
+	1    0    0    -1
+$EndComp
+Wire Wire Line
+	4700 5400 4700 5550
 Wire Wire Line
 	5500 4150 5300 4150
@@
 Connection ~ 4650 4150
 Wire Wire Line
-	3250 3800 3250 3750
-Wire Wire Line
-	3100 3500 2900 3500
-Wire Wire Line
-	3100 3600 2900 3600
-Wire Wire Line
-	3100 3700 2900 3700
-Wire Wire Line
-	2900 3800 3250 3800
-Wire Wire Line
-	2900 3900 3250 3900
+	2750 3300 2550 3300
+Wire Wire Line
+	2750 3400 2550 3400
+Wire Wire Line
+	2750 4350 2550 4350
 Wire Wire Line
 	7300 3600 7100 3600
@@
 	6100 3500 5850 3500
 Wire Wire Line
-	3050 4850 3050 5050
+	4700 4900 4700 5100
 $Comp
 L R R1
 U 1 1 589D33B2
-P 3450 4950
-F 0 "R1" V 3530 4950 50  0000 C CNN
-F 1 "10k" V 3450 4950 50  0000 C CNN
-F 2 "Resistors_SMD:R_0805" V 3380 4950 50  0001 C CNN
-F 3 "" H 3450 4950 50  0000 C CNN
-	1    3450 4950
-	0    1    1    0
-$EndComp
-Wire Wire Line
-	2750 4950 3300 4950
-Connection ~ 3050 4950
-Wire Wire Line
-	3850 4950 3600 4950
-Text HLabel 2750 4950 0    60   Input ~ 0
+P 5100 5000
+F 0 "R1" V 5180 5000 50  0000 C CNN
+F 1 "10k" V 5100 5000 50  0000 C CNN
+F 2 "Resistors_SMD:R_0805" V 5030 5000 50  0001 C CNN
+F 3 "" H 5100 5000 50  0000 C CNN
+	1    5100 5000
+	0    1    1    0
+$EndComp
+Wire Wire Line
+	4400 5000 4950 5000
+Connection ~ 4700 5000
+Wire Wire Line
+	5500 5000 5250 5000
+Text HLabel 4400 5000 0    60   Input ~ 0
 ~SD
+$Comp
+L GND #PWR030
+U 1 1 589F56B8
+P 2750 3500
+F 0 "#PWR030" H 2750 3250 50  0001 C CNN
+F 1 "GND" H 2750 3350 50  0000 C CNN
+F 2 "" H 2750 3500 50  0000 C CNN
+F 3 "" H 2750 3500 50  0000 C CNN
+	1    2750 3500
+	1    0    0    -1
+$EndComp
+$Comp
+L CONN_01X03 P1
+U 1 1 589F6E36
+P 2350 3400
+F 0 "P1" H 2350 3600 50  0000 C CNN
+F 1 "CONN_01X03" V 2450 3400 50  0000 C CNN
+F 2 "Socket_Strips:Socket_Strip_Straight_1x03_Pitch2.54mm" H 2350 3400 50  0001 C CNN
+F 3 "" H 2350 3400 50  0000 C CNN
+	1    2350 3400
+	-1   0    0    -1
+$EndComp
+$Comp
+L CONN_01X03 P5
+U 1 1 589F6FB9
+P 2350 4350
+F 0 "P5" H 2350 4550 50  0000 C CNN
+F 1 "CONN_01X03" V 2450 4350 50  0000 C CNN
+F 2 "Socket_Strips:Socket_Strip_Straight_1x03_Pitch2.54mm" H 2350 4350 50  0001 C CNN
+F 3 "" H 2350 4350 50  0000 C CNN
+	1    2350 4350
+	-1   0    0    -1
+$EndComp
+Wire Wire Line
+	2750 4250 2550 4250
+Wire Wire Line
+	2750 4450 2550 4450
+Wire Wire Line
+	2550 3500 2750 3500
 $EndSCHEMATC

Commit message: Actualizacion ref. DigitKey
by Rubén
Parts:
- U1: value PAM8302A -> PAM8302AASCR; DIGIKEY REF (none) -> PAM8302AASCRDI-ND
Changed lines of the file:
@@
 P 6600 3650
 F 0 "U1" H 6600 3950 60  0000 C CNN
-F 1 "PAM8302A" H 6600 3350 60  0000 C CNN
+F 1 "PAM8302AASCR" H 6600 3350 60  0000 C CNN
 F 2 "Housings_SSOP:MSOP-8_3x3mm_Pitch0.65mm" H 6600 3950 60  0001 C CNN
-F 3 "" H 6600 3950 60  0001 C CNN
+F 3 "https://www.diodes.com/assets/Datasheets/PAM8302A.pdf" H 6600 3950 60  0001 C CNN
+F 4 "PAM8302AASCRDI-ND" H 6600 3650 60  0001 C CNN "DIGIKEY REF"
 	1    6600 3650
 	1    0    0    -1
