File: hard/hw/Basic_pcb/Audio.sch (KiCad schematic (older format))
At the start: 15 parts, among them P1 CONN_01X03, P2 CONN_01X02, P5 CONN_01X03, U1 PAM8302AASCR

Commit message: Organizando PIN OUT vr.:0.1
by Ruben
Parts:
- P1: footprint Socket_Strips:Socket_Strip_Straight_1x03_Pitch2.54mm -> Socket_Strips:Socket_Strip_Straight_1x03_Pitch1.27mm
- RV1: REF DIGIKEY (none) -> 3135X103P-ND
Connections:
- wire segments 36 -> 35
Changed lines of the file:
@@
 F 0 "RV1" V 4475 3700 50  0000 C CNN
 F 1 "10K POT_TRIM" V 4550 3700 50  0000 C CNN
-F 2 "Potentiometers:Potentiometer_Trimmer-EVM3E" V 4400 3700 50  0001 C CNN
-F 3 "" H 4650 3700 50  0000 C CNN
+F 2 "Potentiometers:Potentiometer_Trimmer-EVM3E" H 4400 3700 50  0001 C CNN
+F 3 "http://www.te.com/commerce/DocumentDelivery/DDEController?Action=srchrtrv&DocNm=1623919&DocType=Customer+Drawing&DocLang=English" H 4650 3700 50  0001 C CNN
+F 4 "3135X103P-ND" V 4650 3700 60  0001 C CNN "REF DIGIKEY"
 	1    4650 3700
 	1    0    0    -1
@@
 	1    0    0    -1
 $EndComp
-$Comp
-L CONN_01X02 P2
-U 1 1 5898CF86
-P 8800 3650
-F 0 "P2" H 8800 3800 50  0000 C CNN
-F 1 "CONN_01X02" V 8900 3650 50  0000 C CNN
-F 2 "Socket_Strips:Socket_Strip_Straight_1x02_Pitch2.54mm" H 8800 3650 50  0001 C CNN
-F 3 "" H 8800 3650 50  0000 C CNN
-	1    8800 3650
-	1    0    0    -1
-$EndComp
-Text Label 2600 3300 0    60   ~ 0
-AIN+
-Text Label 2600 3400 0    60   ~ 0
-AIN-
-Text Label 2600 4350 0    60   ~ 0
+Text Label 2700 4350 0    60   ~ 0
 ~SD
 $Comp
-L GND #PWR022
+L GND #PWR019
 U 1 1 5898CF87
 P 2750 4450
-F 0 "#PWR022" H 2750 4200 50  0001 C CNN
+F 0 "#PWR019" H 2750 4200 50  0001 C CNN
 F 1 "GND" H 2750 4300 50  0000 C CNN
 F 2 "" H 2750 4450 50  0000 C CNN
@@
 $EndComp
 $Comp
-L +5V #PWR023
+L +5V #PWR020
 U 1 1 5898CF88
 P 2750 4250
-F 0 "#PWR023" H 2750 4100 50  0001 C CNN
+F 0 "#PWR020" H 2750 4100 50  0001 C CNN
 F 1 "+5V" H 2750 4390 50  0000 C CNN
 F 2 "" H 2750 4250 50  0000 C CNN
@@
 $EndComp
 $Comp
-L GND #PWR024
+L GND #PWR021
 U 1 1 5898CF89
 P 7300 3600
-F 0 "#PWR024" H 7300 3350 50  0001 C CNN
+F 0 "#PWR021" H 7300 3350 50  0001 C CNN
 F 1 "GND" H 7300 3450 50  0000 C CNN
 F 2 "" H 7300 3600 50  0000 C CNN
@@
 $EndComp
 $Comp
-L +5V #PWR025
+L +5V #PWR022
 U 1 1 5898CF8A
 P 7150 3700
-F 0 "#PWR025" H 7150 3550 50  0001 C CNN
+F 0 "#PWR022" H 7150 3550 50  0001 C CNN
 F 1 "+5V" H 7150 3840 50  0000 C CNN
 F 2 "" H 7150 3700 50  0000 C CNN
@@
 $EndComp
 $Comp
-L GND #PWR026
+L GND #PWR023
 U 1 1 5898CF90
 P 8200 3700
-F 0 "#PWR026" H 8200 3450 50  0001 C CNN
+F 0 "#PWR023" H 8200 3450 50  0001 C CNN
 F 1 "GND" H 8200 3550 50  0000 C CNN
 F 2 "" H 8200 3700 50  0000 C CNN
@@
 $EndComp
 $Comp
-L GND #PWR027
+L GND #PWR024
 U 1 1 5898CF92
 P 8200 4500
-F 0 "#PWR027" H 8200 4250 50  0001 C CNN
+F 0 "#PWR024" H 8200 4250 50  0001 C CNN
 F 1 "GND" H 8200 4350 50  0000 C CNN
 F 2 "" H 8200 4500 50  0000 C CNN
@@
 ~SD
 $Comp
-L +5V #PWR028
+L +5V #PWR025
 U 1 1 589F6407
 P 4700 4900
-F 0 "#PWR028" H 4700 4750 50  0001 C CNN
+F 0 "#PWR025" H 4700 4750 50  0001 C CNN
 F 1 "+5V" H 4700 5040 50  0000 C CNN
 F 2 "" H 4700 4900 50  0000 C CNN
@@
 $EndComp
 $Comp
-L GND #PWR029
+L GND #PWR026
 U 1 1 589F6490
 P 4700 5550
-F 0 "#PWR029" H 4700 5300 50  0001 C CNN
+F 0 "#PWR026" H 4700 5300 50  0001 C CNN
 F 1 "GND" H 4700 5400 50  0000 C CNN
 F 2 "" H 4700 5550 50  0000 C CNN
@@
 	1    0    0    -1
 $EndComp
-Wire Wire Line
-	4700 5400 4700 5550
-Wire Wire Line
-	5500 4150 5300 4150
-Wire Wire Line
-	5500 3700 5300 3700
-Wire Wire Line
-	7800 4000 8600 4000
-Wire Wire Line
-	7800 3250 8600 3250
-Connection ~ 4650 4150
-Wire Wire Line
-	2750 3300 2550 3300
-Wire Wire Line
-	2750 3400 2550 3400
-Wire Wire Line
-	2750 4350 2550 4350
-Wire Wire Line
-	7300 3600 7100 3600
-Wire Wire Line
-	7150 3700 7100 3700
-Wire Wire Line
-	6100 3700 5800 3700
-Wire Wire Line
-	6100 3800 6100 4150
-Wire Wire Line
-	6100 4150 5800 4150
-Wire Wire Line
-	5000 3700 4800 3700
-Wire Wire Line
-	4650 3850 4650 4150
-Wire Wire Line
-	4350 4150 5000 4150
-Wire Wire Line
-	4650 3550 4650 3300
-Wire Wire Line
-	7500 3250 7250 3250
-Wire Wire Line
-	7250 3250 7250 3500
-Wire Wire Line
-	7250 3500 7100 3500
-Wire Wire Line
-	7500 4000 7250 4000
-Wire Wire Line
-	7250 4000 7250 3800
-Wire Wire Line
-	7250 3800 7100 3800
-Connection ~ 8200 4000
-Wire Wire Line
-	8200 4400 8200 4500
-Wire Wire Line
-	8200 3350 8200 3250
-Wire Wire Line
-	8200 3650 8200 3700
-Wire Wire Line
-	8200 4000 8200 4100
-Connection ~ 8200 3250
-Wire Wire Line
-	8600 3250 8600 3600
-Wire Wire Line
-	8600 4000 8600 3700
-Wire Wire Line
-	6100 3500 5850 3500
-Wire Wire Line
-	4700 4900 4700 5100
 $Comp
 L R R1
@@
 	0    1    1    0
 $EndComp
-Wire Wire Line
-	4400 5000 4950 5000
-Connection ~ 4700 5000
-Wire Wire Line
-	5500 5000 5250 5000
-Text HLabel 4400 5000 0    60   Input ~ 0
+Text HLabel 2900 4350 2    60   Input ~ 0
 ~SD
 $Comp
-L GND #PWR030
+L GND #PWR027
 U 1 1 589F56B8
 P 2750 3500
-F 0 "#PWR030" H 2750 3250 50  0001 C CNN
+F 0 "#PWR027" H 2750 3250 50  0001 C CNN
 F 1 "GND" H 2750 3350 50  0000 C CNN
 F 2 "" H 2750 3500 50  0000 C CNN
@@
 F 0 "P1" H 2350 3600 50  0000 C CNN
 F 1 "CONN_01X03" V 2450 3400 50  0000 C CNN
-F 2 "Socket_Strips:Socket_Strip_Straight_1x03_Pitch2.54mm" H 2350 3400 50  0001 C CNN
+F 2 "Socket_Strips:Socket_Strip_Straight_1x03_Pitch1.27mm" H 2350 3400 50  0001 C CNN
 F 3 "" H 2350 3400 50  0000 C CNN
 	1    2350 3400
@@
 	-1   0    0    -1
 $EndComp
+Text Label 2600 3400 0    60   ~ 0
+AIN-
+Text Label 2600 3300 0    60   ~ 0
+AIN+
+Wire Wire Line
+	4700 5400 4700 5550
+Wire Wire Line
+	5500 4150 5300 4150
+Wire Wire Line
+	5500 3700 5300 3700
+Wire Wire Line
+	7800 4000 8600 4000
+Wire Wire Line
+	7800 3250 8600 3250
+Connection ~ 4650 4150
+Wire Wire Line
+	2750 3300 2550 3300
+Wire Wire Line
+	2750 3400 2550 3400
+Wire Wire Line
+	7300 3600 7100 3600
+Wire Wire Line
+	7150 3700 7100 3700
+Wire Wire Line
+	6100 3700 5800 3700
+Wire Wire Line
+	6100 3800 6100 4150
+Wire Wire Line
+	6100 4150 5800 4150
+Wire Wire Line
+	5000 3700 4800 3700
+Wire Wire Line
+	4650 3850 4650 4150
+Wire Wire Line
+	4350 4150 5000 4150
+Wire Wire Line
+	4650 3550 4650 3300
+Wire Wire Line
+	7500 3250 7250 3250
+Wire Wire Line
+	7250 3250 7250 3500
+Wire Wire Line
+	7250 3500 7100 3500
+Wire Wire Line
+	7500 4000 7250 4000
+Wire Wire Line
+	7250 4000 7250 3800
+Wire Wire Line
+	7250 3800 7100 3800
+Connection ~ 8200 4000
+Wire Wire Line
+	8200 4400 8200 4500
+Wire Wire Line
+	8200 3350 8200 3250
+Wire Wire Line
+	8200 3650 8200 3700
+Wire Wire Line
+	8200 4000 8200 4100
+Connection ~ 8200 3250
+Wire Wire Line
+	8600 3250 8600 3600
+Wire Wire Line
+	8600 4000 8600 3700
+Wire Wire Line
+	6100 3500 5850 3500
+Wire Wire Line
+	4700 4900 4700 5100
+Connection ~ 4700 5000
+Wire Wire Line
+	5500 5000 5250 5000
 Wire Wire Line
 	2750 4250 2550 4250
@@
 Wire Wire Line
 	2550 3500 2750 3500
+$Comp
+L CONN_01X02 P2
+U 1 1 5898CF86
+P 8800 3650
+F 0 "P2" H 8800 3800 50  0000 C CNN
+F 1 "CONN_01X02" V 8900 3650 50  0000 C CNN
+F 2 "Socket_Strips:Socket_Strip_Straight_1x02_Pitch2.54mm" H 8800 3650 50  0001 C CNN
+F 3 "" H 8800 3650 50  0000 C CNN
+	1    8800 3650
+	1    0    0    -1
+$EndComp
+Wire Wire Line
+	2900 4350 2550 4350
 $EndSCHEMATC

Commit message: Terminado Shield
by Ruben
Connections:
- wire segments 35 -> 36
Changed lines of the file:
@@
 Wire Wire Line
 	2900 4350 2550 4350
+Wire Wire Line
+	4950 5000 4700 5000
 $EndSCHEMATC
