File: hard/hw/Basic_pcb/serial_interface.sch (KiCad schematic (older format))
At the start: 20 parts

Commit message: Actualizacion Power
Parts:
- removed PS1: BARREL_JACK, Connect:JACK_ALIM, symbol BARREL_JACK
Connections:
- wire segments 92 -> 88
Changed lines of the file:
@@
 LIBS:rj45_stamp
 LIBS:HDMIspartan6_Board-cache
-LIBS:pam8302-cache
 EELAYER 25 0
 EELAYER END
 $Descr A3 16535 11693
 encoding utf-8
-Sheet 3 5
+Sheet 2 5
 Title ""
 Date "9 aug 2012"
@@
 	8250 3900 9600 3900
 $Comp
-L GND #PWR047
+L GND #PWR036
 U 1 1 4FC6CFCA
 P 11500 6700
-F 0 "#PWR047" H 11500 6700 30  0001 C CNN
+F 0 "#PWR036" H 11500 6700 30  0001 C CNN
 F 1 "GND" H 11500 6630 30  0001 C CNN
 F 2 "" H 11500 6700 60  0001 C CNN
@@
 $EndComp
 $Comp
-L GND #PWR048
+L GND #PWR037
 U 1 1 4FC6CFB6
 P 8850 5200
-F 0 "#PWR048" H 8850 5200 30  0001 C CNN
+F 0 "#PWR037" H 8850 5200 30  0001 C CNN
 F 1 "GND" H 8850 5130 30  0001 C CNN
 F 2 "" H 8850 5200 60  0001 C CNN
@@
 P 13500 6100
 AR Path="/4FC6C4A2" Ref="#PWR061"  Part="1"
-AR Path="/555AB8C7/4FC6C4A2" Ref="#PWR049"  Part="1"
-F 0 "#PWR049" H 13500 6050 20  0001 C CNN
+AR Path="/555AB8C7/4FC6C4A2" Ref="#PWR038"  Part="1"
+F 0 "#PWR038" H 13500 6050 20  0001 C CNN
 F 1 "+3.3V" H 13500 6200 30  0000 C CNN
 F 2 "" H 13500 6100 60  0001 C CNN
@@
 P 13500 4600
 AR Path="/4FC6C462" Ref="#PWR062"  Part="1"
-AR Path="/555AB8C7/4FC6C462" Ref="#PWR050"  Part="1"
-F 0 "#PWR050" H 13500 4550 20  0001 C CNN
+AR Path="/555AB8C7/4FC6C462" Ref="#PWR039"  Part="1"
+F 0 "#PWR039" H 13500 4550 20  0001 C CNN
 F 1 "+3.3V" H 13500 4700 30  0000 C CNN
 F 2 "" H 13500 4600 60  0001 C CNN
@@
 $EndComp
 $Comp
-L GND #PWR051
+L GND #PWR040
 U 1 1 4FC6C3D8
 P 10650 5750
-F 0 "#PWR051" H 10650 5750 30  0001 C CNN
+F 0 "#PWR040" H 10650 5750 30  0001 C CNN
 F 1 "GND" H 10650 5680 30  0001 C CNN
 F 2 "" H 10650 5750 60  0001 C CNN
@@
 $EndComp
 $Comp
-L GND #PWR052
+L GND #PWR041
 U 1 1 4FC6C3BF
 P 10250 3350
-F 0 "#PWR052" H 10250 3350 30  0001 C CNN
+F 0 "#PWR041" H 10250 3350 30  0001 C CNN
 F 1 "GND" H 10250 3280 30  0001 C CNN
 F 2 "" H 10250 3350 60  0001 C CNN
@@
 $EndComp
 $Comp
-L +5VA #PWR053
+L +5VA #PWR042
 U 1 1 4FC6C374
 P 10150 4700
-F 0 "#PWR053" H 10150 4830 20  0001 C CNN
+F 0 "#PWR042" H 10150 4830 20  0001 C CNN
 F 1 "+5VA" H 10150 4800 30  0000 C CNN
 F 2 "" H 10150 4700 60  0001 C CNN
@@
 $EndComp
 $Comp
-L +5V #PWR054
+L +5V #PWR043
 U 1 1 4FC6C320
 P 9650 1650
-F 0 "#PWR054" H 9650 1740 20  0001 C CNN
+F 0 "#PWR043" H 9650 1740 20  0001 C CNN
 F 1 "+5V" H 9650 1740 30  0000 C CNN
 F 2 "" H 9650 1650 60  0001 C CNN
@@
 $EndComp
 $Comp
-L GND #PWR055
+L GND #PWR044
 U 1 1 4FC6C2CD
 P 10450 2200
-F 0 "#PWR055" H 10450 2200 30  0001 C CNN
+F 0 "#PWR044" H 10450 2200 30  0001 C CNN
 F 1 "GND" H 10450 2130 30  0001 C CNN
 F 2 "" H 10450 2200 60  0001 C CNN
@@
 $EndComp
 $Comp
-L +5VA #PWR056
+L +5VA #PWR045
 U 1 1 4FC6C137
 P 10850 1700
-F 0 "#PWR056" H 10850 1830 20  0001 C CNN
+F 0 "#PWR045" H 10850 1830 20  0001 C CNN
 F 1 "+5VA" H 10850 1800 30  0000 C CNN
 F 2 "" H 10850 1700 60  0001 C CNN
@@
 $EndComp
 $Comp
-L GND #PWR057
+L GND #PWR046
 U 1 1 4FC6C11B
 P 9650 2150
-F 0 "#PWR057" H 9650 2150 30  0001 C CNN
+F 0 "#PWR046" H 9650 2150 30  0001 C CNN
 F 1 "GND" H 9650 2080 30  0001 C CNN
 F 2 "" H 9650 2150 60  0001 C CNN
@@
 P 12000 2800
 AR Path="/4FC6C10C" Ref="#PWR070"  Part="1"
-AR Path="/555AB8C7/4FC6C10C" Ref="#PWR058"  Part="1"
-F 0 "#PWR058" H 12000 2750 20  0001 C CNN
+AR Path="/555AB8C7/4FC6C10C" Ref="#PWR047"  Part="1"
+F 0 "#PWR047" H 12000 2750 20  0001 C CNN
 F 1 "+3.3V" H 12000 2900 30  0000 C CNN
 F 2 "" H 12000 2800 60  0001 C CNN
@@
 $EndComp
 $Comp
-L +5VA #PWR059
+L +5VA #PWR048
 U 1 1 4FC6BDF3
 P 9900 5500
-F 0 "#PWR059" H 9900 5630 20  0001 C CNN
+F 0 "#PWR048" H 9900 5630 20  0001 C CNN
 F 1 "+5VA" H 9900 5600 30  0000 C CNN
 F 2 "" H 9900 5500 60  0001 C CNN
@@
 $EndComp
 $Comp
-L GND #PWR060
+L GND #PWR049
 U 1 1 4FC6BCE8
 P 11100 2650
-F 0 "#PWR060" H 11100 2650 30  0001 C CNN
+F 0 "#PWR049" H 11100 2650 30  0001 C CNN
 F 1 "GND" H 11100 2580 30  0001 C CNN
 F 2 "" H 11100 2650 60  0001 C CNN
@@
 P 10250 2900
 AR Path="/4FC6BCE7" Ref="#PWR073"  Part="1"
-AR Path="/555AB8C7/4FC6BCE7" Ref="#PWR061"  Part="1"
-F 0 "#PWR061" H 10250 2850 20  0001 C CNN
+AR Path="/555AB8C7/4FC6BCE7" Ref="#PWR050"  Part="1"
+F 0 "#PWR050" H 10250 2850 20  0001 C CNN
 F 1 "+3.3V" H 10250 3000 30  0000 C CNN
 F 2 "" H 10250 2900 60  0001 C CNN
@@
 $EndComp
 $Comp
-L VDD5V #PWR062
+L VDD5V #PWR051
 U 1 1 51CC37E0
 P 9500 1650
-F 0 "#PWR062" H 9500 1750 30  0001 C CNN
+F 0 "#PWR051" H 9500 1750 30  0001 C CNN
 F 1 "VDD5V" H 9500 1750 30  0000 C CNN
 F 2 "" H 9500 1650 60  0001 C CNN
@@
 P 13700 4000
 AR Path="/51CD7AF5" Ref="#PWR075"  Part="1"
-AR Path="/555AB8C7/51CD7AF5" Ref="#PWR063"  Part="1"
-F 0 "#PWR063" H 13700 3950 20  0001 C CNN
+AR Path="/555AB8C7/51CD7AF5" Ref="#PWR052"  Part="1"
+F 0 "#PWR052" H 13700 3950 20  0001 C CNN
 F 1 "+3.3V" H 13700 4100 30  0000 C CNN
 F 2 "" H 13700 4000 60  0001 C CNN
@@
 	8250 4100 8000 4100
 $Comp
-L VDD5V #PWR064
-U 1 1 555AD256
-P 7750 5650
-F 0 "#PWR064" H 7750 5750 30  0001 C CNN
-F 1 "VDD5V" H 7750 5750 30  0000 C CNN
-F 2 "" H 7750 5650 60  0001 C CNN
-F 3 "" H 7750 5650 60  0001 C CNN
-	1    7750 5650
-	1    0    0    -1
-$EndComp
-$Comp
-L GND #PWR065
-U 1 1 555AD25C
-P 7750 6000
-F 0 "#PWR065" H 7750 6000 30  0001 C CNN
-F 1 "GND" H 7750 5930 30  0001 C CNN
-F 2 "" H 7750 6000 60  0001 C CNN
-F 3 "" H 7750 6000 60  0001 C CNN
-	1    7750 6000
-	1    0    0    -1
-$EndComp
-Wire Wire Line
-	7750 5650 7750 5750
-Wire Wire Line
-	7750 5750 7550 5750
-Wire Wire Line
-	7550 5950 7750 5950
-Wire Wire Line
-	7750 5950 7750 6000
-$Comp
-L BARREL_JACK PS1
-U 1 1 555AD266
-P 7250 5850
-F 0 "PS1" H 7250 6100 60  0000 C CNN
-F 1 "BARREL_JACK" H 7250 5650 60  0000 C CNN
-F 2 "Connect:JACK_ALIM" H 7250 5850 60  0001 C CNN
-F 3 "" H 7250 5850 60  0000 C CNN
-	1    7250 5850
-	1    0    0    -1
-$EndComp
-$Comp
-L GND #PWR066
+L GND #PWR055
 U 1 1 555AD26D
 P 8200 4350
-F 0 "#PWR066" H 8200 4350 30  0001 C CNN
+F 0 "#PWR055" H 8200 4350 30  0001 C CNN
 F 1 "GND" H 8200 4280 30  0001 C CNN
 F 2 "" H 8200 4350 60  0001 C CNN
@@
 Connection ~ 8100 5900
 $Comp
-L GND #PWR067
+L GND #PWR056
 U 1 1 555AD27C
 P 8100 6050
-F 0 "#PWR067" H 8100 6050 30  0001 C CNN
+F 0 "#PWR056" H 8100 6050 30  0001 C CNN
 F 1 "GND" H 8100 5980 30  0001 C CNN
 F 2 "" H 8100 6050 60  0001 C CNN
@@
 $EndComp
 $Comp
-L VDD5V #PWR068
+L VDD5V #PWR057
 U 1 1 555AD28D
 P 8150 3300
-F 0 "#PWR068" H 8150 3400 30  0001 C CNN
+F 0 "#PWR057" H 8150 3400 30  0001 C CNN
 F 1 "VDD5V" H 8150 3400 30  0000 C CNN
 F 2 "" H 8150 3300 60  0001 C CNN
@@
 	8150 3900 8150 3800
 $Comp
-L GND #PWR069
+L GND #PWR058
 U 1 1 555AD296
 P 6850 4350
-F 0 "#PWR069" H 6850 4350 30  0001 C CNN
+F 0 "#PWR058" H 6850 4350 30  0001 C CNN
 F 1 "GND" H 6850 4280 30  0001 C CNN
 F 2 "" H 6850 4350 60  0001 C CNN

Commit message: Fuente 12V
by Luis Yaya
Parts:
- added P3: CONN_02X02, symbol CONN_02X02
Connections:
- wire segments 88 -> 83
Changed lines of the file:
@@
 LIBS:rj45_stamp
 LIBS:HDMIspartan6_Board-cache
-LIBS:fuente-cache
 EELAYER 25 0
 EELAYER END
@@
 	8250 3900 9600 3900
 $Comp
-L GND #PWR036
+L GND #PWR06
 U 1 1 4FC6CFCA
 P 11500 6700
-F 0 "#PWR036" H 11500 6700 30  0001 C CNN
+F 0 "#PWR06" H 11500 6700 30  0001 C CNN
 F 1 "GND" H 11500 6630 30  0001 C CNN
 F 2 "" H 11500 6700 60  0001 C CNN
@@
 $EndComp
 $Comp
-L GND #PWR037
+L GND #PWR07
 U 1 1 4FC6CFB6
 P 8850 5200
-F 0 "#PWR037" H 8850 5200 30  0001 C CNN
+F 0 "#PWR07" H 8850 5200 30  0001 C CNN
 F 1 "GND" H 8850 5130 30  0001 C CNN
 F 2 "" H 8850 5200 60  0001 C CNN
@@
 P 13500 6100
 AR Path="/4FC6C4A2" Ref="#PWR061"  Part="1"
-AR Path="/555AB8C7/4FC6C4A2" Ref="#PWR038"  Part="1"
-F 0 "#PWR038" H 13500 6050 20  0001 C CNN
+AR Path="/555AB8C7/4FC6C4A2" Ref="#PWR08"  Part="1"
+F 0 "#PWR08" H 13500 6050 20  0001 C CNN
 F 1 "+3.3V" H 13500 6200 30  0000 C CNN
 F 2 "" H 13500 6100 60  0001 C CNN
@@
 P 13500 4600
 AR Path="/4FC6C462" Ref="#PWR062"  Part="1"
-AR Path="/555AB8C7/4FC6C462" Ref="#PWR039"  Part="1"
-F 0 "#PWR039" H 13500 4550 20  0001 C CNN
+AR Path="/555AB8C7/4FC6C462" Ref="#PWR09"  Part="1"
+F 0 "#PWR09" H 13500 4550 20  0001 C CNN
 F 1 "+3.3V" H 13500 4700 30  0000 C CNN
 F 2 "" H 13500 4600 60  0001 C CNN
@@
 $EndComp
 $Comp
-L GND #PWR040
+L GND #PWR010
 U 1 1 4FC6C3D8
 P 10650 5750
-F 0 "#PWR040" H 10650 5750 30  0001 C CNN
+F 0 "#PWR010" H 10650 5750 30  0001 C CNN
 F 1 "GND" H 10650 5680 30  0001 C CNN
 F 2 "" H 10650 5750 60  0001 C CNN
@@
 $EndComp
 $Comp
-L GND #PWR041
+L GND #PWR011
 U 1 1 4FC6C3BF
 P 10250 3350
-F 0 "#PWR041" H 10250 3350 30  0001 C CNN
+F 0 "#PWR011" H 10250 3350 30  0001 C CNN
 F 1 "GND" H 10250 3280 30  0001 C CNN
 F 2 "" H 10250 3350 60  0001 C CNN
@@
 $EndComp
 $Comp
-L +5VA #PWR042
+L +5VA #PWR012
 U 1 1 4FC6C374
 P 10150 4700
-F 0 "#PWR042" H 10150 4830 20  0001 C CNN
+F 0 "#PWR012" H 10150 4830 20  0001 C CNN
 F 1 "+5VA" H 10150 4800 30  0000 C CNN
 F 2 "" H 10150 4700 60  0001 C CNN
@@
 $EndComp
 $Comp
-L +5V #PWR043
+L +5V #PWR013
 U 1 1 4FC6C320
 P 9650 1650
-F 0 "#PWR043" H 9650 1740 20  0001 C CNN
+F 0 "#PWR013" H 9650 1740 20  0001 C CNN
 F 1 "+5V" H 9650 1740 30  0000 C CNN
 F 2 "" H 9650 1650 60  0001 C CNN
@@
 $EndComp
 $Comp
-L GND #PWR044
+L GND #PWR014
 U 1 1 4FC6C2CD
 P 10450 2200
-F 0 "#PWR044" H 10450 2200 30  0001 C CNN
+F 0 "#PWR014" H 10450 2200 30  0001 C CNN
 F 1 "GND" H 10450 2130 30  0001 C CNN
 F 2 "" H 10450 2200 60  0001 C CNN
@@
 $EndComp
 $Comp
-L +5VA #PWR045
+L +5VA #PWR015
 U 1 1 4FC6C137
 P 10850 1700
-F 0 "#PWR045" H 10850 1830 20  0001 C CNN
+F 0 "#PWR015" H 10850 1830 20  0001 C CNN
 F 1 "+5VA" H 10850 1800 30  0000 C CNN
 F 2 "" H 10850 1700 60  0001 C CNN
@@
 $EndComp
 $Comp
-L GND #PWR046
+L GND #PWR016
 U 1 1 4FC6C11B
 P 9650 2150
-F 0 "#PWR046" H 9650 2150 30  0001 C CNN
+F 0 "#PWR016" H 9650 2150 30  0001 C CNN
 F 1 "GND" H 9650 2080 30  0001 C CNN
 F 2 "" H 9650 2150 60  0001 C CNN
@@
 P 12000 2800
 AR Path="/4FC6C10C" Ref="#PWR070"  Part="1"
-AR Path="/555AB8C7/4FC6C10C" Ref="#PWR047"  Part="1"
-F 0 "#PWR047" H 12000 2750 20  0001 C CNN
+AR Path="/555AB8C7/4FC6C10C" Ref="#PWR017"  Part="1"
+F 0 "#PWR017" H 12000 2750 20  0001 C CNN
 F 1 "+3.3V" H 12000 2900 30  0000 C CNN
 F 2 "" H 12000 2800 60  0001 C CNN
@@
 $EndComp
 $Comp
-L +5VA #PWR048
+L +5VA #PWR018
 U 1 1 4FC6BDF3
 P 9900 5500
-F 0 "#PWR048" H 9900 5630 20  0001 C CNN
+F 0 "#PWR018" H 9900 5630 20  0001 C CNN
 F 1 "+5VA" H 9900 5600 30  0000 C CNN
 F 2 "" H 9900 5500 60  0001 C CNN
@@
 $EndComp
 $Comp
-L GND #PWR049
+L GND #PWR019
 U 1 1 4FC6BCE8
 P 11100 2650
-F 0 "#PWR049" H 11100 2650 30  0001 C CNN
+F 0 "#PWR019" H 11100 2650 30  0001 C CNN
 F 1 "GND" H 11100 2580 30  0001 C CNN
 F 2 "" H 11100 2650 60  0001 C CNN
@@
 P 10250 2900
 AR Path="/4FC6BCE7" Ref="#PWR073"  Part="1"
-AR Path="/555AB8C7/4FC6BCE7" Ref="#PWR050"  Part="1"
-F 0 "#PWR050" H 10250 2850 20  0001 C CNN
+AR Path="/555AB8C7/4FC6BCE7" Ref="#PWR020"  Part="1"
+F 0 "#PWR020" H 10250 2850 20  0001 C CNN
 F 1 "+3.3V" H 10250 3000 30  0000 C CNN
 F 2 "" H 10250 2900 60  0001 C CNN
@@
 $EndComp
 $Comp
-L VDD5V #PWR051
+L VDD5V #PWR021
 U 1 1 51CC37E0
 P 9500 1650
-F 0 "#PWR051" H 9500 1750 30  0001 C CNN
+F 0 "#PWR021" H 9500 1750 30  0001 C CNN
 F 1 "VDD5V" H 9500 1750 30  0000 C CNN
 F 2 "" H 9500 1650 60  0001 C CNN
@@
 P 13700 4000
 AR Path="/51CD7AF5" Ref="#PWR075"  Part="1"
-AR Path="/555AB8C7/51CD7AF5" Ref="#PWR052"  Part="1"
-F 0 "#PWR052" H 13700 3950 20  0001 C CNN
+AR Path="/555AB8C7/51CD7AF5" Ref="#PWR022"  Part="1"
+F 0 "#PWR022" H 13700 3950 20  0001 C CNN
 F 1 "+3.3V" H 13700 4100 30  0000 C CNN
 F 2 "" H 13700 4000 60  0001 C CNN
@@
 	8250 4100 8000 4100
 $Comp
-L GND #PWR055
+L GND #PWR023
 U 1 1 555AD26D
 P 8200 4350
-F 0 "#PWR055" H 8200 4350 30  0001 C CNN
+F 0 "#PWR023" H 8200 4350 30  0001 C CNN
 F 1 "GND" H 8200 4280 30  0001 C CNN
 F 2 "" H 8200 4350 60  0001 C CNN
@@
 Wire Wire Line
 	8200 4300 8200 4350
-Wire Wire Line
-	8200 5700 8100 5700
-Wire Wire Line
-	8100 5700 8100 6050
-Wire Wire Line
-	8100 5800 8200 5800
-Wire Wire Line
-	8100 5900 8200 5900
-Connection ~ 8100 5800
-Wire Wire Line
-	8100 6000 8200 6000
-Connection ~ 8100 5900
-$Comp
-L GND #PWR056
-U 1 1 555AD27C
-P 8100 6050
-F 0 "#PWR056" H 8100 6050 30  0001 C CNN
-F 1 "GND" H 8100 5980 30  0001 C CNN
-F 2 "" H 8100 6050 60  0001 C CNN
-F 3 "" H 8100 6050 60  0001 C CNN
-	1    8100 6050
-	1    0    0    -1
-$EndComp
-Connection ~ 8100 6000
 Wire Wire Line
 	6850 3950 6850 4350
@@
 $EndComp
 $Comp
-L VDD5V #PWR057
+L VDD5V #PWR024
 U 1 1 555AD28D
 P 8150 3300
-F 0 "#PWR057" H 8150 3400 30  0001 C CNN
+F 0 "#PWR024" H 8150 3400 30  0001 C CNN
 F 1 "VDD5V" H 8150 3400 30  0000 C CNN
 F 2 "" H 8150 3300 60  0001 C CNN
@@
 	8150 3900 8150 3800
 $Comp
-L GND #PWR058
+L GND #PWR025
 U 1 1 555AD296
 P 6850 4350
-F 0 "#PWR058" H 6850 4350 30  0001 C CNN
+F 0 "#PWR025" H 6850 4350 30  0001 C CNN
 F 1 "GND" H 6850 4280 30  0001 C CNN
 F 2 "" H 6850 4350 60  0001 C CNN
@@
 	10250 2850 10250 2950
 Connection ~ 10250 2900
+$Comp
+L CONN_02X02 P3
+U 1 1 5899737F
+P 7600 4900
+F 0 "P3" H 7600 5050 50  0000 C CNN
+F 1 "CONN_02X02" H 7600 4750 50  0000 C CNN
+F 2 "" H 7600 3700 50  0001 C CNN
+F 3 "" H 7600 3700 50  0000 C CNN
+	1    7600 4900
+	1    0    0    -1
+$EndComp
 $EndSCHEMATC

Commit message: Actualización PinOut LVDS
by Rubén Parra
Connections:
- net labels added: +3V3
- net labels removed: +3.3V
- wire segments 83 -> 85
Changed lines of the file:
@@
 	11900 2800 12000 2800
 Wire Wire Line
-	12000 2800 12000 3000
+	12000 2750 12000 3000
 Wire Wire Line
 	9650 2050 9650 2150
@@
 $EndComp
 $Comp
-L +3.3V #PWR061
-U 1 1 4FC6C4A2
-P 13500 6100
-AR Path="/4FC6C4A2" Ref="#PWR061"  Part="1"
-AR Path="/555AB8C7/4FC6C4A2" Ref="#PWR08"  Part="1"
-F 0 "#PWR08" H 13500 6050 20  0001 C CNN
-F 1 "+3.3V" H 13500 6200 30  0000 C CNN
-F 2 "" H 13500 6100 60  0001 C CNN
-F 3 "" H 13500 6100 60  0001 C CNN
-	1    13500 6100
-	1    0    0    -1
-$EndComp
-$Comp
-L +3.3V #PWR062
-U 1 1 4FC6C462
-P 13500 4600
-AR Path="/4FC6C462" Ref="#PWR062"  Part="1"
-AR Path="/555AB8C7/4FC6C462" Ref="#PWR09"  Part="1"
-F 0 "#PWR09" H 13500 4550 20  0001 C CNN
-F 1 "+3.3V" H 13500 4700 30  0000 C CNN
-F 2 "" H 13500 4600 60  0001 C CNN
-F 3 "" H 13500 4600 60  0001 C CNN
-	1    13500 4600
-	1    0    0    -1
-$EndComp
-$Comp
 L R RF19
 U 1 1 4FC6C443
@@
 F 3 "" H 9650 2150 60  0001 C CNN
 	1    9650 2150
-	1    0    0    -1
-$EndComp
-$Comp
-L +3.3V #PWR070
-U 1 1 4FC6C10C
-P 12000 2800
-AR Path="/4FC6C10C" Ref="#PWR070"  Part="1"
-AR Path="/555AB8C7/4FC6C10C" Ref="#PWR017"  Part="1"
-F 0 "#PWR017" H 12000 2750 20  0001 C CNN
-F 1 "+3.3V" H 12000 2900 30  0000 C CNN
-F 2 "" H 12000 2800 60  0001 C CNN
-F 3 "" H 12000 2800 60  0001 C CNN
-	1    12000 2800
 	1    0    0    -1
 $EndComp
@@
 $EndComp
 $Comp
-L +3.3V #PWR073
-U 1 1 4FC6BCE7
-P 10250 2900
-AR Path="/4FC6BCE7" Ref="#PWR073"  Part="1"
-AR Path="/555AB8C7/4FC6BCE7" Ref="#PWR020"  Part="1"
-F 0 "#PWR020" H 10250 2850 20  0001 C CNN
-F 1 "+3.3V" H 10250 3000 30  0000 C CNN
-F 2 "" H 10250 2900 60  0001 C CNN
-F 3 "" H 10250 2900 60  0001 C CNN
-	1    10250 2900
-	1    0    0    -1
-$EndComp
-$Comp
 L R RF17
 U 1 1 4FC6BC62
@@
 $EndComp
 Connection ~ 13700 4900
-$Comp
-L +3.3V #PWR075
-U 1 1 51CD7AF5
-P 13700 4000
-AR Path="/51CD7AF5" Ref="#PWR075"  Part="1"
-AR Path="/555AB8C7/51CD7AF5" Ref="#PWR022"  Part="1"
-F 0 "#PWR022" H 13700 3950 20  0001 C CNN
-F 1 "+3.3V" H 13700 4100 30  0000 C CNN
-F 2 "" H 13700 4000 60  0001 C CNN
-F 3 "" H 13700 4000 60  0001 C CNN
-	1    13700 4000
-	1    0    0    -1
-$EndComp
-Wire Wire Line
-	13700 4000 13700 4150
 Wire Wire Line
 	13300 3400 12800 3400
@@
 	1    0    0    -1
 $EndComp
+$Comp
+L +3V3 #PWR?
+U 1 1 589F5460
+P 13500 6050
+F 0 "#PWR?" H 13500 5900 50  0001 C CNN
+F 1 "+3V3" H 13500 6190 50  0000 C CNN
+F 2 "" H 13500 6050 50  0000 C CNN
+F 3 "" H 13500 6050 50  0000 C CNN
+	1    13500 6050
+	1    0    0    -1
+$EndComp
+Wire Wire Line
+	13500 6100 13500 6050
+$Comp
+L +3V3 #PWR?
+U 1 1 589F5F40
+P 13500 4350
+F 0 "#PWR?" H 13500 4200 50  0001 C CNN
+F 1 "+3V3" H 13500 4490 50  0000 C CNN
+F 2 "" H 13500 4350 50  0000 C CNN
+F 3 "" H 13500 4350 50  0000 C CNN
+	1    13500 4350
+	1    0    0    -1
+$EndComp
+Wire Wire Line
+	13500 4600 13500 4350
+$Comp
+L +3V3 #PWR?
+U 1 1 589F6257
+P 13700 4100
+F 0 "#PWR?" H 13700 3950 50  0001 C CNN
+F 1 "+3V3" H 13700 4240 50  0000 C CNN
+F 2 "" H 13700 4100 50  0000 C CNN
+F 3 "" H 13700 4100 50  0000 C CNN
+	1    13700 4100
+	1    0    0    -1
+$EndComp
+Wire Wire Line
+	13700 4100 13700 4150
+$Comp
+L +3V3 #PWR?
+U 1 1 589F6BB3
+P 12000 2750
+F 0 "#PWR?" H 12000 2600 50  0001 C CNN
+F 1 "+3V3" H 12000 2890 50  0000 C CNN
+F 2 "" H 12000 2750 50  0000 C CNN
+F 3 "" H 12000 2750 50  0000 C CNN
+	1    12000 2750
+	1    0    0    -1
+$EndComp
+Connection ~ 12000 2800
+$Comp
+L +3V3 #PWR?
+U 1 1 589F72F3
+P 10250 2850
+F 0 "#PWR?" H 10250 2700 50  0001 C CNN
+F 1 "+3V3" H 10250 2990 50  0000 C CNN
+F 2 "" H 10250 2850 50  0000 C CNN
+F 3 "" H 10250 2850 50  0000 C CNN
+	1    10250 2850
+	1    0    0    -1
+$EndComp

Commit message: Actualizacion Raiz
por Rubén
Parts:
- removed P3: CONN_02X02, symbol CONN_02X02
Other:
- moved on the sheet: CF36, CF37, CF38, CF39, CF40, CF41, DP1, FT1, JMS1, LF11, RF14, RF15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

Commit message: Actualización Raiz
by Rubén
Parts:
- removed DP1: DIODE, opendous:SM0603_Opendous, symbol DIODE
- added R16: 0, symbol R
Connections:
- net +3V3: no longer CF39.1, FT1.6 (3V3OUT)
- net at JMS1.1 (VBUS): now also R16.2
- net +5V renamed USB_5V
- net USB_5V: now also R16.1
- net nSRST: no longer names the net of FT1.17 (ADBUS6)
- net nTRST: no longer names the net of FT1.20 (ADBUS4)
- new net: CF39.1, FT1.6 (3V3OUT)
Other:
- moved on the sheet: CF39

Commit message: Actualizacion ref. DigitKey
by Rubén
Parts:
- FT1: value FT2232D -> FT2232D-REEL; DIGIKEY REF (none) -> 768-1010-1-ND
- XF2: DIGIKEY REF (none) -> 490-1218-2-ND
Changed lines of the file:
@@
 P 8600 5400
 F 0 "FT1" H 8600 5500 50  0000 C CNN
-F 1 "FT2232D" H 8600 5400 50  0000 C CNN
+F 1 "FT2232D-REEL" H 8600 5400 50  0000 C CNN
 F 2 "Housings_QFP:LQFP-48_7x7mm_Pitch0.5mm" H 8600 5550 50  0001 C CNN
-F 3 "" H 8600 5400 60  0001 C CNN
+F 3 "http://www.ftdichip.com/Support/Documents/DataSheets/ICs/DS_FT2232D.pdf" H 8600 5400 60  0001 C CNN
+F 4 "768-1010-1-ND" H 8600 5400 60  0001 C CNN "DIGIKEY REF"
 	1    8600 5400
 	1    0    0    -1
@@
 F 1 "6MHz" H 6300 5650 60  0000 C CNN
 F 2 "resonator:CSTCR6M00G53Z" H 6300 5800 60  0001 C CNN
-F 3 "" H 6300 5800 60  0001 C CNN
+F 3 "http://www.murata.com/~/media/webrenewal/support/library/catalog/products/timingdevice/ceralock/p16e.ashx" H 6300 5800 60  0001 C CNN
+F 4 "490-1218-2-ND" H 6300 5800 60  0001 C CNN "DIGIKEY REF"
 	1    6300 5800
 	0    1    1    0
