File: hard/hw/Basic_pcb/serial_interface.sch (KiCad schematic (older format))
At the start: 19 parts

Commit message: Actualización huellas y fusible
by Rubén
Parts:
- removed R16: 0, symbol R
- added F1: MF-MSMF050-2, Resistors_SMD:R_1812, symbol Fuse
Connections:
- net USB_5V: now also F1.1
- net at JMS1.1 (VBUS): now also F1.2
Changed lines of the file:
@@
 	1    0    0    -1
 $EndComp
-Text HLabel 4750 4050 0    60   Input ~ 0
+Text HLabel 4750 3850 0    60   Input ~ 0
 USB_5V
-$Comp
-L R R16
-U 1 1 589E93C4
-P 4950 4350
-F 0 "R16" V 5030 4350 50  0000 C CNN
-F 1 "0" V 4950 4350 50  0000 C CNN
-F 2 "" V 4880 4350 50  0001 C CNN
-F 3 "" H 4950 4350 50  0000 C CNN
-	1    4950 4350
-	1    0    0    -1
-$EndComp
 Connection ~ 8300 7350
 Wire Wire Line
@@
 Wire Wire Line
 	4800 4600 4950 4600
-Wire Wire Line
-	4950 4600 4950 4500
 Connection ~ 3650 4950
 Wire Wire Line
@@
 Connection ~ 6950 4900
 Wire Wire Line
-	4950 4200 4950 4050
-Wire Wire Line
 	7600 4300 7450 4300
 Wire Wire Line
@@
 Wire Wire Line
 	7650 2350 7650 2400
-Connection ~ 4950 4050
+Connection ~ 4950 3850
 Wire Wire Line
-	5150 4050 4750 4050
-Text Label 5000 4050 0    60   ~ 0
+	5150 3850 4750 3850
+Text Label 5000 3850 0    60   ~ 0
 +5V_USB
 Text Label 5900 2400 0    60   ~ 0
@@
 Wire Wire Line
 	6450 2450 6450 2400
+$Comp
+L Fuse F1
+U 1 1 58A342AC
+P 4950 4250
+F 0 "F1" V 5030 4250 50  0000 C CNN
+F 1 "MF-MSMF050-2" V 4850 4250 50  0000 C CNN
+F 2 "Resistors_SMD:R_1812" V 4880 4250 50  0001 C CNN
+F 3 "http://www.bourns.com/docs/Product-Datasheets/mfmsmf.pdf" H 4950 4250 50  0001 C CNN
+F 4 "MF-MSMF050-2TR-ND" V 4950 4250 60  0001 C CNN "REF DIGIKEY"
+	1    4950 4250
+	1    0    0    -1
+$EndComp
+Wire Wire Line
+	4950 3850 4950 4100
+Wire Wire Line
+	4950 4600 4950 4400
 $EndSCHEMATC

Commit message: todas las huellas
by Ruben
Parts:
- F1: value MF-MSMF050-2 -> PTS08056V050; REF DIGIKEY MF-MSMF050-2TR-ND -> PTS08056V050-ND
Connections:
- no-connect marks 0 -> 22
Changed lines of the file:
@@
 L +5VA #PWR012
 U 1 1 4FC6C137
-P 7650 2350
-F 0 "#PWR012" H 7650 2480 20  0001 C CNN
-F 1 "+5VA" H 7650 2500 30  0000 C CNN
-F 2 "" H 7650 2350 60  0001 C CNN
-F 3 "" H 7650 2350 60  0001 C CNN
-	1    7650 2350
+P 7250 2300
+F 0 "#PWR012" H 7250 2430 20  0001 C CNN
+F 1 "+5VA" H 7250 2450 30  0000 C CNN
+F 2 "" H 7250 2300 60  0001 C CNN
+F 3 "" H 7250 2300 60  0001 C CNN
+	1    7250 2300
 	1    0    0    -1
 $EndComp
@@
 	7250 2800 7250 2900
 Wire Wire Line
-	7250 2400 7250 2500
+	7250 2300 7250 2500
 Connection ~ 7250 2400
 Wire Wire Line
 	7150 2400 8500 2400
 Connection ~ 7900 2400
-Connection ~ 7650 2400
 Wire Wire Line
 	7450 6400 7450 6450
@@
 Wire Wire Line
 	6700 6300 6950 6300
-Wire Wire Line
-	7650 2350 7650 2400
 Connection ~ 4950 3850
 Wire Wire Line
@@
 P 4950 4250
 F 0 "F1" V 5030 4250 50  0000 C CNN
-F 1 "MF-MSMF050-2" V 4850 4250 50  0000 C CNN
+F 1 "PTS08056V050" V 4850 4250 50  0000 C CNN
 F 2 "Resistors_SMD:R_1812" V 4880 4250 50  0001 C CNN
-F 3 "http://www.bourns.com/docs/Product-Datasheets/mfmsmf.pdf" H 4950 4250 50  0001 C CNN
-F 4 "MF-MSMF050-2TR-ND" V 4950 4250 60  0001 C CNN "REF DIGIKEY"
+F 3 "http://www.belfuse.com/pdfs/0ZCK.pdf" H 4950 4250 50  0001 C CNN
+F 4 "PTS08056V050-ND" V 4950 4250 60  0001 C CNN "REF DIGIKEY"
 	1    4950 4250
 	1    0    0    -1
@@
 Wire Wire Line
 	4950 4600 4950 4400
+NoConn ~ 9600 4400
+NoConn ~ 9600 4500
+NoConn ~ 9600 4600
+NoConn ~ 9600 4700
+NoConn ~ 9600 4900
+NoConn ~ 9600 5000
+NoConn ~ 9600 5100
+NoConn ~ 9600 5200
+NoConn ~ 9600 5700
+NoConn ~ 9600 5800
+NoConn ~ 9600 5900
+NoConn ~ 9600 6000
+NoConn ~ 9600 6100
+NoConn ~ 9600 6200
+NoConn ~ 9600 6400
+NoConn ~ 9600 6500
+NoConn ~ 9600 6600
+NoConn ~ 9600 6700
+NoConn ~ 9600 6900
+NoConn ~ 7600 6200
+NoConn ~ 7600 6100
+NoConn ~ 4800 4900
 $EndSCHEMATC

Commit message: Organizando PIN OUT vr.:0.1
by Ruben
Connections:
- wire segments 76 -> 75
Other:
- moved on the sheet: CF36, RF16
Changed lines of the file:
@@
 $EndDescr
-$Comp
-L GND #PWR06
-U 1 1 4FC6CFCA
-P 8300 7400
-F 0 "#PWR06" H 8300 7400 30  0001 C CNN
-F 1 "GND" H 8300 7330 30  0001 C CNN
-F 2 "" H 8300 7400 60  0001 C CNN
-F 3 "" H 8300 7400 60  0001 C CNN
-	1    8300 7400
-	1    0    0    -1
-$EndComp
-$Comp
-L GND #PWR07
-U 1 1 4FC6CFB6
-P 5650 5900
-F 0 "#PWR07" H 5650 5900 30  0001 C CNN
-F 1 "GND" H 5650 5830 30  0001 C CNN
-F 2 "" H 5650 5900 60  0001 C CNN
-F 3 "" H 5650 5900 60  0001 C CNN
-	1    5650 5900
-	1    0    0    -1
-$EndComp
 $Comp
 L C CF40
@@
 	1    10000 5300
 	0    -1   -1   0
-$EndComp
-$Comp
-L GND #PWR08
-U 1 1 4FC6C3D8
-P 7450 6450
-F 0 "#PWR08" H 7450 6450 30  0001 C CNN
-F 1 "GND" H 7450 6380 30  0001 C CNN
-F 2 "" H 7450 6450 60  0001 C CNN
-F 3 "" H 7450 6450 60  0001 C CNN
-	1    7450 6450
-	1    0    0    -1
 $EndComp
 $Comp
@@
 $EndComp
 $Comp
-L GND #PWR09
-U 1 1 4FC6C3BF
-P 7000 4300
-F 0 "#PWR09" H 7000 4300 30  0001 C CNN
-F 1 "GND" H 7000 4230 30  0001 C CNN
-F 2 "" H 7000 4300 60  0001 C CNN
-F 3 "" H 7000 4300 60  0001 C CNN
-	1    7000 4300
-	0    1    1    0
-$EndComp
-$Comp
-L +5VA #PWR010
-U 1 1 4FC6C374
-P 6950 5400
-F 0 "#PWR010" H 6950 5530 20  0001 C CNN
-F 1 "+5VA" H 6950 5550 30  0000 C CNN
-F 2 "" H 6950 5400 60  0001 C CNN
-F 3 "" H 6950 5400 60  0001 C CNN
-	1    6950 5400
-	1    0    0    -1
-$EndComp
-$Comp
-L GND #PWR011
-U 1 1 4FC6C2CD
-P 7250 2900
-F 0 "#PWR011" H 7250 2900 30  0001 C CNN
-F 1 "GND" H 7250 2830 30  0001 C CNN
-F 2 "" H 7250 2900 60  0001 C CNN
-F 3 "" H 7250 2900 60  0001 C CNN
-	1    7250 2900
-	1    0    0    -1
-$EndComp
-$Comp
 L INDUCTOR LF11
 U 1 1 4FC6C26A
@@
 F 3 "" H 7250 2650 60  0001 C CNN
 	1    7250 2650
-	1    0    0    -1
-$EndComp
-$Comp
-L +5VA #PWR012
-U 1 1 4FC6C137
-P 7250 2300
-F 0 "#PWR012" H 7250 2430 20  0001 C CNN
-F 1 "+5VA" H 7250 2450 30  0000 C CNN
-F 2 "" H 7250 2300 60  0001 C CNN
-F 3 "" H 7250 2300 60  0001 C CNN
-	1    7250 2300
-	1    0    0    -1
-$EndComp
-$Comp
-L GND #PWR013
-U 1 1 4FC6C11B
-P 6450 2850
-F 0 "#PWR013" H 6450 2850 30  0001 C CNN
-F 1 "GND" H 6450 2780 30  0001 C CNN
-F 2 "" H 6450 2850 60  0001 C CNN
-F 3 "" H 6450 2850 60  0001 C CNN
-	1    6450 2850
 	1    0    0    -1
 $EndComp
@@
 $EndComp
 $Comp
-L +5VA #PWR014
-U 1 1 4FC6BDF3
-P 6700 6250
-F 0 "#PWR014" H 6700 6380 20  0001 C CNN
-F 1 "+5VA" H 6700 6400 30  0000 C CNN
-F 2 "" H 6700 6250 60  0001 C CNN
-F 3 "" H 6700 6250 60  0001 C CNN
-	1    6700 6250
-	1    0    0    -1
-$EndComp
-$Comp
 L R RF16
 U 1 1 4FC6BD44
-P 7100 6300
-F 0 "RF16" V 7180 6300 50  0000 C CNN
-F 1 "10K" V 7100 6300 50  0000 C CNN
-F 2 "opendous:SM0603_Opendous" H 7100 6300 60  0001 C CNN
-F 3 "" H 7100 6300 60  0001 C CNN
-	1    7100 6300
+P 7250 6300
+F 0 "RF16" V 7330 6300 50  0000 C CNN
+F 1 "10K" V 7250 6300 50  0000 C CNN
+F 2 "opendous:SM0603_Opendous" H 7250 6300 60  0001 C CNN
+F 3 "" H 7250 6300 60  0001 C CNN
+	1    7250 6300
 	0    -1   -1   0
 $EndComp
@@
 L C CF36
 U 1 1 4FC6BCE9
-P 6450 2600
-F 0 "CF36" H 6500 2700 50  0000 L CNN
-F 1 "10nF" H 6500 2500 50  0000 L CNN
-F 2 "opendous:SM0603_Opendous" H 6450 2600 60  0001 C CNN
-F 3 "" H 6450 2600 60  0001 C CNN
-	1    6450 2600
-	1    0    0    -1
-$EndComp
-$Comp
-L GND #PWR015
-U 1 1 4FC6BCE8
-P 7900 3350
-F 0 "#PWR015" H 7900 3350 30  0001 C CNN
-F 1 "GND" H 7900 3280 30  0001 C CNN
-F 2 "" H 7900 3350 60  0001 C CNN
-F 3 "" H 7900 3350 60  0001 C CNN
-	1    7900 3350
+P 6450 2650
+F 0 "CF36" H 6500 2750 50  0000 L CNN
+F 1 "10nF" H 6500 2550 50  0000 L CNN
+F 2 "opendous:SM0603_Opendous" H 6450 2650 60  0001 C CNN
+F 3 "" H 6450 2650 60  0001 C CNN
+	1    6450 2650
 	1    0    0    -1
 $EndComp
@@
 $EndComp
 $Comp
-L GND #PWR016
-U 1 1 555AD26D
-P 5000 5050
-F 0 "#PWR016" H 5000 5050 30  0001 C CNN
-F 1 "GND" H 5000 4980 30  0001 C CNN
-F 2 "" H 5000 5050 60  0001 C CNN
-F 3 "" H 5000 5050 60  0001 C CNN
-	1    5000 5050
-	-1   0    0    -1
-$EndComp
-$Comp
-L GND #PWR017
-U 1 1 555AD296
-P 3650 5050
-F 0 "#PWR017" H 3650 5050 30  0001 C CNN
-F 1 "GND" H 3650 4980 30  0001 C CNN
-F 2 "" H 3650 5050 60  0001 C CNN
-F 3 "" H 3650 5050 60  0001 C CNN
-	1    3650 5050
-	-1   0    0    -1
-$EndComp
-$Comp
-L +3V3 #PWR018
+L +3V3 #PWR06
 U 1 1 589F5460
 P 10300 6750
-F 0 "#PWR018" H 10300 6600 50  0001 C CNN
+F 0 "#PWR06" H 10300 6600 50  0001 C CNN
 F 1 "+3V3" H 10300 6890 50  0000 C CNN
 F 2 "" H 10300 6750 50  0000 C CNN
@@
 $EndComp
 $Comp
-L +3V3 #PWR019
+L +3V3 #PWR07
 U 1 1 589F5F40
 P 10300 5050
-F 0 "#PWR019" H 10300 4900 50  0001 C CNN
+F 0 "#PWR07" H 10300 4900 50  0001 C CNN
 F 1 "+3V3" H 10300 5190 50  0000 C CNN
 F 2 "" H 10300 5050 50  0000 C CNN
@@
 $EndComp
 $Comp
-L +3V3 #PWR020
+L +3V3 #PWR08
 U 1 1 589F6257
 P 10500 4800
-F 0 "#PWR020" H 10500 4650 50  0001 C CNN
+F 0 "#PWR08" H 10500 4650 50  0001 C CNN
 F 1 "+3V3" H 10500 4940 50  0000 C CNN
 F 2 "" H 10500 4800 50  0000 C CNN
@@
 $EndComp
 $Comp
-L +3V3 #PWR021
+L +3V3 #PWR09
 U 1 1 589F6BB3
 P 8800 3450
-F 0 "#PWR021" H 8800 3300 50  0001 C CNN
+F 0 "#PWR09" H 8800 3300 50  0001 C CNN
 F 1 "+3V3" H 8800 3590 50  0000 C CNN
 F 2 "" H 8800 3450 50  0000 C CNN
@@
 Wire Wire Line
 	7600 6400 7450 6400
-Wire Wire Line
-	6950 5400 7600 5400
 Connection ~ 8500 3450
 Wire Wire Line
@@
 Wire Wire Line
 	7900 2900 8300 2900
-Wire Wire Line
-	7250 6300 7600 6300
 Wire Wire Line
 	6950 5200 6950 4900
@@
 	8800 3450 8800 3700
 Wire Wire Line
-	6450 2750 6450 2850
-Wire Wire Line
 	7250 2800 7250 2900
-Wire Wire Line
-	7250 2300 7250 2500
 Connection ~ 7250 2400
-Wire Wire Line
-	7150 2400 8500 2400
 Connection ~ 7900 2400
 Wire Wire Line
@@
 	5800 5500 5750 5500
 Wire Wire Line
-	7900 2500 7900 2400
+	7900 2400 7900 2500
 Wire Wire Line
 	7900 2800 7900 2950
@@
 Wire Wire Line
 	7150 4300 7000 4300
-Wire Wire Line
-	6700 6250 6700 6300
-Wire Wire Line
-	6700 6300 6950 6300
 Connection ~ 4950 3850
 Wire Wire Line
-	5150 3850 4750 3850
+	4750 3850 5150 3850
 Text Label 5000 3850 0    60   ~ 0
 +5V_USB
@@
 Wire Wire Line
 	5850 2400 6550 2400
-Wire Wire Line
-	6450 2450 6450 2400
 $Comp
 L Fuse F1
@@
 NoConn ~ 7600 6100
 NoConn ~ 4800 4900
+Wire Wire Line
+	6450 2500 6450 2400
+$Comp
+L GND #PWR010
+U 1 1 58A66750
+P 6450 2900
+F 0 "#PWR010" H 6450 2650 50  0001 C CNN
+F 1 "GND" H 6450 2750 50  0000 C CNN
+F 2 "" H 6450 2900 50  0000 C CNN
+F 3 "" H 6450 2900 50  0000 C CNN
+	1    6450 2900
+	1    0    0    -1
+$EndComp
+Wire Wire Line
+	6450 2800 6450 2900
+Connection ~ 7250 2850
+Connection ~ 6450 2850
+Connection ~ 8500 2400
+Text Label 8600 2400 0    60   ~ 0
++5VA
+Wire Wire Line
+	7150 2400 8900 2400
+Wire Wire Line
+	7250 2500 7250 2400
+Text Label 7300 5400 0    60   ~ 0
++5VA
+Wire Wire Line
+	7600 6300 7400 6300
+Text Label 6800 6300 0    60   ~ 0
++5VA
+Wire Wire Line
+	7600 5400 7200 5400
+Wire Wire Line
+	7100 6300 6750 6300
+$Comp
+L GND #PWR011
+U 1 1 58A8D1C3
+P 7250 2900
+F 0 "#PWR011" H 7250 2650 50  0001 C CNN
+F 1 "GND" H 7250 2750 50  0000 C CNN
+F 2 "" H 7250 2900 50  0000 C CNN
+F 3 "" H 7250 2900 50  0000 C CNN
+	1    7250 2900
+	1    0    0    -1
+$EndComp
+$Comp
+L GND #PWR012
+U 1 1 58A8D267
+P 7900 3350
+F 0 "#PWR012" H 7900 3100 50  0001 C CNN
+F 1 "GND" H 7900 3200 50  0000 C CNN
+F 2 "" H 7900 3350 50  0000 C CNN
+F 3 "" H 7900 3350 50  0000 C CNN
+	1    7900 3350
+	1    0    0    -1
+$EndComp
+$Comp
+L GND #PWR013
+U 1 1 58A8D7DD
+P 8300 7400
+F 0 "#PWR013" H 8300 7150 50  0001 C CNN
+F 1 "GND" H 8300 7250 50  0000 C CNN
+F 2 "" H 8300 7400 50  0000 C CNN
+F 3 "" H 8300 7400 50  0000 C CNN
+	1    8300 7400
+	1    0    0    -1
+$EndComp
+$Comp
+L GND #PWR014
+U 1 1 58A8DF8B
+P 7450 6450
+F 0 "#PWR014" H 7450 6200 50  0001 C CNN
+F 1 "GND" H 7450 6300 50  0000 C CNN
+F 2 "" H 7450 6450 50  0000 C CNN
+F 3 "" H 7450 6450 50  0000 C CNN
+	1    7450 6450
+	1    0    0    -1
+$EndComp
+$Comp
+L GND #PWR015
+U 1 1 58A8E746
+P 5650 5900
+F 0 "#PWR015" H 5650 5650 50  0001 C CNN
+F 1 "GND" H 5650 5750 50  0000 C CNN
+F 2 "" H 5650 5900 50  0000 C CNN
+F 3 "" H 5650 5900 50  0000 C CNN
+	1    5650 5900
+	1    0    0    -1
+$EndComp
+$Comp
+L GND #PWR016
+U 1 1 58A8EFD2
+P 5000 5050
+F 0 "#PWR016" H 5000 4800 50  0001 C CNN
+F 1 "GND" H 5000 4900 50  0000 C CNN
+F 2 "" H 5000 5050 50  0000 C CNN
+F 3 "" H 5000 5050 50  0000 C CNN
+	1    5000 5050
+	1    0    0    -1
+$EndComp
+$Comp
+L GND #PWR017
+U 1 1 58A8F696
+P 3650 5050
+F 0 "#PWR017" H 3650 4800 50  0001 C CNN
+F 1 "GND" H 3650 4900 50  0000 C CNN
+F 2 "" H 3650 5050 50  0000 C CNN
+F 3 "" H 3650 5050 50  0000 C CNN
+	1    3650 5050
+	1    0    0    -1
+$EndComp
+$Comp
+L GND #PWR018
+U 1 1 58A8F991
+P 7000 4300
+F 0 "#PWR018" H 7000 4050 50  0001 C CNN
+F 1 "GND" H 7000 4150 50  0000 C CNN
+F 2 "" H 7000 4300 50  0000 C CNN
+F 3 "" H 7000 4300 50  0000 C CNN
+	1    7000 4300
+	0    1    1    0
+$EndComp
 $EndSCHEMATC
