File: hard/hw/Basic_pcb/Power.sch (KiCad schematic (older format))
At the start: 0 parts

Commit message: Actualizacion Power
Parts:
- added CF30, CF32, CF33, CF35: 33uF, opendous:SM1206_Opendous, symbol C
- added CF31, CF34: 100n, opendous:SM0603, symbol C
- added PS?: BARREL_JACK, Connect:JACK_ALIM, symbol BARREL_JACK
- added UF2: ZLDO1117G33TA, SMD_Packages:SOT-223, symbol LT1117CST
- added UF3: ZLDO1117G12TA, SMD_Packages:SOT-223, symbol LT1117CST
Connections:
- net labels added: +1V2, +3.3VDAC, GND, VDD5V
- wire segments 0 -> 26

Commit message: Power: fuente de 5v - 2A
by Luis Yaya
Parts:
- added C? (x4): 10u, ~, symbol C
- added C? (x3): 22u, ~, symbol C
- added C?: 100n, ~, symbol C
- added L?: INDUCTOR, ~, symbol INDUCTOR
- added R?: 10k, ~, symbol R
- added R?: 100k, ~, symbol R
- added R?: 680k, ~, symbol R
- added R?: 130k, ~, symbol R
- added U?: TPS63071, symbol TPS63071
Connections:
- net labels added: +12V, +5V
- wire segments 26 -> 77
Other:
- moved on the sheet: CF30, CF31, CF32, CF33, CF34, CF35, PS?, UF2, UF3

Commit message: Fuente 12V
by Luis Yaya
Parts:
- C10, C6, C7, C8: renamed from C?; footprint ~ -> Capacitors_SMD:C_0603
- C11, C12, C13: renamed from C?; footprint ~ -> Capacitors_SMD:C_0805
- C9: renamed from C?; footprint ~ -> Capacitors_SMD:C_0402
- L3: renamed from L?; value INDUCTOR -> XFL4020-152ME; footprint ~ -> (none)
- R12, R13, R14, R15: renamed from R?; footprint ~ -> (none)
- gave numbers to parts that had none: 2
Other:
- moved on the sheet: C10, C11, C12, C13, C6, C7, C8, C9, CF30, CF31, CF32, CF33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

Commit message: Actualización PinOut LVDS
by Rubén Parra
Connections:
- net labels added: +3V3
- net labels removed: +3.3VDAC
- wire segments 77 -> 76
Other:
- moved on the sheet: C10, C11, C12, C13, C6, C7, C8, R12, R13, R14, R15

Commit message: Actualizacion Raiz
por Rubén
Parts:
- added P3, P4: CONN_02X02, symbol CONN_02X02
Connections:
- net VDD5V is gone; now on net +9V: PS1.1
- net +3V3: now also P3.1 (P1), P4.1 (P1)
- net +5V: now also P3.2 (P2), P4.2 (P2)
- net GND: now also P3.3 (P3), P3.4 (P4), P4.3 (P3), P4.4 (P4)
- net +12V renamed +9V
- no-connect marks 0 -> 1
Changed lines of the file:
@@
 $EndComp
 $Comp
-L GND #PWR067
+L GND #PWR068
 U 1 1 589983B5
 P 2450 1950
-F 0 "#PWR067" H 2450 1950 30  0001 C CNN
+F 0 "#PWR068" H 2450 1950 30  0001 C CNN
 F 1 "GND" H 2450 1880 30  0001 C CNN
 F 2 "" H 2450 1950 60  0001 C CNN
@@
 $EndComp
 $Comp
-L GND #PWR068
+L GND #PWR069
 U 1 1 589983BB
 P 3300 2350
-F 0 "#PWR068" H 3300 2350 30  0001 C CNN
+F 0 "#PWR069" H 3300 2350 30  0001 C CNN
 F 1 "GND" H 3300 2280 30  0001 C CNN
 F 2 "" H 3300 2350 60  0001 C CNN
@@
 $EndComp
 $Comp
-L GND #PWR069
+L GND #PWR070
 U 1 1 589983CF
 P 3700 2350
-F 0 "#PWR069" H 3700 2350 30  0001 C CNN
+F 0 "#PWR070" H 3700 2350 30  0001 C CNN
 F 1 "GND" H 3700 2280 30  0001 C CNN
 F 2 "" H 3700 2350 60  0001 C CNN
@@
 $EndComp
 $Comp
-L GND #PWR070
+L GND #PWR071
 U 1 1 589983D5
 P 2250 2350
-F 0 "#PWR070" H 2250 2350 30  0001 C CNN
+F 0 "#PWR071" H 2250 2350 30  0001 C CNN
 F 1 "GND" H 2250 2280 30  0001 C CNN
 F 2 "" H 2250 2350 60  0001 C CNN
@@
 $EndComp
 $Comp
-L GND #PWR071
+L GND #PWR072
 U 1 1 589983EF
 P 4850 1950
-F 0 "#PWR071" H 4850 1950 30  0001 C CNN
+F 0 "#PWR072" H 4850 1950 30  0001 C CNN
 F 1 "GND" H 4850 1880 30  0001 C CNN
 F 2 "" H 4850 1950 60  0001 C CNN
@@
 $EndComp
 $Comp
-L GND #PWR072
+L GND #PWR073
 U 1 1 589983F5
 P 5700 2350
-F 0 "#PWR072" H 5700 2350 30  0001 C CNN
+F 0 "#PWR073" H 5700 2350 30  0001 C CNN
 F 1 "GND" H 5700 2280 30  0001 C CNN
 F 2 "" H 5700 2350 60  0001 C CNN
@@
 $EndComp
 $Comp
-L GND #PWR073
+L GND #PWR074
 U 1 1 58998409
 P 6100 2350
-F 0 "#PWR073" H 6100 2350 30  0001 C CNN
+F 0 "#PWR074" H 6100 2350 30  0001 C CNN
 F 1 "GND" H 6100 2280 30  0001 C CNN
 F 2 "" H 6100 2350 60  0001 C CNN
@@
 $EndComp
 $Comp
-L GND #PWR074
+L GND #PWR075
 U 1 1 5899840F
 P 4650 2350
-F 0 "#PWR074" H 4650 2350 30  0001 C CNN
+F 0 "#PWR075" H 4650 2350 30  0001 C CNN
 F 1 "GND" H 4650 2280 30  0001 C CNN
 F 2 "" H 4650 2350 60  0001 C CNN
 F 3 "" H 4650 2350 60  0001 C CNN
 	1    4650 2350
-	1    0    0    -1
-$EndComp
-$Comp
-L VDD5V #PWR075
-U 1 1 58A05816
-P 8300 1650
-F 0 "#PWR075" H 8300 1750 30  0001 C CNN
-F 1 "VDD5V" H 8300 1750 30  0000 C CNN
-F 2 "" H 8300 1650 60  0001 C CNN
-F 3 "" H 8300 1650 60  0001 C CNN
-	1    8300 1650
 	1    0    0    -1
 $EndComp
@@
 $EndComp
 $Comp
-L GND #PWR078
+L GND #PWR077
 U 1 1 5898FCE6
 P 2700 4950
-F 0 "#PWR078" H 2700 4950 30  0001 C CNN
+F 0 "#PWR077" H 2700 4950 30  0001 C CNN
 F 1 "GND" H 2700 4880 30  0001 C CNN
 F 2 "" H 2700 4950 60  0000 C CNN
@@
 $EndComp
 $Comp
-L GND #PWR080
+L GND #PWR078
 U 1 1 5898FCE9
 P 4800 5700
-F 0 "#PWR080" H 4800 5700 30  0001 C CNN
+F 0 "#PWR078" H 4800 5700 30  0001 C CNN
 F 1 "GND" H 4800 5630 30  0001 C CNN
 F 2 "" H 4800 5700 60  0000 C CNN
@@
 $EndComp
 $Comp
-L +12V #PWR085
-U 1 1 5898FCEF
-P 2300 4250
-F 0 "#PWR085" H 2300 4200 20  0001 C CNN
-F 1 "+12V" H 2300 4400 30  0000 C CNN
-F 2 "" H 2300 4250 60  0000 C CNN
-F 3 "" H 2300 4250 60  0000 C CNN
-	1    2300 4250
-	1    0    0    -1
-$EndComp
-$Comp
-L +5V #PWR086
+L +5V #PWR079
 U 1 1 5898FCF0
 P 7900 4200
-F 0 "#PWR086" H 7900 4290 20  0001 C CNN
+F 0 "#PWR079" H 7900 4290 20  0001 C CNN
 F 1 "+5V" H 7900 4350 30  0000 C CNN
 F 2 "" H 7900 4200 60  0000 C CNN
@@
 $EndComp
 $Comp
-L GND #PWR089
+L GND #PWR080
 U 1 1 5899D723
 P 3900 4700
-F 0 "#PWR089" H 3900 4450 50  0001 C CNN
+F 0 "#PWR080" H 3900 4450 50  0001 C CNN
 F 1 "GND" H 3900 4550 50  0000 C CNN
 F 2 "" H 3900 4700 50  0000 C CNN
@@
 $EndComp
 $Comp
-L GND #PWR?
+L GND #PWR081
 U 1 1 589BCFDB
 P 7600 5050
-F 0 "#PWR?" H 7600 5050 30  0001 C CNN
+F 0 "#PWR081" H 7600 5050 30  0001 C CNN
 F 1 "GND" H 7600 4980 30  0001 C CNN
 F 2 "" H 7600 5050 60  0000 C CNN
@@
 	3100 4900 3100 4850
 $Comp
-L +5V #PWR?
+L +5V #PWR082
 U 1 1 589C1DD8
 P 2250 1700
-F 0 "#PWR?" H 2250 1550 50  0001 C CNN
+F 0 "#PWR082" H 2250 1550 50  0001 C CNN
 F 1 "+5V" H 2250 1840 50  0000 C CNN
 F 2 "" H 2250 1700 50  0000 C CNN
@@
 	4650 1700 4650 1900
 $Comp
-L +1V2 #PWR065
+L +1V2 #PWR083
 U 1 1 5899839B
 P 6100 1700
-F 0 "#PWR065" H 6100 1550 60  0001 C CNN
+F 0 "#PWR083" H 6100 1550 60  0001 C CNN
 F 1 "+1V2" H 6100 1840 60  0000 C CNN
 F 2 "" H 6100 1700 60  0000 C CNN
@@
 $EndComp
 $Comp
-L +3V3 #PWR?
+L +3V3 #PWR084
 U 1 1 589C32B2
 P 3700 1700
-F 0 "#PWR?" H 3700 1550 50  0001 C CNN
+F 0 "#PWR084" H 3700 1550 50  0001 C CNN
 F 1 "+3V3" H 3700 1840 50  0000 C CNN
 F 2 "" H 3700 1700 50  0000 C CNN
@@
 $EndComp
 $Comp
-L +3V3 #PWR?
+L +3V3 #PWR085
 U 1 1 589C347B
 P 4650 1700
-F 0 "#PWR?" H 4650 1550 50  0001 C CNN
+F 0 "#PWR085" H 4650 1550 50  0001 C CNN
 F 1 "+3V3" H 4650 1840 50  0000 C CNN
 F 2 "" H 4650 1700 50  0000 C CNN
@@
 Wire Wire Line
 	6100 1900 6100 1700
+$Comp
+L +9V #PWR086
+U 1 1 58A01D1E
+P 8300 1650
+F 0 "#PWR086" H 8300 1500 50  0001 C CNN
+F 1 "+9V" H 8300 1790 50  0000 C CNN
+F 2 "" H 8300 1650 50  0000 C CNN
+F 3 "" H 8300 1650 50  0000 C CNN
+	1    8300 1650
+	1    0    0    -1
+$EndComp
+$Comp
+L +9V #PWR087
+U 1 1 58A02321
+P 2300 4250
+F 0 "#PWR087" H 2300 4100 50  0001 C CNN
+F 1 "+9V" H 2300 4390 50  0000 C CNN
+F 2 "" H 2300 4250 50  0000 C CNN
+F 3 "" H 2300 4250 50  0000 C CNN
+	1    2300 4250
+	1    0    0    -1
+$EndComp
+$Comp
+L CONN_02X02 P3
+U 1 1 58A16893
+P 9550 1800
+F 0 "P3" H 9550 1950 50  0000 C CNN
+F 1 "CONN_02X02" H 9550 1650 50  0000 C CNN
+F 2 "" H 9550 600 50  0001 C CNN
+F 3 "" H 9550 600 50  0000 C CNN
+	1    9550 1800
+	1    0    0    -1
+$EndComp
+$Comp
+L GND #PWR088
+U 1 1 58A16B54
+P 9900 1950
+F 0 "#PWR088" H 9900 1700 50  0001 C CNN
+F 1 "GND" H 9900 1800 50  0000 C CNN
+F 2 "" H 9900 1950 50  0000 C CNN
+F 3 "" H 9900 1950 50  0000 C CNN
+	1    9900 1950
+	1    0    0    -1
+$EndComp
+Wire Wire Line
+	9900 1950 9900 1850
+Wire Wire Line
+	9900 1850 9800 1850
+$Comp
+L GND #PWR089
+U 1 1 58A16FAA
+P 9200 1950
+F 0 "#PWR089" H 9200 1700 50  0001 C CNN
+F 1 "GND" H 9200 1800 50  0000 C CNN
+F 2 "" H 9200 1950 50  0000 C CNN
+F 3 "" H 9200 1950 50  0000 C CNN
+	1    9200 1950
+	1    0    0    -1
+$EndComp
+Wire Wire Line
+	9300 1850 9200 1850
+$Comp
+L +5V #PWR090
+U 1 1 58A17073
+P 9900 1650
+F 0 "#PWR090" H 9900 1500 50  0001 C CNN
+F 1 "+5V" H 9900 1790 50  0000 C CNN
+F 2 "" H 9900 1650 50  0000 C CNN
+F 3 "" H 9900 1650 50  0000 C CNN
+	1    9900 1650
+	1    0    0    -1
+$EndComp
+$Comp
+L +3V3 #PWR091
+U 1 1 58A17387
+P 9200 1650
+F 0 "#PWR091" H 9200 1500 50  0001 C CNN
+F 1 "+3V3" H 9200 1790 50  0000 C CNN
+F 2 "" H 9200 1650 50  0000 C CNN
+F 3 "" H 9200 1650 50  0000 C CNN
+	1    9200 1650
+	1    0    0    -1
+$EndComp
+Wire Wire Line
+	9900 1650 9900 1750
+Wire Wire Line
+	9900 1750 9800 1750
+Wire Wire Line
+	9200 1650 9200 1750
+Wire Wire Line
+	9200 1750 9300 1750
+Wire Wire Line
+	9200 1850 9200 1950
+$Comp
+L CONN_02X02 P4
+U 1 1 58A196D4
+P 9550 2650
+F 0 "P4" H 9550 2800 50  0000 C CNN
+F 1 "CONN_02X02" H 9550 2500 50  0000 C CNN
+F 2 "" H 9550 1450 50  0001 C CNN
+F 3 "" H 9550 1450 50  0000 C CNN
+	1    9550 2650
+	1    0    0    -1
+$EndComp
+$Comp
+L GND #PWR092
+U 1 1 58A196DA
+P 9900 2800
+F 0 "#PWR092" H 9900 2550 50  0001 C CNN
+F 1 "GND" H 9900 2650 50  0000 C CNN
+F 2 "" H 9900 2800 50  0000 C CNN
+F 3 "" H 9900 2800 50  0000 C CNN
+	1    9900 2800
+	1    0    0    -1
+$EndComp
+Wire Wire Line
+	9900 2800 9900 2700
+Wire Wire Line
+	9900 2700 9800 2700
+$Comp
+L GND #PWR093
+U 1 1 58A196E2
+P 9200 2800
+F 0 "#PWR093" H 9200 2550 50  0001 C CNN
+F 1 "GND" H 9200 2650 50  0000 C CNN
+F 2 "" H 9200 2800 50  0000 C CNN
+F 3 "" H 9200 2800 50  0000 C CNN
+	1    9200 2800
+	1    0    0    -1
+$EndComp
+Wire Wire Line
+	9300 2700 9200 2700
+$Comp
+L +5V #PWR094
+U 1 1 58A196E9
+P 9900 2500
+F 0 "#PWR094" H 9900 2350 50  0001 C CNN
+F 1 "+5V" H 9900 2640 50  0000 C CNN
+F 2 "" H 9900 2500 50  0000 C CNN
+F 3 "" H 9900 2500 50  0000 C CNN
+	1    9900 2500
+	1    0    0    -1
+$EndComp
+$Comp
+L +3V3 #PWR095
+U 1 1 58A196EF
+P 9200 2500
+F 0 "#PWR095" H 9200 2350 50  0001 C CNN
+F 1 "+3V3" H 9200 2640 50  0000 C CNN
+F 2 "" H 9200 2500 50  0000 C CNN
+F 3 "" H 9200 2500 50  0000 C CNN
+	1    9200 2500
+	1    0    0    -1
+$EndComp
+Wire Wire Line
+	9900 2500 9900 2600
+Wire Wire Line
+	9900 2600 9800 2600
+Wire Wire Line
+	9200 2500 9200 2600
+Wire Wire Line
+	9200 2600 9300 2600
+Wire Wire Line
+	9200 2700 9200 2800
+NoConn ~ 8100 1850
 $EndSCHEMATC

Commit message: Actualización Raiz
by Rubén
Parts:
- added CF1, CF10, CF12, CF14, CF15, CF16, CF17, CF18, CF19, CF2, CF20, CF21, CF22, CF23, CF24, CF25, CF3, CF4, CF5, CF6, CF7, CF8, CF9: 0.1uF, opendous:SM0603, symbol C
- added CF11, CF26, CF27: 1uF, opendous:SM0603, symbol C
- added CF13, CF28, CF29: 4.7uF, opendous:SM1206_Opendous, symbol C
- added J2: CONN_3X1F, Socket_Strips:Socket_Strip_Straight_1x03_Pitch2.54mm, symbol CONN_3X1F
- P3, P4: footprint (none) -> Socket_Strips:Socket_Strip_Straight_2x02_Pitch2.54mm
Connections:
- net +1V2: now also CF16.1, CF18.1, CF19.1, CF22.1, CF24.1, CF26.1, CF28.1
- net +3V3: now also CF1.1, CF10.1, CF11.1, CF12.1, CF13.1, CF14.1, CF15.1, CF17.1, CF2.1, CF20.1, CF21.1, CF23.1, CF25.1, CF27.1, CF29.1, CF3.1, CF4.1, CF5.1, CF6.1, CF7.1, CF8.1, CF9.1
- net +5V: now also J2.2; no longer C10.1, C11.1, C12.1, C13.1, R13.1, R15.1, U2.7 (Vout), U2.8 (Vout)
- net GND: now also CF1.2, CF10.2, CF11.2, CF12.2, CF13.2, CF14.2, CF15.2, CF16.2, CF17.2, CF18.2, CF19.2, CF2.2, CF20.2, CF21.2, CF22.2, CF23.2, CF24.2, CF25.2, CF26.2, CF27.2, CF28.2, CF29.2, CF3.2, CF4.2, CF5.2, CF6.2, CF7.2, CF8.2, CF9.2
- new net USBVCC: J2.3
- new net VDD5V: C10.1, C11.1, C12.1, C13.1, J2.1, R13.1, R15.1, U2.7 (Vout), U2.8 (Vout)
Other:
- note added: "Conector para seleccionar fuente \npor medio de un jumper.\n\n> VDD5V: Fuente jack DC de 9VDC \n a 5VDC.\n> +5V: Referencia de 5VDC de toda \n la tarjeta.\n> USBVCC: 5VDC obtenido por \n conector USB"
- moved on the sheet: C10, C11, C12, C13, C6, C7, C8, C9, CF30, CF31, CF32, CF33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

Commit message: Actualizacion ref. DigitKey
by Rubén
Parts:
- U2: value TPS63071 -> TPS63070; DIGIKEY REF (none) -> TPS63070RNMR
- UF2: DIGIKEY REF (none) -> ZLDO1117G33DITR-ND
- UF3: DIGIKEY REF (none) -> ZLDO1117G12DITR-ND
Changed lines of the file:
@@
 F 1 "ZLDO1117G33TA" H 4400 1450 40  0000 C CNN
 F 2 "SMD_Packages:SOT-223" H 4400 1450 60  0001 C CNN
-F 3 "" H 4400 1450 60  0001 C CNN
+F 3 "https://www.diodes.com/assets/Datasheets/ZLDO1117.pdf" H 4400 1450 60  0001 C CNN
+F 4 "ZLDO1117G33DITR-ND" H 4400 1450 60  0001 C CNN "DIGIKEY REF"
 	1    4400 1450
 	1    0    0    -1
@@
 F 1 "ZLDO1117G12TA" H 6800 1450 40  0000 C CNN
 F 2 "SMD_Packages:SOT-223" H 6800 1450 60  0001 C CNN
-F 3 "" H 6800 1450 60  0001 C CNN
+F 3 "https://www.diodes.com/assets/Datasheets/ZLDO1117.pdf" H 6800 1450 60  0001 C CNN
+F 4 "ZLDO1117G12DITR-ND" H 6800 1450 60  0001 C CNN "DIGIKEY REF"
 	1    6800 1450
 	1    0    0    -1
@@
 P 4450 3850
 F 0 "U2" H 4450 4600 60  0000 C CNN
-F 1 "TPS63071" H 4450 3850 60  0000 C CNN
+F 1 "TPS63070" H 4450 3850 60  0000 C CNN
 F 2 "" H 4450 3850 60  0001 C CNN
-F 3 "" H 4450 3850 60  0000 C CNN
+F 3 "http://www.ti.com/lit/ds/symlink/tps63070.pdf" H 4450 3850 60  0001 C CNN
+F 4 "TPS63070RNMR" H 4450 3850 60  0001 C CNN "DIGIKEY REF"
 	1    4450 3850
 	1    0    0    -1

Commit message: Actualización huellas y fusible
by Rubén
Parts:
- L3: footprint (none) -> resonator:XFL4020
- R12, R13, R14, R15: footprint (none) -> Resistors_SMD:R_0603
- U2: footprint (none) -> resonator:TPS63071
Changed lines of the file:
@@
 F 0 "L3" V 4400 2900 40  0000 C CNN
 F 1 "XFL4020-152ME" V 4550 2900 40  0000 C CNN
-F 2 "" H 4450 2900 60  0001 C CNN
+F 2 "resonator:XFL4020" H 4450 2900 60  0001 C CNN
 F 3 "~" H 4450 2900 60  0000 C CNN
 	1    4450 2900
@@
 F 0 "R12" V 3180 3750 40  0000 C CNN
 F 1 "10k" V 3107 3751 40  0000 C CNN
-F 2 "" V 3030 3750 30  0001 C CNN
+F 2 "Resistors_SMD:R_0603" V 3030 3750 30  0001 C CNN
 F 3 "~" H 3100 3750 30  0000 C CNN
 	1    3100 3750
@@
 F 0 "R15" V 7630 3700 40  0000 C CNN
 F 1 "100k" V 7557 3701 40  0000 C CNN
-F 2 "" V 7480 3700 30  0001 C CNN
+F 2 "Resistors_SMD:R_0603" V 7480 3700 30  0001 C CNN
 F 3 "~" H 7550 3700 30  0000 C CNN
 	1    7550 3700
@@
 F 0 "U2" H 4450 4600 60  0000 C CNN
 F 1 "TPS63070" H 4450 3850 60  0000 C CNN
-F 2 "" H 4450 3850 60  0001 C CNN
+F 2 "resonator:TPS63071" H 4450 3850 60  0001 C CNN
 F 3 "http://www.ti.com/lit/ds/symlink/tps63070.pdf" H 4450 3850 60  0001 C CNN
 F 4 "TPS63070RNMR" H 4450 3850 60  0001 C CNN "DIGIKEY REF"
@@
 F 0 "R13" V 5880 3700 40  0000 C CNN
 F 1 "680k" V 5807 3701 40  0000 C CNN
-F 2 "" V 5730 3700 30  0001 C CNN
+F 2 "Resistors_SMD:R_0603" V 5730 3700 30  0001 C CNN
 F 3 "~" H 5800 3700 30  0000 C CNN
 	1    5800 3700
@@
 F 0 "R14" V 6080 4050 40  0000 C CNN
 F 1 "130k" V 6007 4051 40  0000 C CNN
-F 2 "" V 5930 4050 30  0001 C CNN
+F 2 "Resistors_SMD:R_0603" V 5930 4050 30  0001 C CNN
 F 3 "~" H 6000 4050 30  0000 C CNN
 	1    6000 4050
