File: hard/hw/Basic_pcb/HDMIspartan6_Board.kicad_pcb (KiCad board)
At the start: 4 copper layers, 53.3 x 85.1 mm, 124 parts, among them IC1 MT48LC4M16A2P, J1 HDMI_A, P1 CONN_02X15, X1 OSCILLATORS-1

Commit message: 3d
Parts:
- moved PS1 4.10 mm to (129.5, 129.9)

Commit message: ok 3d
Parts:
- moved JMS1 0.95 mm to (126.2, 53.6)
Changed lines of the file:
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@@
     (links 375)
     (no_connects 371)
-    (area 19.3 14.004 185.494 148.439)
+    (area 79.924999 49.854999 133.415001 135.095001)
     (thickness 1.6)
     (drawings 16)
@@
       (rotate (xyz 0 0 0))
     )
+    (model TO_SOT_Packages_SMD.3dshapes/SOT-223.wrl
+      (at (xyz 0 0 0))
+      (scale (xyz 0.4 0.4 0.4))
+      (rotate (xyz 0 0 0))
+    )
   )
   (module SMD_Packages:SOT-223 (layer F.Cu)
@@
       (rotate (xyz 0 0 0))
     )
+    (model TO_SOT_Packages_SMD.3dshapes/SOT-223.wrl
+      (at (xyz 0 0 0))
+      (scale (xyz 0.4 0.4 0.4))
+      (rotate (xyz 0 0 0))
+    )
   )
   (module SM0603 (layer F.Cu)
@@
   )
   (module Connect:USB_Mini-B (layer F.Cu)
-    (at 125.974 54.502 270)
+    (at 126.23 53.59 270)
     (descr "USB Mini-B 5-pin SMD connector")
     (tags "USB USB_B USB_Mini connector")
@@
     (pad "" np_thru_hole circle (at 0.8509 -2.19964 270) (size 0.89916 0.89916) (drill 0.89916) (layers *.Cu *.Mask F.SilkS))
     (pad "" np_thru_hole circle (at 0.8509 2.19964 270) (size 0.89916 0.89916) (drill 0.89916) (layers *.Cu *.Mask F.SilkS))
+    (model C:/Users/Administrador/Documents/kit3/hdmi-fpga/hard/hw/Basic_pcb/packsges3d/usb.wrl
+      (at (xyz 0.15 0 0))
+      (scale (xyz 0.4 0.4 0.4))
+      (rotate (xyz -90 0 90))
+    )
   )
   (module opendous:SM0603_Opendous (layer F.Cu)
@@
     (pad 2 smd rect (at 2.90068 2.10058 180) (size 1.80086 1.99898) (layers F.Cu F.Paste F.Mask)
       (net 1 GND))
+    (model Crystals.3dshapes/Crystal_SMD_5032_4Pads.wrl
+      (at (xyz 0 0 0))
+      (scale (xyz 1.2 1.2 1.2))
+      (rotate (xyz 0 0 0))
+    )
   )
   (module Pin_Headers:Pin_Header_Straight_2x15_Pitch2.00mm (layer F.Cu)

Commit message: todas las huellas
by Ruben
Parts:
- removed P1 (x2): CONN_02X15, hackrf:GSG-HEADER-2x2
- added C1: 10uF, Capacitors_SMD:C_0805, F.Cu at (146.2, 139.5)
- added C10: 10u, Capacitors_SMD:C_0603, F.Cu at (151.6, 164.2)
- added C11: 22u, Capacitors_SMD:C_0805, F.Cu at (158.2, 139.6)
- added C12: 22u, Capacitors_SMD:C_0805, F.Cu at (146.0, 156.1)
- added C13: 22u, Capacitors_SMD:C_0805, F.Cu at (159.2, 157.6)
- added C2: 1uF, Capacitors_SMD:C_0805, F.Cu at (146.5, 144.9)
- added C3: 1uF, Capacitors_SMD:C_0805, F.Cu at (151.9, 145.0)
- added C4: 220pF, Capacitors_SMD:C_0805, F.Cu at (152.2, 139.5)
- added C5: 220pF, Capacitors_SMD:C_0805, F.Cu at (146.5, 150.5)
- added C6: 10u, Capacitors_SMD:C_0603, F.Cu at (152.1, 150.8)
- added C7: 10u, Capacitors_SMD:C_0603, F.Cu at (159.0, 152.0)
- added C8: 10u, Capacitors_SMD:C_0603, F.Cu at (152.1, 157.4)
- added C9: 100n, Capacitors_SMD:C_0402, F.Cu at (146.0, 163.2)
- added F1: MF-MSMF050-2, Resistors_SMD:R_1812, F.Cu at (159.8, 145.9)
- added J2: CONN_3X1F, Socket_Strips:Socket_Strip_Straight_1x03_Pitch2.54mm, F.Cu at (169.9, 144.2)
- added L1: Ferrite_Bead, Resistors_SMD:R_0805, F.Cu at (165.1, 138.8)
- added L2: Ferrite_Bead, Resistors_SMD:R_0805, F.Cu at (144.5, 179.0)
- added L3: XFL4020-152ME, resonator:XFL4020, F.Cu at (157.7, 134.3)
- added P2: CONN_01X02, Socket_Strips:Socket_Strip_Straight_1x02_Pitch2.54mm, F.Cu at (171.2, 155.6)
- added P3: CONN_02X02, Socket_Strips:Socket_Strip_Straight_2x02_Pitch2.54mm, F.Cu at (82.8, 121.3)
- added P4: CONN_02X02, Socket_Strips:Socket_Strip_Straight_2x02_Pitch2.54mm, F.Cu at (85.3, 131.2)
- added P5: CONN_01X03, Socket_Strips:Socket_Strip_Straight_1x03_Pitch2.54mm, F.Cu at (177.0, 144.7)
- added R1: 10k, Resistors_SMD:R_0805, F.Cu at (151.6, 170.6)
- added R10: 51, Resistors_SMD:R_0805, F.Cu at (144.3, 194.7)
- added R11: 51, Resistors_SMD:R_0805, F.Cu at (139.2, 156.1)
- added R12: 10k, Resistors_SMD:R_0603, F.Cu at (160.0, 169.6)
- added R13: 680k, Resistors_SMD:R_0603, F.Cu at (139.2, 161.7)
- added R14: 130k, Resistors_SMD:R_0603, F.Cu at (138.7, 172.4)
- added R15: 100k, Resistors_SMD:R_0603, F.Cu at (138.2, 180.7)
- added R2: 100, Resistors_SMD:R_0805, F.Cu at (144.8, 171.3)
- added R3: 100, Resistors_SMD:R_0805, F.Cu at (160.5, 179.0)
- added R4: 51, Resistors_SMD:R_0805, F.Cu at (152.4, 179.0)
- added R5: 51, Resistors_SMD:R_0805, F.Cu at (161.0, 187.1)
- added R6: 51, Resistors_SMD:R_0805, F.Cu at (152.4, 187.9)
- added R7: 51, Resistors_SMD:R_0805, F.Cu at (144.3, 186.6)
- added R8: 51, Resistors_SMD:R_0805, F.Cu at (160.8, 193.9)
- added R9: 51, Resistors_SMD:R_0805, F.Cu at (152.1, 195.2)
- added RV1: 10K POT_TRIM, Potentiometers:Potentiometer_Trimmer-EVM3E, F.Cu at (190.0, 149.0)
- added U1: PAM8302AASCR, Housings_SSOP:MSOP-8_3x3mm_Pitch0.65mm, F.Cu at (190.5, 157.9)
- added U2: TPS63070, resonator:TPS63071, F.Cu at (159.5, 164.5)
- CF11, CF26, CF27: value 0.1uF -> 1uF
- CF13: value 0.1uF -> 4.7uF
- CF14, CF21: value 1uF -> 0.1uF
- CF15, CF22: value 4.7uF -> 0.1uF
- CF28: value 1uF -> 4.7uF
- CF33: value 100n -> 33uF
- CF34: value 33uF -> 100n
- FT1: value FT2232D -> FT2232D-REEL
- IC1: value MT48LC4M16A2P -> W9812G6KH
- UF2: value ZLDO1117G12TA -> ZLDO1117G33TA
- UF3: value ZLDO1117G33TA -> ZLDO1117G12TA
- X1: value OSCILLATORS-1 -> ASV-32.000MHZ-E-T
- moved JMS1 1.28 mm to (127.5, 53.7)
Connections:
- net /F_TDO renamed /spartan6/F_TDO
- net /serial_interface/nSRST renamed Net-(FT1-Pad17)
- net /serial_interface/nTRST renamed Net-(FT1-Pad20)
- net /spartan6/AS0 renamed Net-(UF1-Pad47)
- net /spartan6/AS7 renamed Net-(UF1-Pad39)
- net /spartan6/CAS renamed /spartan6/~CAS
- net /spartan6/CS renamed /spartan6/~CS
- net /spartan6/IO15 renamed Net-(UF1-Pad34)
- net /spartan6/IO46 renamed Net-(PFIO2-Pad10)
- net /spartan6/IO56 renamed /spartan6/TMDS_D2_N
- net /spartan6/IO57 renamed /spartan6/TMDS_D2_P
- net /spartan6/IO58 renamed /spartan6/TMDS_D1_N
- net /spartan6/IO59 renamed /spartan6/TMDS_D1_P
- net /spartan6/IO62 renamed /spartan6/TMDS_D0_N
- net /spartan6/IO63 renamed /spartan6/TMDS_D0_P
- net /spartan6/IO72 renamed /spartan6/TMDS_CLK_N
- net /spartan6/IO73 renamed /spartan6/TMDS_CLK_P
- net /spartan6/RAS renamed /spartan6/~RAS
- net /spartan6/WE renamed /spartan6/~WE
- net Net-(RF1-Pad2) renamed /spartan6/REBOOT
- CF1 pad 1: +3.3VDAC -> +3V3
- CF10 pad 1: +3.3VDAC -> +3V3
- CF11 pad 1: +3.3VDAC -> +3V3
- CF12 pad 1: +3.3VDAC -> +3V3
- CF13 pad 1: +3.3VDAC -> +3V3
- CF14 pad 1: +3.3VDAC -> +3V3
- CF15 pad 1: +3.3VDAC -> +3V3
- CF16 pad 1: +3.3VDAC -> +1V2
- CF17 pad 1: +3.3VDAC -> +3V3
- CF18 pad 1: +3.3VDAC -> +1V2
- CF19 pad 1: +3.3VDAC -> +1V2
- CF2 pad 1: +3.3VDAC -> +3V3
- CF20 pad 1: +3.3VDAC -> +3V3
- CF21 pad 1: +3.3VDAC -> +3V3
- CF22 pad 1: +3.3VDAC -> +1V2
- CF23 pad 1: +1V2 -> +3V3
- CF25 pad 1: +1V2 -> +3V3
- CF27 pad 1: +1V2 -> +3V3
- CF29 pad 1: +1V2 -> +3V3
- CF3 pad 1: +3.3VDAC -> +3V3
- CF30 pad 1: +3.3VDAC -> +5V
- CF31 pad 1: +1V2 -> +3V3
- CF32 pad 1: +1V2 -> +3V3
- CF33 pad 1: +3.3VDAC -> +3V3
- CF34 pad 1: +3.3VDAC -> +1V2
- CF35 pad 1: +5V -> +1V2
- CF36 pad 1: +5V -> /Power/USBVCC
- CF39 pad 1: +3V3 -> Net-(CF39-Pad1)
- CF4 pad 1: +3.3VDAC -> +3V3
- CF5 pad 1: +3.3VDAC -> +3V3
- CF6 pad 1: +3.3VDAC -> +3V3
- CF7 pad 1: +3.3VDAC -> +3V3
- CF8 pad 1: +3.3VDAC -> +3V3
- CF9 pad 1: +3.3VDAC -> +3V3
- FT1 pad 23: /serial_interface/TDI -> /spartan6/F_TDI
- FT1 pad 39: /serial_interface/RXD -> /spartan6/F_RXD
- FT1 pad 40: /serial_interface/TXD -> /spartan6/F_TXD
- FT1 pad 6: +3V3 -> Net-(CF39-Pad1)
- IC1 pad 1: +3.3VDAC -> +3V3
- IC1 pad 14: +3.3VDAC -> +3V3
- IC1 pad 27: +3.3VDAC -> +3V3
- IC1 pad 3: +3.3VDAC -> +3V3
- IC1 pad 43: +3.3VDAC -> +3V3
- IC1 pad 49: +3.3VDAC -> +3V3
- IC1 pad 9: +3.3VDAC -> +3V3
- JMS1 pad 1: Net-(DP1-Pad1) -> Net-(F1-Pad2)
- LF11 pad 1: +5V -> /Power/USBVCC
- PFIO1 pad 1: /spartan6/IO70 -> Net-(PFIO1-Pad1)
- PFIO1 pad 11: /spartan6/IO60 -> Net-(PFIO1-Pad11)
- PFIO1 pad 12: /spartan6/IO61 -> Net-(PFIO1-Pad12)
- PFIO1 pad 13: GND -> Net-(PFIO1-Pad13)
- PFIO1 pad 14: /spartan6/IO31 -> Net-(PFIO1-Pad14)
- PFIO1 pad 15: /spartan6/IO30 -> Net-(PFIO1-Pad15)
- PFIO1 pad 16: /spartan6/IO29 -> Net-(PFIO1-Pad16)
- PFIO1 pad 17: /spartan6/IO28 -> Net-(PFIO1-Pad17)
- PFIO1 pad 18: /spartan6/IO27 -> Net-(PFIO1-Pad18)
- PFIO1 pad 19: /spartan6/IO26 -> Net-(PFIO1-Pad19)
- PFIO1 pad 2: /spartan6/IO71 -> Net-(PFIO1-Pad2)
- PFIO1 pad 20: /spartan6/IO25 -> Net-(PFIO1-Pad20)
- PFIO1 pad 21: /spartan6/IO24 -> Net-(PFIO1-Pad21)
- PFIO1 pad 22: /spartan6/IO23 -> Net-(PFIO1-Pad22)
- PFIO1 pad 23: /spartan6/IO22 -> Net-(PFIO1-Pad23)
- PFIO1 pad 24: /spartan6/IO21 -> Net-(PFIO1-Pad24)
- PFIO1 pad 25: /spartan6/IO20 -> Net-(PFIO1-Pad25)
- PFIO1 pad 26: /spartan6/IO19 -> Net-(PFIO1-Pad26)
- PFIO1 pad 27: /spartan6/IO18 -> Net-(PFIO1-Pad27)
- PFIO1 pad 28: /spartan6/IO17 -> Net-(PFIO1-Pad28)
- PFIO1 pad 29: GND -> Net-(PFIO1-Pad29)
- PFIO1 pad 3: /spartan6/IO68 -> Net-(PFIO1-Pad3)
- PFIO1 pad 30: +3.3VDAC -> Net-(PFIO1-Pad30)
- PFIO1 pad 4: /spartan6/IO69 -> Net-(PFIO1-Pad4)
- PFIO1 pad 5: /spartan6/IO66 -> Net-(PFIO1-Pad5)
- PFIO1 pad 6: /spartan6/IO67 -> Net-(PFIO1-Pad6)
- PFIO1 pad 7: /spartan6/IO64 -> Net-(PFIO1-Pad7)
- PFIO1 pad 8: /spartan6/IO65 -> Net-(PFIO1-Pad8)
- PFIO2 pad 1: /spartan6/IO55 -> Net-(PFIO2-Pad1)
- PFIO2 pad 11: /spartan6/IO45 -> Net-(PFIO2-Pad11)
- PFIO2 pad 12: /spartan6/IO44 -> Net-(PFIO2-Pad12)
- PFIO2 pad 13: /spartan6/IO43 -> Net-(PFIO2-Pad13)
- PFIO2 pad 14: /spartan6/IO42 -> Net-(PFIO2-Pad14)
- PFIO2 pad 15: /spartan6/IO41 -> Net-(PFIO2-Pad15)
- PFIO2 pad 16: /spartan6/IO40 -> Net-(PFIO2-Pad16)
- PFIO2 pad 17: /spartan6/IO39 -> Net-(PFIO2-Pad17)
- PFIO2 pad 18: /spartan6/IO38 -> Net-(PFIO2-Pad18)
- PFIO2 pad 19: /spartan6/IO37 -> Net-(PFIO2-Pad19)
- PFIO2 pad 2: /spartan6/IO54 -> Net-(PFIO2-Pad2)
- PFIO2 pad 20: /spartan6/IO36 -> Net-(PFIO2-Pad20)
- PFIO2 pad 21: /spartan6/IO35 -> Net-(PFIO2-Pad21)
- PFIO2 pad 22: /spartan6/IO34 -> Net-(PFIO2-Pad22)
- PFIO2 pad 23: /spartan6/IO33 -> Net-(PFIO2-Pad23)
- PFIO2 pad 24: /spartan6/IO32 -> Net-(PFIO2-Pad24)
- PFIO2 pad 3: /spartan6/IO53 -> Net-(PFIO2-Pad3)
- PFIO2 pad 4: /spartan6/IO52 -> Net-(PFIO2-Pad4)
- PFIO2 pad 5: /spartan6/IO51 -> Net-(PFIO2-Pad5)
- PFIO2 pad 6: /spartan6/IO50 -> Net-(PFIO2-Pad6)
- PFIO2 pad 7: /spartan6/IO49 -> Net-(PFIO2-Pad7)
- PFIO2 pad 8: /spartan6/IO48 -> Net-(PFIO2-Pad8)
- PFIO2 pad 9: /spartan6/IO47 -> Net-(PFIO2-Pad9)
- PS1 pad 1: +5V -> +9V
- Pl1 pad 1: +3.3VDAC -> +3V3
- Pl1 pad 10: /spartan6/IO21 -> /spartan6/CH2P
- Pl1 pad 11: /spartan6/IO24 -> /spartan6/CH3N
- Pl1 pad 12: /spartan6/IO23 -> /spartan6/CH3P
- Pl1 pad 15: /spartan6/IO25 -> /spartan6/CLKN
- Pl1 pad 16: /spartan6/IO26 -> /spartan6/CLKP
- Pl1 pad 17: /spartan6/IO24 -> /spartan6/CH4N
- Pl1 pad 18: /spartan6/IO28 -> /spartan6/CH4P
- Pl1 pad 2: +3.3VDAC -> +3V3
- Pl1 pad 3: +3.3VDAC -> +3V3
- Pl1 pad 7: /spartan6/IO18 -> /spartan6/CH1N
- Pl1 pad 8: /spartan6/IO19 -> /spartan6/CH1P
- Pl1 pad 9: /spartan6/IO20 -> /spartan6/CH2N
- RF1 pad 1: +3.3VDAC -> +3V3
- RF2 pad 1: +3.3VDAC -> Net-(RF2-Pad1)
- RF2 pad 2: Net-(RF2-Pad2) -> +3V3
- RF21 pad 2: /serial_interface/RXD -> /spartan6/F_RXD
- RF3 pad 1: /P_TDO -> /spartan6/F_TDI
- UF1 pad 100: /spartan6/IO51 -> Net-(UF1-Pad100)
- UF1 pad 101: /spartan6/IO52 -> /spartan6/F_TXD
- UF1 pad 102: /spartan6/IO53 -> Net-(UF1-Pad102)
- UF1 pad 103: +3.3VDAC -> +3V3
- UF1 pad 104: /spartan6/IO54 -> Net-(UF1-Pad104)
- UF1 pad 105: /spartan6/IO55 -> /spartan6/F_RXD
- UF1 pad 116: /spartan6/IO60 -> Net-(UF1-Pad116)
- UF1 pad 117: /spartan6/IO61 -> Net-(UF1-Pad117)
- UF1 pad 120: /spartan6/IO64 -> Net-(UF1-Pad120)
- UF1 pad 121: /spartan6/IO65 -> Net-(UF1-Pad121)
- UF1 pad 122: +3.3VDAC -> +3V3
- UF1 pad 123: /spartan6/IO66 -> Net-(UF1-Pad123)
- UF1 pad 124: /spartan6/IO67 -> Net-(UF1-Pad124)
- UF1 pad 125: +3.3VDAC -> +3V3
- UF1 pad 126: /spartan6/IO68 -> Net-(UF1-Pad126)
- UF1 pad 127: /spartan6/IO69 -> Net-(UF1-Pad127)
- UF1 pad 129: +3.3VDAC -> +3V3
- UF1 pad 131: /spartan6/IO70 -> Net-(UF1-Pad131)
- UF1 pad 132: /spartan6/IO71 -> Net-(UF1-Pad132)
- UF1 pad 135: +3.3VDAC -> +3V3
- UF1 pad 144: +3.3VDAC -> +3V3
- UF1 pad 18: +3.3VDAC -> +3V3
- UF1 pad 20: +3.3VDAC -> +3V3
- UF1 pad 31: +3.3VDAC -> +3V3
- UF1 pad 36: +3.3VDAC -> +3V3
- UF1 pad 38: Net-(RF2-Pad2) -> Net-(RF2-Pad1)
- UF1 pad 4: +3.3VDAC -> +3V3
- UF1 pad 42: +3.3VDAC -> +3V3
- UF1 pad 48: /spartan6/IO17 -> Net-(UF1-Pad48)
- UF1 pad 50: /spartan6/IO18 -> /spartan6/CH1N
- UF1 pad 51: /spartan6/IO19 -> /spartan6/CH1P
- UF1 pad 53: +3.3VDAC -> +3V3
- UF1 pad 55: /spartan6/IO20 -> /spartan6/CH2N
- UF1 pad 56: /spartan6/IO21 -> /spartan6/CH2P
- UF1 pad 57: /spartan6/IO22 -> /spartan6/CH3N
- UF1 pad 58: /spartan6/IO23 -> /spartan6/CH3P
- UF1 pad 59: /spartan6/IO24 -> Net-(UF1-Pad59)
- UF1 pad 61: /spartan6/IO25 -> /spartan6/CLKN
- UF1 pad 62: /spartan6/IO26 -> /spartan6/CLKP
- UF1 pad 63: +3.3VDAC -> +3V3
- UF1 pad 64: /spartan6/IO27 -> /spartan6/CH4N
- UF1 pad 65: /spartan6/IO28 -> /spartan6/CH4P
- UF1 pad 66: /spartan6/IO29 -> Net-(UF1-Pad66)
- UF1 pad 67: /spartan6/IO30 -> Net-(UF1-Pad67)
- UF1 pad 69: +3.3VDAC -> +3V3
- UF1 pad 70: /spartan6/IO31 -> Net-(UF1-Pad70)
- UF1 pad 74: /spartan6/IO32 -> Net-(UF1-Pad74)
- UF1 pad 75: /spartan6/IO33 -> Net-(UF1-Pad75)
- UF1 pad 76: +3.3VDAC -> +3V3
- UF1 pad 78: /spartan6/IO34 -> Net-(UF1-Pad78)
- UF1 pad 79: /spartan6/IO35 -> Net-(UF1-Pad79)
- UF1 pad 80: /spartan6/IO36 -> Net-(UF1-Pad80)
- UF1 pad 81: /spartan6/IO37 -> Net-(UF1-Pad81)
- UF1 pad 82: /spartan6/IO38 -> Net-(UF1-Pad82)
- UF1 pad 83: /spartan6/IO39 -> Net-(UF1-Pad83)
- UF1 pad 84: /spartan6/IO40 -> Net-(UF1-Pad84)
- UF1 pad 85: /spartan6/IO41 -> Net-(UF1-Pad85)
- UF1 pad 86: +3.3VDAC -> +3V3
- UF1 pad 87: /spartan6/IO42 -> Net-(UF1-Pad87)
- UF1 pad 88: /spartan6/IO43 -> Net-(UF1-Pad88)
- UF1 pad 90: +3.3VDAC -> +3V3
- UF1 pad 92: /spartan6/IO44 -> Net-(UF1-Pad92)
- UF1 pad 93: /spartan6/IO45 -> Net-(UF1-Pad93)
- UF1 pad 95: /spartan6/IO47 -> Net-(UF1-Pad95)
- UF1 pad 97: /spartan6/IO48 -> Net-(UF1-Pad97)
- UF1 pad 98: /spartan6/IO49 -> Net-(UF1-Pad98)
- UF1 pad 99: /spartan6/IO50 -> Net-(UF1-Pad99)
- UF2 pad 2: +1V2 -> +3V3
- UF2 pad 3: +3.3VDAC -> +5V
- UF2 pad 4: +1V2 -> +3V3
- UF3 pad 2: +3.3VDAC -> +1V2
- UF3 pad 3: +5V -> +3V3
- UF3 pad 4: +3.3VDAC -> +1V2
- X1 pad 1: +3.3VDAC -> +3V3
- X1 pad 4: +3.3VDAC -> +3V3
Routing:
- net Net-(PFIO1-Pad16): track 0.00 -> 24.4 mm, vias 0 -> 1
- net /spartan6/IO29: track 23.6 -> 0.00 mm, vias 1 -> 0
- net +3V3: track 0.00 -> 8.70 mm
- net +3.3VDAC: track 8.70 -> 0.00 mm
- net Net-(PFIO1-Pad7): track 0.00 -> 8.00 mm, vias 0 -> 4
- net /spartan6/IO64: track 8.00 -> 0.00 mm, vias 4 -> 0
- net Net-(PFIO1-Pad8): track 0.00 -> 6.86 mm, vias 0 -> 1
- net /spartan6/IO65: track 6.86 -> 0.00 mm, vias 1 -> 0
- net /spartan6/IO27: track 5.63 -> 0.00 mm
- net Net-(PFIO1-Pad18): track 0.00 -> 4.78 mm
- net Net-(PFIO1-Pad1): track 0.00 -> 1.73 mm
- net /spartan6/IO70: track 1.73 -> 0.00 mm
- net Net-(PFIO1-Pad3): vias 0 -> 1
- net /spartan6/IO68: vias 1 -> 0

Commit message: Organizando PIN OUT vr.:0.1
by Ruben
Parts:
- removed PFIO1, PFIO2: CONN_02X15, Socket_Strips:Socket_Strip_Straight_2x15_Pitch2.54mm
- added LVDS1: CONN_02X15, Pin_Headers:Pin_Header_Straight_2x15_Pitch2.00mm, F.Cu at (106.7, 145.1)
- added P1: CONN_01X03, Socket_Strips:Socket_Strip_Straight_1x03_Pitch1.27mm, F.Cu at (130.3, 159.9)
- added PIO1: CONN_02X20, Socket_Strips:Socket_Strip_Straight_2x20_Pitch2.54mm, F.Cu at (130.0, 66.9)
- added S1: B3SL-1002P, Buttons_Switches_SMD:SW_SPST_B3SL-1002P, F.Cu at (117.3, 159.4)
- added SW1: B3SL-1002P, Buttons_Switches_SMD:SW_SPST_B3SL-1002P, F.Cu at (106.7, 145.1)
- F1: value MF-MSMF050-2 -> PTS08056V050
- moved TH1 83.6 mm to (88.9, 153.6)
- moved TH12 83.6 mm to (91.4, 153.6)
- moved TH15 83.6 mm to (94.0, 153.6)
- moved J2 51.0 mm to (125.0, 120.0), turned to 90 degrees
- moved RV1 29.6 mm to (170.9, 171.6)
- moved U1 20.0 mm to (171.2, 163.0)
- moved FT1 6.40 mm to (120.4, 75.6)
- moved UF1 5.09 mm to (98.0, 75.6)
Connections:
- net +5VA renamed /serial_interface/+5VA
- DF1 pad 1: /spartan6/IO7 -> /spartan6/IO_LED
- P5 pad 2: +5V -> /spartan6/F_~SD
- R1 pad 1: +5V -> /spartan6/F_~SD
- R1 pad 2: +5V -> Net-(R1-Pad2)
- U1 pad 1: +5V -> /spartan6/F_~SD
- UF1 pad 100: Net-(UF1-Pad100) -> /spartan6/IO25
- UF1 pad 102: Net-(UF1-Pad102) -> /spartan6/IO26
- UF1 pad 104: Net-(UF1-Pad104) -> /spartan6/IO27
- UF1 pad 116: Net-(UF1-Pad116) -> /spartan6/IO28
- UF1 pad 117: Net-(UF1-Pad117) -> /spartan6/IO29
- UF1 pad 120: Net-(UF1-Pad120) -> /spartan6/IO30
- UF1 pad 121: Net-(UF1-Pad121) -> /spartan6/IO31
- UF1 pad 123: Net-(UF1-Pad123) -> /spartan6/IO32
- UF1 pad 124: Net-(UF1-Pad124) -> /spartan6/IO33
- UF1 pad 126: Net-(UF1-Pad126) -> /spartan6/IO34
- UF1 pad 127: Net-(UF1-Pad127) -> /spartan6/IO35
- UF1 pad 131: Net-(UF1-Pad131) -> /spartan6/IO36
- UF1 pad 132: Net-(UF1-Pad132) -> /spartan6/IO37
- UF1 pad 34: Net-(UF1-Pad34) -> /spartan6/F_~SD
- UF1 pad 39: Net-(UF1-Pad39) -> /spartan6/IO01
- UF1 pad 47: Net-(UF1-Pad47) -> /spartan6/IO02
- UF1 pad 48: Net-(UF1-Pad48) -> /spartan6/IO03
- UF1 pad 59: Net-(UF1-Pad59) -> /spartan6/IO_LED
- UF1 pad 66: Net-(UF1-Pad66) -> /spartan6/IO04
- UF1 pad 67: Net-(UF1-Pad67) -> /spartan6/IO05
- UF1 pad 70: Net-(UF1-Pad70) -> +3V3
- UF1 pad 74: Net-(UF1-Pad74) -> /spartan6/IO07
- UF1 pad 75: Net-(UF1-Pad75) -> /spartan6/IO08
- UF1 pad 78: Net-(UF1-Pad78) -> /spartan6/IO09
- UF1 pad 79: Net-(UF1-Pad79) -> /spartan6/IO10
- UF1 pad 80: Net-(UF1-Pad80) -> /spartan6/IO11
- UF1 pad 81: Net-(UF1-Pad81) -> /spartan6/IO12
- UF1 pad 82: Net-(UF1-Pad82) -> /spartan6/IO13
- UF1 pad 83: Net-(UF1-Pad83) -> /spartan6/IO14
- UF1 pad 84: Net-(UF1-Pad84) -> /spartan6/IO15
- UF1 pad 85: Net-(UF1-Pad85) -> /spartan6/IO16
- UF1 pad 87: Net-(UF1-Pad87) -> /spartan6/IO17
- UF1 pad 88: Net-(UF1-Pad88) -> /spartan6/IO18
- UF1 pad 92: Net-(UF1-Pad92) -> /spartan6/IO19
- UF1 pad 93: Net-(UF1-Pad93) -> /spartan6/IO20
- UF1 pad 95: Net-(UF1-Pad95) -> /spartan6/IO21
- UF1 pad 97: Net-(UF1-Pad97) -> /spartan6/IO22
- UF1 pad 98: Net-(UF1-Pad98) -> /spartan6/IO23
- UF1 pad 99: Net-(UF1-Pad99) -> /spartan6/IO24
Routing:
- net (no net): track 3280.1 -> 3325.9 mm, vias 172 -> 179
- net Net-(PFIO1-Pad16): track 24.4 -> 0.00 mm, vias 1 -> 0
- net Net-(PFIO1-Pad7): track 8.00 -> 0.00 mm, vias 4 -> 0
- net Net-(PFIO1-Pad8): track 6.86 -> 0.00 mm, vias 1 -> 0
- net Net-(PFIO1-Pad18): track 4.78 -> 0.00 mm
- net Net-(PFIO1-Pad1): track 1.73 -> 0.00 mm
- net Net-(PFIO1-Pad3): vias 1 -> 0

Commit message: Terminado Shield
by Ruben
Parts:
- moved J2 18.6 mm to (143.5, 118.3)
- moved PIO1 3.31 mm to (130.3, 70.2)
Routing:
- net (no net): track 3325.9 -> 3259.9 mm
- net GND: track 0.00 -> 35.1 mm
- net /spartan6/TMDS_CLK_P: track 0.00 -> 30.8 mm
Changed lines of the file:
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@@
   (general
     (links 472)
-    (no_connects 467)
-    (area 79.924999 49.854999 133.415001 135.095001)
+    (no_connects 464)
+    (area 19.3 14.004 185.494 198.343)
     (thickness 1.6)
     (drawings 14)
@@
   )
   (module Socket_Strips:Socket_Strip_Straight_1x03_Pitch2.54mm (layer F.Cu)
-    (at 124.958 120.034 90)
+    (at 143.5 118.256 90)
     (descr "Through hole straight socket strip, 1x03, 2.54mm pitch, single row")
     (tags "Through hole socket strip THT 1x03 2.54mm single row")
@@
   )
   (module Socket_Strips:Socket_Strip_Straight_2x20_Pitch2.54mm (layer F.Cu)
-    (at 130.038 66.948)
+    (at 130.292 70.25)
     (descr "Through hole straight socket strip, 2x20, 2.54mm pitch, double rows")
     (tags "Through hole socket strip THT 2x20 2.54mm double row")
@@
   (segment (start 89.37 73.1) (end 89.37 73.11184) (width 0.2) (layer B.Cu) (net 0) (status 30))
   (segment (start 87.04 72.89) (end 86.83 73.1) (width 0.2) (layer F.Cu) (net 0) (status 30))
-  (segment (start 86.81152 70.54152) (end 86.83 70.56) (width 0.2) (layer F.Cu) (net 0) (status 30))
-  (segment (start 89.37 68.02) (end 89.37 68.042) (width 0.2) (layer F.Cu) (net 0) (status 30))
   (segment (start 28.89 95.64) (end 28.89 98.0278) (width 0.2) (layer F.Cu) (net 0) (status 30))
   (segment (start 28.89 98.0278) (end 28.72224 98.19556) (width 0.2) (layer F.Cu) (net 0) (status 30))
@@
   (segment (start 77.95 79.8) (end 77.95 76.6) (width 0.2) (layer F.Cu) (net 0))
   (segment (start 83.58 75.37) (end 84.02 75.37) (width 0.2) (layer F.Cu) (net 0) (status 30))
-  (segment (start 88.77964 69.00036) (end 85.01312 69.00036) (width 0.2) (layer F.Cu) (net 0))
-  (segment (start 90.07 67.71) (end 88.77964 69.00036) (width 0.2) (layer F.Cu) (net 0))
-  (segment (start 85.01312 69.00036) (end 84.33748 69.676) (width 0.2) (layer F.Cu) (net 0))
-  (segment (start 84.33748 69.676) (end 66.6032 69.676) (width 0.2) (layer F.Cu) (net 0))
-  (segment (start 66.6032 69.676) (end 62.03 74.2492) (width 0.2) (layer F.Cu) (net 0))
-  (segment (start 62.03 74.2492) (end 62.03 78.6) (width 0.2) (layer F.Cu) (net 0) (status 20))
   (segment (start 82.39 73.65) (end 84.07 75.33) (width 0.2) (layer F.Cu) (net 0))
   (segment (start 52.5824 93.9584) (end 52.9908 93.55) (width 0.2) (layer F.Cu) (net 0))
@@
   (segment (start 85.6634 67.71) (end 84.2054 69.168) (width 0.2) (layer F.Cu) (net 0))
   (segment (start 87.53 67.71) (end 85.6634 67.71) (width 0.2) (layer F.Cu) (net 0))
-  (segment (start 87.53 70.25) (end 66.80644 70.25) (width 0.2) (layer F.Cu) (net 0))
-  (segment (start 62.53 74.52644) (end 62.53 78.6) (width 0.2) (layer F.Cu) (net 0))
-  (segment (start 66.80644 70.25) (end 62.53 74.52644) (width 0.2) (layer F.Cu) (net 0))
   (segment (start 68.53 78.6) (end 68.53 76.9622) (width 0.2) (layer F.Cu) (net 0))
   (segment (start 68.1526 72.0636) (end 68.178 72.0636) (width 0.2) (layer B.Cu) (net 0))
@@
   (segment (start 86 95.55) (end 86 96.95) (width 0.2) (layer B.Cu) (net 0))
   (segment (start 87.19536 94.35464) (end 86 95.55) (width 0.2) (layer B.Cu) (net 0))
+  (segment (start 88.77964 69.00036) (end 85.01312 69.00036) (width 0.2) (layer F.Cu) (net 1))
+  (segment (start 90.07 67.71) (end 88.77964 69.00036) (width 0.2) (layer F.Cu) (net 1))
+  (segment (start 85.01312 69.00036) (end 84.33748 69.676) (width 0.2) (layer F.Cu) (net 1))
+  (segment (start 84.33748 69.676) (end 66.6032 69.676) (width 0.2) (layer F.Cu) (net 1))
+  (segment (start 66.6032 69.676) (end 62.03 74.2492) (width 0.2) (layer F.Cu) (net 1))
+  (segment (start 62.03 74.2492) (end 62.03 78.6) (width 0.2) (layer F.Cu) (net 1) (status 20))
+  (segment (start 89.37 68.02) (end 89.37 68.042) (width 0.2) (layer F.Cu) (net 2) (status 30))
+  (segment (start 86.81152 70.54152) (end 86.83 70.56) (width 0.2) (layer F.Cu) (net 23) (status 30))
   (segment (start 83.46058 121.13) (end 83.50068 121.1701) (width 0.2) (layer F.Cu) (net 23) (status 30))
   (segment (start 79.402 121.13) (end 83.46058 121.13) (width 0.2) (layer F.Cu) (net 23) (status 30))
@@
   (segment (start 79.822 123.34) (end 79.582 123.58) (width 0.2) (layer F.Cu) (net 23) (status 30))
   (segment (start 80.94 123.34) (end 79.822 123.34) (width 0.5) (layer F.Cu) (net 23) (status 20))
+  (segment (start 87.53 70.25) (end 66.80644 70.25) (width 0.2) (layer F.Cu) (net 130))
+  (segment (start 62.53 74.52644) (end 62.53 78.6) (width 0.2) (layer F.Cu) (net 130))
+  (segment (start 66.80644 70.25) (end 62.53 74.52644) (width 0.2) (layer F.Cu) (net 130))
   (zone (net 1) (net_name GND) (layer F.Cu) (hatch edge 0.508)
     (connect_pads (clearance 0.2))

Commit message: shield 2.0
Parts:
- removed Pl1: CONN_02X15, Pin_Headers:Pin_Header_Straight_2x15_Pitch2.00mm
- moved SW1 11.4 mm to (117.8, 142.9)
- moved PIO1 4.10 mm to (130.8, 66.2)
