File: hard/hw/Basic_pcb/HDMIspartan6_Board.kicad_pcb (KiCad board)
At the start: 4 copper layers, 53.3 x 85.1 mm, 164 parts, among them IC1 W9812G6KH, J1 HDMI_A, P1 CONN_01X03, P2 CONN_01X02, P3 CONN_02X02, P4 CONN_02X02, P5 CONN_01X03, P7 B6B-PH-K-S(LF)(SN), SW1 B3SL-1002P, U1 PAM8302AASCR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

Commit message: update
Parts:
- added P6: CONN_01X03, Socket_Strips:Socket_Strip_Straight_1x03_Pitch2.54mm, F.Cu at (103.9, 93.2)
- added PIO1: CONN_02X10, Socket_Strips:Socket_Strip_Straight_2x10_Pitch2.54mm, F.Cu at (49.3, 59.7)
- added PIO2: CONN_02X10, Socket_Strips:Socket_Strip_Straight_2x10_Pitch2.54mm, F.Cu at (106.4, 82.8)
- DF1, RF1, RF5: moved to F.Cu
- U1, XF2: moved to B.Cu
- moved LF11 84.1 mm to (125.7, 28.0)
- moved CF36 73.7 mm to (120.1, 45.5)
- moved DF1 71.3 mm to (97.9, 136.3)
- moved CF1 63.5 mm to (162.5, 79.2)
- moved CF5 63.5 mm to (160.3, 72.3)
- moved CF21 63.5 mm to (160.3, 74.3)
- moved R14 62.4 mm to (137.2, 122.2)
- moved RF5 61.1 mm to (97.8, 139.1)
- moved RF1 60.5 mm to (137.7, 78.1)
- moved RF4 60.2 mm to (156.3, 62.5)
- moved CF20 60.2 mm to (156.4, 67.2)
- moved CF3 60.2 mm to (156.8, 79.7)
- moved RF3 60.2 mm to (156.3, 61.1)
- moved RF6 60.2 mm to (156.3, 64.0)
- moved RF7 60.2 mm to (156.4, 65.6)
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
Commit message: LVDS ultimate test
by LUIS
Parts:
- C1, C2, C3, C4, C5, L1, L2, R1, R2, R3, RF1: moved to B.Cu
- moved P1 54.1 mm to (20.3, 62.6)
- moved RV1 52.2 mm to (24.8, 66.7), turned to 180 degrees
- moved P5 47.7 mm to (21.6, 74.6)
- moved U1 43.5 mm to (26.9, 78.9), turned to 270 degrees
- moved R1 43.3 mm to (16.3, 73.9), turned to 270 degrees
- moved R3 42.7 mm to (28.7, 74.1), turned to 90 degrees
- moved P2 41.7 mm to (20.3, 81.4), turned to 180 degrees
- moved R2 40.5 mm to (26.8, 74.1), turned to 90 degrees
- moved C1 39.6 mm to (24.3, 74.6), turned to 270 degrees
- moved RF1 38.3 mm to (100.1, 85.9), turned to 180 degrees
- moved C2 36.5 mm to (25.7, 71.4), turned to 180 degrees
- moved L1 33.9 mm to (23.4, 81.1), turned to 180 degrees
- moved C5 33.4 mm to (23.5, 77.3), turned to 180 degrees
- moved C3 27.8 mm to (30.2, 69.4), turned to 180 degrees
- moved C4 27.2 mm to (23.5, 83.0), turned to 180 degrees
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Other:
- board size 53.3 x 85.1 mm -> 60 x 85.1 mm

Commit message: Update board
by Ruben
Parts:
- C1, C4, C5, L1, L2, R1: moved to F.Cu
- moved R1 50.3 mm to (63.5, 91.6), turned to 90 degrees
- moved P1 50.0 mm to (64.8, 85.5)
- moved P2 45.6 mm to (61.0, 102.0)
- moved C4 45.3 mm to (64.0, 103.3)
- moved L1 45.3 mm to (64.0, 101.2)
- moved L2 45.3 mm to (64.0, 99.2)
- moved C5 45.1 mm to (64.0, 97.2)
- moved C1 44.5 mm to (65.5, 91.3)
- moved U1 43.0 mm to (64.3, 100.2)
- moved C2 42.7 mm to (63.5, 91.3), turned to 90 degrees
- moved P5 42.4 mm to (61.0, 90.3), turned to 0 degrees
- moved R3 42.2 mm to (65.5, 94.6)
- moved R2 42.1 mm to (63.5, 94.6)
- moved C3 41.6 mm to (65.5, 91.3), turned to 90 degrees
- moved RV1 40.4 mm to (62.5, 81.4), turned to 90 degrees
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Other:
- outline, holes or cut-outs redrawn
