File: hard/PCB/serial_interface.sch (KiCad schematic (older format))
At the start: 19 parts

Commit message: Update supply power
Parts:
- removed XF2: 6MHz, resonator:CSTCR6M00G53Z, symbol ABM8G
- added X2: CSTCR6M00G53Z-R0, Project:CSTCR6M00G53Z, symbol CSTCR6M00G53Z-R0
- CF36, CF38, CF39, CF40, CF41: footprint opendous:SM0603_Opendous -> Capacitors_SMD:C_0603
- CF37: footprint opendous:SM1210_Opendous -> Capacitors_SMD:C_0603
- FT1: footprint Housings_QFP:LQFP-48_7x7mm_Pitch0.5mm -> Project:LQFP-48_7x7mm_Pitch0.5mm
- JMS1: footprint Connect:USB_Mini-B -> Project:USB_Mini-B; DIGIKEY REF (none) -> ED2992TR-ND
- LF11: footprint opendous:SM0805 -> Resistors_SMD:R_0805_HandSoldering
- RF14, RF15, RF16, RF17, RF18, RF19, RF20, RF21: footprint opendous:SM0603_Opendous -> Resistors_SMD:R_0603
Connections:
- wire segments 75 -> 73
Other:
- note removed: "ED2992TR-ND"

Commit message: Corrección esquematico
Parts:
- LF1: renamed from LF11; DIGIKEY REF (none) -> 240-2398-1-ND
- renumbered CF40 to CF1, CF41 to CF2, CF36 to CF3, CF37 to CF4, CF39 to CF5, CF38 to CF6, RF14 to RF1, RF15 to RF2, RF17 to RF3, RF16 to RF4, RF18 to RF5, RF19 to RF6, RF20 to RF7, RF21 to RF8, X2 to XF1
Changed lines of the file:
@@
 $EndDescr
 $Comp
-L C CF40
+L C CF1
 U 1 1 4FC6CF8D
 P 5950 5500
-F 0 "CF40" H 6000 5600 50  0000 L CNN
+F 0 "CF1" H 6000 5600 50  0000 L CNN
 F 1 "47pF" V 6050 5250 50  0000 L CNN
 F 2 "Capacitors_SMD:C_0603" H 5950 5500 60  0001 C CNN
@@
 $EndComp
 $Comp
-L C CF41
+L C CF2
 U 1 1 4FC6CF5C
 P 5950 6100
-F 0 "CF41" H 6000 6200 50  0000 L CNN
+F 0 "CF2" H 6000 6200 50  0000 L CNN
 F 1 "47pF" V 6050 5850 50  0000 L CNN
 F 2 "Capacitors_SMD:C_0603" H 5950 6100 60  0001 C CNN
@@
 $EndComp
 $Comp
-L R RF20
+L R RF7
 U 1 1 4FC6C4A3
 P 10000 6800
-F 0 "RF20" V 10080 6800 50  0000 C CNN
+F 0 "RF7" V 10080 6800 50  0000 C CNN
 F 1 "10k" V 10000 6800 50  0000 C CNN
 F 2 "Resistors_SMD:R_0603" H 10000 6800 60  0001 C CNN
@@
 $EndComp
 $Comp
-L R RF19
+L R RF6
 U 1 1 4FC6C443
 P 10000 5300
-F 0 "RF19" V 10080 5300 50  0000 C CNN
+F 0 "RF6" V 10080 5300 50  0000 C CNN
 F 1 "10k" V 10000 5300 50  0000 C CNN
 F 2 "Resistors_SMD:R_0603" H 10000 5300 60  0001 C CNN
@@
 $EndComp
 $Comp
-L C CF39
+L C CF5
 U 1 1 4FC6C3C0
 P 7300 4300
-F 0 "CF39" V 7350 4400 50  0000 L CNN
+F 0 "CF5" V 7350 4400 50  0000 L CNN
 F 1 "33nF" V 7350 4050 50  0000 L CNN
 F 2 "Capacitors_SMD:C_0603" H 7300 4300 60  0001 C CNN
@@
 $EndComp
 $Comp
-L INDUCTOR LF11
+L INDUCTOR LF1
 U 1 1 4FC6C26A
 P 6850 2400
-F 0 "LF11" V 6800 2400 40  0000 C CNN
+F 0 "LF1" V 6800 2400 40  0000 C CNN
 F 1 "HZ0805D152R-10" V 6950 2400 40  0000 C CNN
 F 2 "Resistors_SMD:R_0805_HandSoldering" H 6850 2400 60  0001 C CNN
-F 3 "" H 6850 2400 60  0001 C CNN
+F 3 "https://assets.lairdtech.com/home/brandworld/files/HZ0805D152R-10.pdf" H 6850 2400 60  0001 C CNN
+F 4 "240-2398-1-ND" V 6850 2400 60  0001 C CNN "DIGIKEY REF"
 	1    6850 2400
 	0    -1   -1   0
 $EndComp
 $Comp
-L C CF37
+L C CF4
 U 1 1 4FC6C1A7
 P 7250 2650
-F 0 "CF37" H 7300 2750 50  0000 L CNN
+F 0 "CF4" H 7300 2750 50  0000 L CNN
 F 1 "10uF" H 7300 2550 50  0000 L CNN
 F 2 "Capacitors_SMD:C_0603" H 7250 2650 60  0001 C CNN
@@
 $EndComp
 $Comp
-L R RF18
+L R RF5
 U 1 1 4FC6BECA
 P 7900 2650
-F 0 "RF18" V 7980 2650 50  0000 C CNN
+F 0 "RF5" V 7980 2650 50  0000 C CNN
 F 1 "470R" V 7900 2650 50  0000 C CNN
 F 2 "Resistors_SMD:R_0603" H 7900 2650 60  0001 C CNN
@@
 $EndComp
 $Comp
-L C CF38
+L C CF6
 U 1 1 4FC6BE12
 P 7900 3100
-F 0 "CF38" H 7950 3200 50  0000 L CNN
+F 0 "CF6" H 7950 3200 50  0000 L CNN
 F 1 "100nF" H 7950 3000 50  0000 L CNN
 F 2 "Capacitors_SMD:C_0603" H 7900 3100 60  0001 C CNN
@@
 $EndComp
 $Comp
-L R RF16
+L R RF4
 U 1 1 4FC6BD44
 P 7250 6300
-F 0 "RF16" V 7330 6300 50  0000 C CNN
+F 0 "RF4" V 7330 6300 50  0000 C CNN
 F 1 "10K" V 7250 6300 50  0000 C CNN
 F 2 "Resistors_SMD:R_0603" H 7250 6300 60  0001 C CNN
@@
 $EndComp
 $Comp
-L C CF36
+L C CF3
 U 1 1 4FC6BCE9
 P 6450 2650
-F 0 "CF36" H 6500 2750 50  0000 L CNN
+F 0 "CF3" H 6500 2750 50  0000 L CNN
 F 1 "10nF" H 6500 2550 50  0000 L CNN
 F 2 "Capacitors_SMD:C_0603" H 6450 2650 60  0001 C CNN
@@
 $EndComp
 $Comp
-L R RF17
+L R RF3
 U 1 1 4FC6BC62
 P 7200 5200
-F 0 "RF17" V 7280 5200 50  0000 C CNN
+F 0 "RF3" V 7280 5200 50  0000 C CNN
 F 1 "1K5" V 7200 5200 50  0000 C CNN
 F 2 "Resistors_SMD:R_0603" H 7200 5200 60  0001 C CNN
@@
 $EndComp
 $Comp
-L R RF15
+L R RF2
 U 1 1 4FC6BC59
 P 6650 4900
-F 0 "RF15" V 6730 4900 50  0000 C CNN
+F 0 "RF2" V 6730 4900 50  0000 C CNN
 F 1 "27R" V 6650 4900 50  0000 C CNN
 F 2 "Resistors_SMD:R_0603" H 6650 4900 60  0001 C CNN
@@
 $EndComp
 $Comp
-L R RF14
+L R RF1
 U 1 1 4FC6BC34
 P 6650 4600
-F 0 "RF14" V 6730 4600 50  0000 C CNN
+F 0 "RF1" V 6730 4600 50  0000 C CNN
 F 1 "27R" V 6650 4600 50  0000 C CNN
 F 2 "Resistors_SMD:R_0603" H 6650 4600 60  0001 C CNN
@@
 RXD
 $Comp
-L R RF21
+L R RF8
 U 1 1 51CD787E
 P 10500 5000
-F 0 "RF21" V 10580 5000 50  0000 C CNN
+F 0 "RF8" V 10580 5000 50  0000 C CNN
 F 1 "15K" V 10500 5000 50  0000 C CNN
 F 2 "Resistors_SMD:R_0603" H 10500 5000 60  0001 C CNN
@@
 $EndComp
 $Comp
-L +3V3 #PWR14
+L +3V3 #PWR16
 U 1 1 589F5F40
 P 10300 5050
-F 0 "#PWR14" H 10300 4900 50  0001 C CNN
+F 0 "#PWR16" H 10300 4900 50  0001 C CNN
 F 1 "+3V3" H 10300 5190 50  0000 C CNN
 F 2 "" H 10300 5050 50  0000 C CNN
@@
 $EndComp
 $Comp
-L +3V3 #PWR11
+L +3V3 #PWR18
 U 1 1 589F6257
 P 10500 4800
-F 0 "#PWR11" H 10500 4650 50  0001 C CNN
+F 0 "#PWR18" H 10500 4650 50  0001 C CNN
 F 1 "+3V3" H 10500 4940 50  0000 C CNN
 F 2 "" H 10500 4800 50  0000 C CNN
@@
 $EndComp
 $Comp
-L +3V3 #PWR9
+L +3V3 #PWR15
 U 1 1 589F6BB3
 P 8800 3450
-F 0 "#PWR9" H 8800 3300 50  0001 C CNN
+F 0 "#PWR15" H 8800 3300 50  0001 C CNN
 F 1 "+3V3" H 8800 3590 50  0000 C CNN
 F 2 "" H 8800 3450 50  0000 C CNN
@@
 	6450 2500 6450 2400
 $Comp
-L GND #PWR6
+L GND #PWR9
 U 1 1 58A66750
 P 6450 2900
-F 0 "#PWR6" H 6450 2650 50  0001 C CNN
+F 0 "#PWR9" H 6450 2650 50  0001 C CNN
 F 1 "GND" H 6450 2750 50  0000 C CNN
 F 2 "" H 6450 2900 50  0000 C CNN
@@
 	7100 6300 6750 6300
 $Comp
-L GND #PWR7
+L GND #PWR11
 U 1 1 58A8D1C3
 P 7250 2900
-F 0 "#PWR7" H 7250 2650 50  0001 C CNN
+F 0 "#PWR11" H 7250 2650 50  0001 C CNN
 F 1 "GND" H 7250 2750 50  0000 C CNN
 F 2 "" H 7250 2900 50  0000 C CNN
@@
 $EndComp
 $Comp
-L GND #PWR8
+L GND #PWR13
 U 1 1 58A8D267
 P 7900 3350
-F 0 "#PWR8" H 7900 3100 50  0001 C CNN
+F 0 "#PWR13" H 7900 3100 50  0001 C CNN
 F 1 "GND" H 7900 3200 50  0000 C CNN
 F 2 "" H 7900 3350 50  0000 C CNN
@@
 $EndComp
 $Comp
-L GND #PWR18
+L GND #PWR14
 U 1 1 58A8D7DD
 P 8300 7400
-F 0 "#PWR18" H 8300 7150 50  0001 C CNN
+F 0 "#PWR14" H 8300 7150 50  0001 C CNN
 F 1 "GND" H 8300 7250 50  0000 C CNN
 F 2 "" H 8300 7400 50  0000 C CNN
@@
 $EndComp
 $Comp
-L GND #PWR16
+L GND #PWR12
 U 1 1 58A8DF8B
 P 7450 6450
-F 0 "#PWR16" H 7450 6200 50  0001 C CNN
+F 0 "#PWR12" H 7450 6200 50  0001 C CNN
 F 1 "GND" H 7450 6300 50  0000 C CNN
 F 2 "" H 7450 6450 50  0000 C CNN
@@
 $EndComp
 $Comp
-L GND #PWR15
+L GND #PWR8
 U 1 1 58A8E746
 P 5650 5900
-F 0 "#PWR15" H 5650 5650 50  0001 C CNN
+F 0 "#PWR8" H 5650 5650 50  0001 C CNN
 F 1 "GND" H 5650 5750 50  0000 C CNN
 F 2 "" H 5650 5900 50  0000 C CNN
@@
 $EndComp
 $Comp
-L GND #PWR13
+L GND #PWR7
 U 1 1 58A8EFD2
 P 5000 5050
-F 0 "#PWR13" H 5000 4800 50  0001 C CNN
+F 0 "#PWR7" H 5000 4800 50  0001 C CNN
 F 1 "GND" H 5000 4900 50  0000 C CNN
 F 2 "" H 5000 5050 50  0000 C CNN
@@
 $EndComp
 $Comp
-L GND #PWR12
+L GND #PWR6
 U 1 1 58A8F696
 P 3650 5050
-F 0 "#PWR12" H 3650 4800 50  0001 C CNN
+F 0 "#PWR6" H 3650 4800 50  0001 C CNN
 F 1 "GND" H 3650 4900 50  0000 C CNN
 F 2 "" H 3650 5050 50  0000 C CNN
@@
 $EndComp
 $Comp
-L CSTCR6M00G53Z-R0 X2
+L CSTCR6M00G53Z-R0 XF1
 U 1 1 592CD31A
 P 6300 5800
-F 0 "X2" H 6300 5700 60  0000 C CNN
+F 0 "XF1" H 6300 5700 60  0000 C CNN
 F 1 "CSTCR6M00G53Z-R0" V 6300 6350 60  0000 C CNN
 F 2 "Project:CSTCR6M00G53Z" H 6300 5800 60  0001 C CNN

Commit message: Correccion SCH
Parts:
- F1: footprint Resistors_SMD:R_1812 -> Project:R_1812
Changed lines of the file:
@@
 F 0 "F1" V 5030 4250 50  0000 C CNN
 F 1 "PTS08056V050" V 4850 4250 50  0000 C CNN
-F 2 "Resistors_SMD:R_1812" V 4880 4250 50  0001 C CNN
+F 2 "Project:R_1812" V 4880 4250 50  0001 C CNN
 F 3 "http://www.belfuse.com/pdfs/0ZCK.pdf" H 4950 4250 50  0001 C CNN
 F 4 "PTS08056V050-ND" V 4950 4250 60  0001 C CNN "REF DIGIKEY"

Commit message: 2xx40 conn
Parts:
- added J1: CONN_02X20, Project:Pin_Header_Straight_2x20_Pitch2.54mm, symbol CONN_02X20
Changed lines of the file:
@@
 	0    1    1    0
 $EndComp
+$Comp
+L CONN_02X20 J1
+U 1 1 592E2A0E
+P 13950 5450
+F 0 "J1" H 13950 6500 50  0000 C CNN
+F 1 "CONN_02X20" V 13950 5450 50  0000 C CNN
+F 2 "Project:Pin_Header_Straight_2x20_Pitch2.54mm" H 13950 4500 50  0001 C CNN
+F 3 "" H 13950 4500 50  0001 C CNN
+	1    13950 5450
+	1    0    0    -1
+$EndComp
 $EndSCHEMATC

Commit message: Add 3d model
Parts:
- removed J1: CONN_02X20, Project:Pin_Header_Straight_2x20_Pitch2.54mm, symbol CONN_02X20
Changed lines of the file:
@@
 	0    1    1    0
 $EndComp
-$Comp
-L CONN_02X20 J1
-U 1 1 592E2A0E
-P 13950 5450
-F 0 "J1" H 13950 6500 50  0000 C CNN
-F 1 "CONN_02X20" V 13950 5450 50  0000 C CNN
-F 2 "Project:Pin_Header_Straight_2x20_Pitch2.54mm" H 13950 4500 50  0001 C CNN
-F 3 "" H 13950 4500 50  0001 C CNN
-	1    13950 5450
-	1    0    0    -1
-$EndComp
 $EndSCHEMATC

Commit message: update 3d models
Parts:
- F1: footprint Project:R_1812 -> Resistors_SMD:R_0805
- renumbered CF3 to CF1, CF4 to CF2, CF6 to CF3, CF5 to CF4, CF1 to CF5, CF2 to CF6, RF5 to RF1, RF1 to RF2, RF2 to RF3, RF8 to RF4, RF3 to RF5, RF4 to RF7, RF7 to RF8
Changed lines of the file:
@@
 $EndDescr
 $Comp
-L C CF1
+L C CF5
 U 1 1 4FC6CF8D
 P 5950 5500
-F 0 "CF1" H 6000 5600 50  0000 L CNN
+F 0 "CF5" H 6000 5600 50  0000 L CNN
 F 1 "47pF" V 6050 5250 50  0000 L CNN
 F 2 "Capacitors_SMD:C_0603" H 5950 5500 60  0001 C CNN
@@
 $EndComp
 $Comp
-L C CF2
+L C CF6
 U 1 1 4FC6CF5C
 P 5950 6100
-F 0 "CF2" H 6000 6200 50  0000 L CNN
+F 0 "CF6" H 6000 6200 50  0000 L CNN
 F 1 "47pF" V 6050 5850 50  0000 L CNN
 F 2 "Capacitors_SMD:C_0603" H 5950 6100 60  0001 C CNN
@@
 $EndComp
 $Comp
-L R RF7
+L R RF8
 U 1 1 4FC6C4A3
 P 10000 6800
-F 0 "RF7" V 10080 6800 50  0000 C CNN
+F 0 "RF8" V 10080 6800 50  0000 C CNN
 F 1 "10k" V 10000 6800 50  0000 C CNN
 F 2 "Resistors_SMD:R_0603" H 10000 6800 60  0001 C CNN
@@
 $EndComp
 $Comp
-L C CF5
+L C CF4
 U 1 1 4FC6C3C0
 P 7300 4300
-F 0 "CF5" V 7350 4400 50  0000 L CNN
+F 0 "CF4" V 7350 4400 50  0000 L CNN
 F 1 "33nF" V 7350 4050 50  0000 L CNN
 F 2 "Capacitors_SMD:C_0603" H 7300 4300 60  0001 C CNN
@@
 $EndComp
 $Comp
-L C CF4
+L C CF2
 U 1 1 4FC6C1A7
 P 7250 2650
-F 0 "CF4" H 7300 2750 50  0000 L CNN
+F 0 "CF2" H 7300 2750 50  0000 L CNN
 F 1 "10uF" H 7300 2550 50  0000 L CNN
 F 2 "Capacitors_SMD:C_0603" H 7250 2650 60  0001 C CNN
@@
 $EndComp
 $Comp
-L R RF5
+L R RF1
 U 1 1 4FC6BECA
 P 7900 2650
-F 0 "RF5" V 7980 2650 50  0000 C CNN
+F 0 "RF1" V 7980 2650 50  0000 C CNN
 F 1 "470R" V 7900 2650 50  0000 C CNN
 F 2 "Resistors_SMD:R_0603" H 7900 2650 60  0001 C CNN
@@
 $EndComp
 $Comp
-L C CF6
+L C CF3
 U 1 1 4FC6BE12
 P 7900 3100
-F 0 "CF6" H 7950 3200 50  0000 L CNN
+F 0 "CF3" H 7950 3200 50  0000 L CNN
 F 1 "100nF" H 7950 3000 50  0000 L CNN
 F 2 "Capacitors_SMD:C_0603" H 7900 3100 60  0001 C CNN
@@
 $EndComp
 $Comp
-L R RF4
+L R RF7
 U 1 1 4FC6BD44
 P 7250 6300
-F 0 "RF4" V 7330 6300 50  0000 C CNN
+F 0 "RF7" V 7330 6300 50  0000 C CNN
 F 1 "10K" V 7250 6300 50  0000 C CNN
 F 2 "Resistors_SMD:R_0603" H 7250 6300 60  0001 C CNN
@@
 $EndComp
 $Comp
-L C CF3
+L C CF1
 U 1 1 4FC6BCE9
 P 6450 2650
-F 0 "CF3" H 6500 2750 50  0000 L CNN
+F 0 "CF1" H 6500 2750 50  0000 L CNN
 F 1 "10nF" H 6500 2550 50  0000 L CNN
 F 2 "Capacitors_SMD:C_0603" H 6450 2650 60  0001 C CNN
@@
 $EndComp
 $Comp
-L R RF3
+L R RF5
 U 1 1 4FC6BC62
 P 7200 5200
-F 0 "RF3" V 7280 5200 50  0000 C CNN
+F 0 "RF5" V 7280 5200 50  0000 C CNN
 F 1 "1K5" V 7200 5200 50  0000 C CNN
 F 2 "Resistors_SMD:R_0603" H 7200 5200 60  0001 C CNN
@@
 $EndComp
 $Comp
-L R RF2
+L R RF3
 U 1 1 4FC6BC59
 P 6650 4900
-F 0 "RF2" V 6730 4900 50  0000 C CNN
+F 0 "RF3" V 6730 4900 50  0000 C CNN
 F 1 "27R" V 6650 4900 50  0000 C CNN
 F 2 "Resistors_SMD:R_0603" H 6650 4900 60  0001 C CNN
@@
 $EndComp
 $Comp
-L R RF1
+L R RF2
 U 1 1 4FC6BC34
 P 6650 4600
-F 0 "RF1" V 6730 4600 50  0000 C CNN
+F 0 "RF2" V 6730 4600 50  0000 C CNN
 F 1 "27R" V 6650 4600 50  0000 C CNN
 F 2 "Resistors_SMD:R_0603" H 6650 4600 60  0001 C CNN
@@
 RXD
 $Comp
-L R RF8
+L R RF4
 U 1 1 51CD787E
 P 10500 5000
-F 0 "RF8" V 10580 5000 50  0000 C CNN
+F 0 "RF4" V 10580 5000 50  0000 C CNN
 F 1 "15K" V 10500 5000 50  0000 C CNN
 F 2 "Resistors_SMD:R_0603" H 10500 5000 60  0001 C CNN
@@
 $EndComp
 $Comp
-L +3V3 #PWR17
+L +3V3 #PWR06
 U 1 1 589F5460
 P 10300 6750
-F 0 "#PWR17" H 10300 6600 50  0001 C CNN
+F 0 "#PWR06" H 10300 6600 50  0001 C CNN
 F 1 "+3V3" H 10300 6890 50  0000 C CNN
 F 2 "" H 10300 6750 50  0000 C CNN
@@
 $EndComp
 $Comp
-L +3V3 #PWR16
+L +3V3 #PWR07
 U 1 1 589F5F40
 P 10300 5050
-F 0 "#PWR16" H 10300 4900 50  0001 C CNN
+F 0 "#PWR07" H 10300 4900 50  0001 C CNN
 F 1 "+3V3" H 10300 5190 50  0000 C CNN
 F 2 "" H 10300 5050 50  0000 C CNN
@@
 $EndComp
 $Comp
-L +3V3 #PWR18
+L +3V3 #PWR08
 U 1 1 589F6257
 P 10500 4800
-F 0 "#PWR18" H 10500 4650 50  0001 C CNN
+F 0 "#PWR08" H 10500 4650 50  0001 C CNN
 F 1 "+3V3" H 10500 4940 50  0000 C CNN
 F 2 "" H 10500 4800 50  0000 C CNN
@@
 $EndComp
 $Comp
-L +3V3 #PWR15
+L +3V3 #PWR09
 U 1 1 589F6BB3
 P 8800 3450
-F 0 "#PWR15" H 8800 3300 50  0001 C CNN
+F 0 "#PWR09" H 8800 3300 50  0001 C CNN
 F 1 "+3V3" H 8800 3590 50  0000 C CNN
 F 2 "" H 8800 3450 50  0000 C CNN
@@
 F 0 "F1" V 5030 4250 50  0000 C CNN
 F 1 "PTS08056V050" V 4850 4250 50  0000 C CNN
-F 2 "Project:R_1812" V 4880 4250 50  0001 C CNN
+F 2 "Resistors_SMD:R_0805" V 4880 4250 50  0001 C CNN
 F 3 "http://www.belfuse.com/pdfs/0ZCK.pdf" H 4950 4250 50  0001 C CNN
 F 4 "PTS08056V050-ND" V 4950 4250 60  0001 C CNN "REF DIGIKEY"
@@
 	6450 2500 6450 2400
 $Comp
-L GND #PWR9
+L GND #PWR010
 U 1 1 58A66750
 P 6450 2900
-F 0 "#PWR9" H 6450 2650 50  0001 C CNN
+F 0 "#PWR010" H 6450 2650 50  0001 C CNN
 F 1 "GND" H 6450 2750 50  0000 C CNN
 F 2 "" H 6450 2900 50  0000 C CNN
@@
 	7100 6300 6750 6300
 $Comp
-L GND #PWR11
+L GND #PWR011
 U 1 1 58A8D1C3
 P 7250 2900
-F 0 "#PWR11" H 7250 2650 50  0001 C CNN
+F 0 "#PWR011" H 7250 2650 50  0001 C CNN
 F 1 "GND" H 7250 2750 50  0000 C CNN
 F 2 "" H 7250 2900 50  0000 C CNN
@@
 $EndComp
 $Comp
-L GND #PWR13
+L GND #PWR012
 U 1 1 58A8D267
 P 7900 3350
-F 0 "#PWR13" H 7900 3100 50  0001 C CNN
+F 0 "#PWR012" H 7900 3100 50  0001 C CNN
 F 1 "GND" H 7900 3200 50  0000 C CNN
 F 2 "" H 7900 3350 50  0000 C CNN
@@
 $EndComp
 $Comp
-L GND #PWR14
+L GND #PWR013
 U 1 1 58A8D7DD
 P 8300 7400
-F 0 "#PWR14" H 8300 7150 50  0001 C CNN
+F 0 "#PWR013" H 8300 7150 50  0001 C CNN
 F 1 "GND" H 8300 7250 50  0000 C CNN
 F 2 "" H 8300 7400 50  0000 C CNN
@@
 $EndComp
 $Comp
-L GND #PWR12
+L GND #PWR014
 U 1 1 58A8DF8B
 P 7450 6450
-F 0 "#PWR12" H 7450 6200 50  0001 C CNN
+F 0 "#PWR014" H 7450 6200 50  0001 C CNN
 F 1 "GND" H 7450 6300 50  0000 C CNN
 F 2 "" H 7450 6450 50  0000 C CNN
@@
 $EndComp
 $Comp
-L GND #PWR8
+L GND #PWR015
 U 1 1 58A8E746
 P 5650 5900
-F 0 "#PWR8" H 5650 5650 50  0001 C CNN
+F 0 "#PWR015" H 5650 5650 50  0001 C CNN
 F 1 "GND" H 5650 5750 50  0000 C CNN
 F 2 "" H 5650 5900 50  0000 C CNN
@@
 $EndComp
 $Comp
-L GND #PWR7
+L GND #PWR016
 U 1 1 58A8EFD2
 P 5000 5050
-F 0 "#PWR7" H 5000 4800 50  0001 C CNN
+F 0 "#PWR016" H 5000 4800 50  0001 C CNN
 F 1 "GND" H 5000 4900 50  0000 C CNN
 F 2 "" H 5000 5050 50  0000 C CNN
@@
 $EndComp
 $Comp
-L GND #PWR6
+L GND #PWR017
 U 1 1 58A8F696
 P 3650 5050
-F 0 "#PWR6" H 3650 4800 50  0001 C CNN
+F 0 "#PWR017" H 3650 4800 50  0001 C CNN
 F 1 "GND" H 3650 4900 50  0000 C CNN
 F 2 "" H 3650 5050 50  0000 C CNN
@@
 $EndComp
 $Comp
-L GND #PWR10
+L GND #PWR018
 U 1 1 58A8F991
 P 7000 4300
-F 0 "#PWR10" H 7000 4050 50  0001 C CNN
+F 0 "#PWR018" H 7000 4050 50  0001 C CNN
 F 1 "GND" H 7000 4150 50  0000 C CNN
 F 2 "" H 7000 4300 50  0000 C CNN
