File: hard/PCB/ADC_DAC.sch (KiCad schematic (older format))
At the start: 5 parts, among them U5 MAX5864

Commit message: Corrección esquematico
Parts:
- removed C5, C6, C7: 330nF, Capacitors_SMD:C_0402, symbol C
- added CA1, CA2, CA3: 330nF, Capacitors_SMD:C_0402, symbol C
Changed lines of the file:
@@
 $Descr A4 11693 8268
 encoding utf-8
-Sheet 5 6
+Sheet 5 5
 Title ""
 Date ""
@@
 $Comp
 L MAX5864 U5
-U 1 1 591DD15D
+U 1 1 592D87CF
 P 4450 3950
 F 0 "U5" H 4450 4000 60  0000 C CNN
@@
 DA0
 $Comp
-L GND #PWR104
-U 1 1 592560AD
+L GND #PWR100
+U 1 1 592D87D0
 P 4300 5150
-F 0 "#PWR104" H 4300 4900 50  0001 C CNN
+F 0 "#PWR100" H 4300 4900 50  0001 C CNN
 F 1 "GND" H 4300 5000 50  0000 C CNN
 F 2 "" H 4300 5150 50  0000 C CNN
@@
 $EndComp
 $Comp
-L +3V3 #PWR105
-U 1 1 59258C29
+L +3V3 #PWR101
+U 1 1 592D87D1
 P 4400 5300
-F 0 "#PWR105" H 4400 5150 50  0001 C CNN
+F 0 "#PWR101" H 4400 5150 50  0001 C CNN
 F 1 "+3V3" H 4500 5450 50  0000 C CNN
 F 2 "" H 4400 5300 50  0000 C CNN
@@
 $EndComp
 $Comp
-L +3V3 #PWR102
-U 1 1 5925CA50
+L +3V3 #PWR96
+U 1 1 592D87D2
 P 2800 4350
-F 0 "#PWR102" H 2800 4200 50  0001 C CNN
+F 0 "#PWR96" H 2800 4200 50  0001 C CNN
 F 1 "+3V3" H 2750 4500 50  0000 C CNN
 F 2 "" H 2800 4350 50  0000 C CNN
@@
 $EndComp
 $Comp
-L GND #PWR103
-U 1 1 5925CAA5
+L GND #PWR97
+U 1 1 592D87D3
 P 2800 4600
-F 0 "#PWR103" H 2800 4350 50  0001 C CNN
+F 0 "#PWR97" H 2800 4350 50  0001 C CNN
 F 1 "GND" H 2800 4450 50  0000 C CNN
 F 2 "" H 2800 4600 50  0000 C CNN
@@
 $EndComp
 $Comp
-L GND #PWR101
-U 1 1 5925CB54
+L GND #PWR95
+U 1 1 592D87D4
 P 2800 3850
-F 0 "#PWR101" H 2800 3600 50  0001 C CNN
+F 0 "#PWR95" H 2800 3600 50  0001 C CNN
 F 1 "GND" H 2800 3700 50  0000 C CNN
 F 2 "" H 2800 3850 50  0000 C CNN
@@
 $EndComp
 $Comp
-L +3V3 #PWR97
-U 1 1 5925CB87
+L +3V3 #PWR94
+U 1 1 592D87D5
 P 2800 3500
-F 0 "#PWR97" H 2800 3350 50  0001 C CNN
+F 0 "#PWR94" H 2800 3350 50  0001 C CNN
 F 1 "+3V3" H 2650 3550 50  0000 C CNN
 F 2 "" H 2800 3500 50  0000 C CNN
@@
 $EndComp
 $Comp
-L GND #PWR95
-U 1 1 5925CCF5
+L GND #PWR98
+U 1 1 592D87D6
 P 2950 2450
-F 0 "#PWR95" H 2950 2200 50  0001 C CNN
+F 0 "#PWR98" H 2950 2200 50  0001 C CNN
 F 1 "GND" H 2950 2300 50  0000 C CNN
 F 2 "" H 2950 2450 50  0000 C CNN
@@
 QA+
 $Comp
-L C C7
-U 1 1 5925E9DF
+L C CA1
+U 1 1 592D87D7
 P 2950 3150
-F 0 "C7" H 2850 3250 50  0000 L CNN
+F 0 "CA1" H 2800 3250 50  0000 L CNN
 F 1 "330nF" H 3000 3050 50  0000 L CNN
 F 2 "Capacitors_SMD:C_0402" H 2988 3000 50  0001 C CNN
@@
 $EndComp
 $Comp
-L C C6
-U 1 1 5925F060
+L C CA3
+U 1 1 592D87D8
 P 3400 2650
-F 0 "C6" H 3300 2750 50  0000 L CNN
+F 0 "CA3" V 3550 2600 50  0000 L CNN
 F 1 "330nF" V 3250 2550 50  0000 L CNN
 F 2 "Capacitors_SMD:C_0402" H 3438 2500 50  0001 C CNN
@@
 $EndComp
 $Comp
-L C C5
-U 1 1 5925F0E3
+L C CA2
+U 1 1 592D87D9
 P 3400 2350
-F 0 "C5" H 3300 2450 50  0000 L CNN
+F 0 "CA2" V 3350 2400 50  0000 L CNN
 F 1 "330nF" V 3250 2250 50  0000 L CNN
 F 2 "Capacitors_SMD:C_0402" H 3438 2200 50  0001 C CNN
@@
 ID+
 $Comp
-L +3V3 #PWR100
-U 1 1 5926096B
+L +3V3 #PWR103
+U 1 1 592D87DA
 P 5950 3700
-F 0 "#PWR100" H 5950 3550 50  0001 C CNN
+F 0 "#PWR103" H 5950 3550 50  0001 C CNN
 F 1 "+3V3" V 5950 3900 50  0000 C CNN
 F 2 "" H 5950 3700 50  0000 C CNN
@@
 $EndComp
 $Comp
-L +3V3 #PWR94
-U 1 1 59261D83
+L +3V3 #PWR99
+U 1 1 592D87DB
 P 4250 2350
-F 0 "#PWR94" H 4250 2200 50  0001 C CNN
+F 0 "#PWR99" H 4250 2200 50  0001 C CNN
 F 1 "+3V3" H 4250 2500 50  0000 C CNN
 F 2 "" H 4250 2350 50  0000 C CNN
@@
 Connection ~ 5000 2400
 $Comp
-L GND #PWR96
-U 1 1 592622C2
+L GND #PWR102
+U 1 1 592D87DC
 P 5200 2500
-F 0 "#PWR96" H 5200 2250 50  0001 C CNN
+F 0 "#PWR102" H 5200 2250 50  0001 C CNN
 F 1 "GND" H 5200 2350 50  0000 C CNN
 F 2 "" H 5200 2500 50  0000 C CNN
@@
 $Comp
 L CONN_02X05 PA1
-U 1 1 5926528A
+U 1 1 592D87DD
 P 8100 3800
 F 0 "PA1" H 8100 4100 50  0000 C CNN
@@
 $EndComp
 $Comp
-L +3V3 #PWR98
-U 1 1 5926544A
+L +3V3 #PWR104
+U 1 1 592D87DE
 P 7550 3550
-F 0 "#PWR98" H 7550 3400 50  0001 C CNN
+F 0 "#PWR104" H 7550 3400 50  0001 C CNN
 F 1 "+3V3" H 7550 3700 50  0000 C CNN
 F 2 "" H 7550 3550 50  0000 C CNN
@@
 $EndComp
 $Comp
-L GND #PWR99
-U 1 1 592655B9
+L GND #PWR105
+U 1 1 592D87DF
 P 8650 3600
-F 0 "#PWR99" H 8650 3350 50  0001 C CNN
+F 0 "#PWR105" H 8650 3350 50  0001 C CNN
 F 1 "GND" V 8650 3400 50  0000 C CNN
 F 2 "" H 8650 3600 50  0000 C CNN

Commit message: update 3d models
Parts:
- renumbered CA2 to CA1, CA3 to CA2, CA1 to CA3
Changed lines of the file:
@@
 DA0
 $Comp
-L GND #PWR100
+L GND #PWR0110
 U 1 1 592D87D0
 P 4300 5150
-F 0 "#PWR100" H 4300 4900 50  0001 C CNN
+F 0 "#PWR0110" H 4300 4900 50  0001 C CNN
 F 1 "GND" H 4300 5000 50  0000 C CNN
 F 2 "" H 4300 5150 50  0000 C CNN
@@
 $EndComp
 $Comp
-L +3V3 #PWR101
+L +3V3 #PWR0111
 U 1 1 592D87D1
 P 4400 5300
-F 0 "#PWR101" H 4400 5150 50  0001 C CNN
+F 0 "#PWR0111" H 4400 5150 50  0001 C CNN
 F 1 "+3V3" H 4500 5450 50  0000 C CNN
 F 2 "" H 4400 5300 50  0000 C CNN
@@
 $EndComp
 $Comp
-L +3V3 #PWR96
+L +3V3 #PWR0112
 U 1 1 592D87D2
 P 2800 4350
-F 0 "#PWR96" H 2800 4200 50  0001 C CNN
+F 0 "#PWR0112" H 2800 4200 50  0001 C CNN
 F 1 "+3V3" H 2750 4500 50  0000 C CNN
 F 2 "" H 2800 4350 50  0000 C CNN
@@
 $EndComp
 $Comp
-L GND #PWR97
+L GND #PWR0113
 U 1 1 592D87D3
 P 2800 4600
-F 0 "#PWR97" H 2800 4350 50  0001 C CNN
+F 0 "#PWR0113" H 2800 4350 50  0001 C CNN
 F 1 "GND" H 2800 4450 50  0000 C CNN
 F 2 "" H 2800 4600 50  0000 C CNN
@@
 $EndComp
 $Comp
-L GND #PWR95
+L GND #PWR0114
 U 1 1 592D87D4
 P 2800 3850
-F 0 "#PWR95" H 2800 3600 50  0001 C CNN
+F 0 "#PWR0114" H 2800 3600 50  0001 C CNN
 F 1 "GND" H 2800 3700 50  0000 C CNN
 F 2 "" H 2800 3850 50  0000 C CNN
@@
 $EndComp
 $Comp
-L +3V3 #PWR94
+L +3V3 #PWR0115
 U 1 1 592D87D5
 P 2800 3500
-F 0 "#PWR94" H 2800 3350 50  0001 C CNN
+F 0 "#PWR0115" H 2800 3350 50  0001 C CNN
 F 1 "+3V3" H 2650 3550 50  0000 C CNN
 F 2 "" H 2800 3500 50  0000 C CNN
@@
 $EndComp
 $Comp
-L GND #PWR98
+L GND #PWR0116
 U 1 1 592D87D6
 P 2950 2450
-F 0 "#PWR98" H 2950 2200 50  0001 C CNN
+F 0 "#PWR0116" H 2950 2200 50  0001 C CNN
 F 1 "GND" H 2950 2300 50  0000 C CNN
 F 2 "" H 2950 2450 50  0000 C CNN
@@
 QA+
 $Comp
-L C CA1
+L C CA3
 U 1 1 592D87D7
 P 2950 3150
-F 0 "CA1" H 2800 3250 50  0000 L CNN
+F 0 "CA3" H 2800 3250 50  0000 L CNN
 F 1 "330nF" H 3000 3050 50  0000 L CNN
 F 2 "Capacitors_SMD:C_0402" H 2988 3000 50  0001 C CNN
@@
 $EndComp
 $Comp
-L C CA3
+L C CA2
 U 1 1 592D87D8
 P 3400 2650
-F 0 "CA3" V 3550 2600 50  0000 L CNN
+F 0 "CA2" V 3550 2600 50  0000 L CNN
 F 1 "330nF" V 3250 2550 50  0000 L CNN
 F 2 "Capacitors_SMD:C_0402" H 3438 2500 50  0001 C CNN
@@
 $EndComp
 $Comp
-L C CA2
+L C CA1
 U 1 1 592D87D9
 P 3400 2350
-F 0 "CA2" V 3350 2400 50  0000 L CNN
+F 0 "CA1" V 3350 2400 50  0000 L CNN
 F 1 "330nF" V 3250 2250 50  0000 L CNN
 F 2 "Capacitors_SMD:C_0402" H 3438 2200 50  0001 C CNN
@@
 ID+
 $Comp
-L +3V3 #PWR103
+L +3V3 #PWR0117
 U 1 1 592D87DA
 P 5950 3700
-F 0 "#PWR103" H 5950 3550 50  0001 C CNN
+F 0 "#PWR0117" H 5950 3550 50  0001 C CNN
 F 1 "+3V3" V 5950 3900 50  0000 C CNN
 F 2 "" H 5950 3700 50  0000 C CNN
@@
 $EndComp
 $Comp
-L +3V3 #PWR99
+L +3V3 #PWR0118
 U 1 1 592D87DB
 P 4250 2350
-F 0 "#PWR99" H 4250 2200 50  0001 C CNN
+F 0 "#PWR0118" H 4250 2200 50  0001 C CNN
 F 1 "+3V3" H 4250 2500 50  0000 C CNN
 F 2 "" H 4250 2350 50  0000 C CNN
@@
 Connection ~ 5000 2400
 $Comp
-L GND #PWR102
+L GND #PWR0119
 U 1 1 592D87DC
 P 5200 2500
-F 0 "#PWR102" H 5200 2250 50  0001 C CNN
+F 0 "#PWR0119" H 5200 2250 50  0001 C CNN
 F 1 "GND" H 5200 2350 50  0000 C CNN
 F 2 "" H 5200 2500 50  0000 C CNN
@@
 $EndComp
 $Comp
-L +3V3 #PWR104
+L +3V3 #PWR0120
 U 1 1 592D87DE
 P 7550 3550
-F 0 "#PWR104" H 7550 3400 50  0001 C CNN
+F 0 "#PWR0120" H 7550 3400 50  0001 C CNN
 F 1 "+3V3" H 7550 3700 50  0000 C CNN
 F 2 "" H 7550 3550 50  0000 C CNN
@@
 $EndComp
 $Comp
-L GND #PWR105
+L GND #PWR0121
 U 1 1 592D87DF
 P 8650 3600
-F 0 "#PWR105" H 8650 3350 50  0001 C CNN
+F 0 "#PWR0121" H 8650 3350 50  0001 C CNN
 F 1 "GND" V 8650 3400 50  0000 C CNN
 F 2 "" H 8650 3600 50  0000 C CNN

Commit message: Changes in HDMISpartan6_Board
Parts:
- added C50, C51, C52, C56: 4.7uF, Capacitors_SMD:C_0805, symbol C
- added C53, C54, C55, C57: 0.47uF, Capacitors_SMD:C_0402, symbol C
Connections:
- net labels added: adCLK, adCS, adDA0, adDA1, adDA2, adDA3, adDA4, adDA5, adDA6, adDA7, adDA[0..7], adDD0, adDD1, adDD2, adDD3, adDD4, adDD5, adDD6, adDD7, adDD8, adDD9, adDD[0..9], adMOSI, adSCK
- net labels removed: CS_AD, DA0, DA1, DA2, DA3, DA4, DA5, DA6, DA7, DA[0..7], DD0, DD1, DD2, DD3, DD4, DD5, DD6, DD7, DD8, DD9, DD[0..9], F_CK, SPI_MOSI, SPI_SCK
- wire segments 75 -> 77
Other:
- note added: "Vcc 18\ndecoupling"
- note added: "Vcc 2,8,43\ndecoupling"
