File: hard/PCB/ADC_DAC.sch (KiCad schematic (older format))
At the start: 13 parts, among them U5 MAX5864

Commit message: versión 1.0
Parts:
- renumbered PA1 to P4
Connections:
- wire segments 77 -> 78
Changed lines of the file:
@@
 adMOSI
 $Comp
-L GND #PWR0119
+L GND #PWR128
 U 1 1 592D87D0
 P 4300 5150
-F 0 "#PWR0119" H 4300 4900 50  0001 C CNN
+F 0 "#PWR128" H 4300 4900 50  0001 C CNN
 F 1 "GND" H 4300 5000 50  0000 C CNN
 F 2 "" H 4300 5150 50  0000 C CNN
@@
 $EndComp
 $Comp
-L +3V3 #PWR0120
+L +3V3 #PWR129
 U 1 1 592D87D1
 P 4400 5300
-F 0 "#PWR0120" H 4400 5150 50  0001 C CNN
+F 0 "#PWR129" H 4400 5150 50  0001 C CNN
 F 1 "+3V3" H 4500 5450 50  0000 C CNN
 F 2 "" H 4400 5300 50  0000 C CNN
@@
 $EndComp
 $Comp
-L +3V3 #PWR0121
+L +3V3 #PWR126
 U 1 1 592D87D2
 P 2800 4350
-F 0 "#PWR0121" H 2800 4200 50  0001 C CNN
+F 0 "#PWR126" H 2800 4200 50  0001 C CNN
 F 1 "+3V3" H 2750 4500 50  0000 C CNN
 F 2 "" H 2800 4350 50  0000 C CNN
@@
 $EndComp
 $Comp
-L GND #PWR0122
+L GND #PWR127
 U 1 1 592D87D3
 P 2800 4600
-F 0 "#PWR0122" H 2800 4350 50  0001 C CNN
+F 0 "#PWR127" H 2800 4350 50  0001 C CNN
 F 1 "GND" H 2800 4450 50  0000 C CNN
 F 2 "" H 2800 4600 50  0000 C CNN
@@
 $EndComp
 $Comp
-L GND #PWR0123
+L GND #PWR124
 U 1 1 592D87D4
 P 3250 3800
-F 0 "#PWR0123" H 3250 3550 50  0001 C CNN
+F 0 "#PWR124" H 3250 3550 50  0001 C CNN
 F 1 "GND" H 3250 3650 50  0000 C CNN
 F 2 "" H 3250 3800 50  0000 C CNN
@@
 $EndComp
 $Comp
-L +3V3 #PWR0124
+L +3V3 #PWR120
 U 1 1 592D87D5
 P 2800 3500
-F 0 "#PWR0124" H 2800 3350 50  0001 C CNN
+F 0 "#PWR120" H 2800 3350 50  0001 C CNN
 F 1 "+3V3" H 2650 3550 50  0000 C CNN
 F 2 "" H 2800 3500 50  0000 C CNN
@@
 $EndComp
 $Comp
-L GND #PWR0125
+L GND #PWR117
 U 1 1 592D87D6
 P 2950 2450
-F 0 "#PWR0125" H 2950 2200 50  0001 C CNN
+F 0 "#PWR117" H 2950 2200 50  0001 C CNN
 F 1 "GND" H 2950 2300 50  0000 C CNN
 F 2 "" H 2950 2450 50  0000 C CNN
@@
 ID+
 $Comp
-L +3V3 #PWR0126
+L +3V3 #PWR123
 U 1 1 592D87DA
 P 5950 3700
-F 0 "#PWR0126" H 5950 3550 50  0001 C CNN
+F 0 "#PWR123" H 5950 3550 50  0001 C CNN
 F 1 "+3V3" V 5950 3900 50  0000 C CNN
 F 2 "" H 5950 3700 50  0000 C CNN
@@
 $EndComp
 $Comp
-L +3V3 #PWR0127
+L +3V3 #PWR116
 U 1 1 592D87DB
 P 4250 2350
-F 0 "#PWR0127" H 4250 2200 50  0001 C CNN
+F 0 "#PWR116" H 4250 2200 50  0001 C CNN
 F 1 "+3V3" H 4250 2500 50  0000 C CNN
 F 2 "" H 4250 2350 50  0000 C CNN
@@
 $EndComp
 $Comp
-L GND #PWR0128
+L GND #PWR118
 U 1 1 592D87DC
 P 5200 2500
-F 0 "#PWR0128" H 5200 2250 50  0001 C CNN
+F 0 "#PWR118" H 5200 2250 50  0001 C CNN
 F 1 "GND" H 5200 2350 50  0000 C CNN
 F 2 "" H 5200 2500 50  0000 C CNN
@@
 adCLK
 $Comp
-L CONN_02X05 PA1
+L CONN_02X05 P4
 U 1 1 592D87DD
 P 8100 3800
-F 0 "PA1" H 8100 4100 50  0000 C CNN
+F 0 "P4" H 8100 4100 50  0000 C CNN
 F 1 "CONN_02X05" H 8100 3500 50  0000 C CNN
 F 2 "Pin_Headers:Pin_Header_Straight_2x05_Pitch2.54mm" H 8100 2600 50  0001 C CNN
@@
 $EndComp
 $Comp
-L +3V3 #PWR0129
+L +3V3 #PWR122
 U 1 1 592D87DE
+P 8650 3550
+F 0 "#PWR122" H 8650 3400 50  0001 C CNN
+F 1 "+3V3" H 8650 3700 50  0000 C CNN
+F 2 "" H 8650 3550 50  0000 C CNN
+F 3 "" H 8650 3550 50  0000 C CNN
+	1    8650 3550
+	1    0    0    -1
+$EndComp
+$Comp
+L GND #PWR121
+U 1 1 592D87DF
 P 7550 3550
-F 0 "#PWR0129" H 7550 3400 50  0001 C CNN
-F 1 "+3V3" H 7550 3700 50  0000 C CNN
+F 0 "#PWR121" H 7550 3300 50  0001 C CNN
+F 1 "GND" V 7550 3350 50  0000 C CNN
 F 2 "" H 7550 3550 50  0000 C CNN
 F 3 "" H 7550 3550 50  0000 C CNN
 	1    7550 3550
-	1    0    0    -1
-$EndComp
-$Comp
-L GND #PWR0130
-U 1 1 592D87DF
-P 8650 3600
-F 0 "#PWR0130" H 8650 3350 50  0001 C CNN
-F 1 "GND" V 8650 3400 50  0000 C CNN
-F 2 "" H 8650 3600 50  0000 C CNN
-F 3 "" H 8650 3600 50  0000 C CNN
-	1    8650 3600
-	0    -1   -1   0
-$EndComp
-Text Label 7650 4000 0    60   ~ 0
+	-1   0    0    1
+$EndComp
+Text Label 7550 4000 0    60   ~ 0
 QA+
-Text Label 8450 4000 0    60   ~ 0
+Text Label 8700 4000 0    60   ~ 0
 QA-
 Text Label 3050 3700 0    60   ~ 0
 IA-
-Text Label 7650 3900 0    60   ~ 0
+Text Label 8700 3900 0    60   ~ 0
 IA+
-Text Label 7650 3800 0    60   ~ 0
+Text Label 8700 3800 0    60   ~ 0
 ID+
-Text Label 7650 3700 0    60   ~ 0
+Text Label 7550 3700 0    60   ~ 0
 QD+
-Text Label 8450 3900 0    60   ~ 0
+Text Label 7550 3900 0    60   ~ 0
 IA-
-Text Label 8450 3800 0    60   ~ 0
+Text Label 7550 3800 0    60   ~ 0
 ID-
-Text Label 8450 3700 0    60   ~ 0
+Text Label 8700 3700 0    60   ~ 0
 QD-
 Text Label 4300 2700 1    60   ~ 0
@@
 adDA7
 $Comp
-L GND #PWR0131
+L GND #PWR125
 U 1 1 59A57EEF
 P 3250 4000
-F 0 "#PWR0131" H 3250 3750 50  0001 C CNN
+F 0 "#PWR125" H 3250 3750 50  0001 C CNN
 F 1 "GND" H 3250 3850 50  0000 C CNN
 F 2 "" H 3250 4000 50  0000 C CNN
@@
 $EndComp
 $Comp
-L +3V3 #PWR0132
+L +3V3 #PWR130
 U 1 1 59A1B273
 P 2500 6450
-F 0 "#PWR0132" H 2500 6300 50  0001 C CNN
+F 0 "#PWR130" H 2500 6300 50  0001 C CNN
 F 1 "+3V3" H 2500 6590 50  0000 C CNN
 F 2 "" H 2500 6450 50  0000 C CNN
@@
 $EndComp
 $Comp
-L GND #PWR0133
+L GND #PWR132
 U 1 1 59A1B279
 P 2500 6750
-F 0 "#PWR0133" H 2500 6500 50  0001 C CNN
+F 0 "#PWR132" H 2500 6500 50  0001 C CNN
 F 1 "GND" H 2500 6600 50  0000 C CNN
 F 2 "" H 2500 6750 50  0000 C CNN
@@
 Connection ~ 2250 6450
 $Comp
-L +3V3 #PWR0134
+L +3V3 #PWR131
 U 1 1 59A1C684
 P 4950 6450
-F 0 "#PWR0134" H 4950 6300 50  0001 C CNN
+F 0 "#PWR131" H 4950 6300 50  0001 C CNN
 F 1 "+3V3" H 4950 6590 50  0000 C CNN
 F 2 "" H 4950 6450 50  0000 C CNN
@@
 $EndComp
 $Comp
-L GND #PWR0135
+L GND #PWR133
 U 1 1 59A1C68A
 P 4950 6750
-F 0 "#PWR0135" H 4950 6500 50  0001 C CNN
+F 0 "#PWR133" H 4950 6500 50  0001 C CNN
 F 1 "GND" H 4950 6600 50  0000 C CNN
 F 2 "" H 4950 6750 50  0000 C CNN
@@
 Vcc 18\ndecoupling
 $Comp
-L +3V3 #PWR0136
+L +3V3 #PWR119
 U 1 1 59AF3E16
 P 4800 2650
-F 0 "#PWR0136" H 4800 2500 50  0001 C CNN
+F 0 "#PWR119" H 4800 2500 50  0001 C CNN
 F 1 "+3V3" H 4800 2800 50  0000 C CNN
 F 2 "" H 4800 2650 50  0000 C CNN
@@
 Wire Wire Line
 	4800 2650 4800 2750
+Wire Wire Line
+	8650 3550 8650 3600
 $EndSCHEMATC
