File: hard/PCB/HDMIspartan6_Board.kicad_pcb (KiCad board)
At the start: 2 copper layers, 58.5 x 99 mm, 249 parts, among them P1 CONN_02X20, P2 CONN_02X03, P3 CONN_01X03, P4 CONN_02X05, P5 CONN_02X05, U1 XC6SLX9-2TQG144C, U2 TPS62133RGTR, U3 ZLDO1117G33TA, U4 ZLDO1117G12TA, U5 MAX5864, U6 S25FL064LABMFI013, U7 ATMEGA32U4-A

Commit message: v1-0
Routing:
- net GND: track 1257.9 -> 1239.6 mm, vias 51 -> 53
- net /spartan6/Dout: track 77.9 -> 77.2 mm
- net /spartan6/Din: track 77.7 -> 77.2 mm
Changed lines of the file:
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@@
     (thickness 1.6)
     (drawings 18)
-    (tracks 4341)
+    (tracks 4345)
     (zones 0)
     (modules 249)
@@
   (segment (start 150.88999 142.646943) (end 150.88999 143.659168) (width 0.2) (layer F.Cu) (net 0))
   (segment (start 151.344 143.597) (end 151.344 142.835) (width 0.2) (layer F.Cu) (net 0))
+  (segment (start 132.802 105.37) (end 130.13706 108.03494) (width 0.2) (layer F.Cu) (net 1))
+  (segment (start 130.13706 108.03494) (end 130.13706 108.41858) (width 0.2) (layer F.Cu) (net 1))
+  (via (at 130.13706 108.41858) (size 0.5) (drill 0.3) (layers F.Cu B.Cu) (net 1))
+  (segment (start 131.024 104.1) (end 131.532 104.1) (width 0.2) (layer B.Cu) (net 1))
+  (via (at 132.802 105.37) (size 0.5) (drill 0.3) (layers F.Cu B.Cu) (net 1))
+  (segment (start 131.532 104.1) (end 132.802 105.37) (width 0.2) (layer B.Cu) (net 1))
+  (segment (start 135.342 99.782) (end 131.024 104.1) (width 0.2) (layer B.Cu) (net 1))
+  (segment (start 134.83458 98.63958) (end 135.342 99.147) (width 0.2) (layer B.Cu) (net 1))
+  (segment (start 135.342 99.147) (end 135.342 99.782) (width 0.2) (layer B.Cu) (net 1))
+  (segment (start 131.28006 98.63958) (end 134.83458 98.63958) (width 0.2) (layer B.Cu) (net 1))
   (segment (start 109.307 84.8976) (end 109.1546 84.8976) (width 0.2) (layer F.Cu) (net 1))
   (segment (start 109.1546 84.8976) (end 108.7228 84.8976) (width 0.2) (layer F.Cu) (net 1))
@@
   (segment (start 111.139063 84.522581) (end 111.279061 84.662579) (width 0.2) (layer F.Cu) (net 1))
   (segment (start 111.279061 84.662579) (end 111.969059 84.662579) (width 0.2) (layer F.Cu) (net 1))
-  (segment (start 108.672 113.752) (end 107.91 114.514) (width 0.7) (layer B.Cu) (net 1))
-  (segment (start 107.91 124.42) (end 108.672 125.182) (width 0.7) (layer B.Cu) (net 1))
-  (segment (start 107.91 114.514) (end 107.91 124.42) (width 0.7) (layer B.Cu) (net 1))
   (segment (start 108.672 137.882) (end 107.91 137.12) (width 0.7) (layer F.Cu) (net 1))
-  (segment (start 107.91 137.12) (end 107.91 114.514) (width 0.7) (layer F.Cu) (net 1))
-  (segment (start 107.91 114.514) (end 108.672 113.752) (width 0.7) (layer F.Cu) (net 1))
   (segment (start 128.768 142.42918) (end 128.768 141.5696) (width 0.2) (layer F.Cu) (net 1))
   (segment (start 128.768 141.5696) (end 128.502 141.3036) (width 0.2) (layer F.Cu) (net 1))
@@
   (segment (start 124.939713 92.797) (end 124.801 92.797) (width 0.2) (layer F.Cu) (net 85))
   (via (at 124.801 92.797) (size 0.5) (drill 0.3) (layers F.Cu B.Cu) (net 85))
-  (segment (start 133.94706 107.770095) (end 130.866493 110.850662) (width 0.2) (layer F.Cu) (net 86))
-  (segment (start 133.94706 101.30658) (end 133.94706 107.770095) (width 0.2) (layer F.Cu) (net 86))
-  (segment (start 130.866493 110.850662) (end 130.247775 111.46938) (width 0.2) (layer F.Cu) (net 86))
+  (segment (start 137.31256 98.63958) (end 134.072 101.88014) (width 0.2) (layer B.Cu) (net 86))
+  (segment (start 137.63006 98.63958) (end 137.31256 98.63958) (width 0.2) (layer B.Cu) (net 86))
+  (segment (start 134.072 102.421553) (end 134.072 102.068) (width 0.2) (layer F.Cu) (net 86))
+  (segment (start 134.072 107.645155) (end 134.072 102.421553) (width 0.2) (layer F.Cu) (net 86))
+  (segment (start 130.247775 111.46938) (end 134.072 107.645155) (width 0.2) (layer F.Cu) (net 86))
+  (segment (start 134.072 101.88014) (end 134.072 102.068) (width 0.2) (layer B.Cu) (net 86))
+  (via (at 134.072 102.068) (size 0.5) (drill 0.3) (layers F.Cu B.Cu) (net 86))
   (segment (start 117.423 94.756) (end 117.423 94.956) (width 0.2) (layer B.Cu) (net 86))
   (segment (start 118.374956 91.069956) (end 118.374956 93.804044) (width 0.2) (layer B.Cu) (net 86))
@@
   (segment (start 118.197 90.003) (end 118.197 90.892) (width 0.2) (layer F.Cu) (net 86))
   (via (at 118.197 90.892) (size 0.5) (drill 0.3) (layers F.Cu B.Cu) (net 86))
-  (segment (start 137.63006 98.63958) (end 137.37606 98.63958) (width 0.2) (layer B.Cu) (net 86))
-  (segment (start 137.37606 98.63958) (end 134.70906 101.30658) (width 0.2) (layer B.Cu) (net 86))
-  (segment (start 134.70906 101.30658) (end 133.94706 101.30658) (width 0.2) (layer B.Cu) (net 86))
-  (segment (start 137.63006 98.63958) (end 137.31256 98.63958) (width 0.2) (layer B.Cu) (net 86))
-  (via (at 133.94706 101.30658) (size 0.5) (drill 0.3) (layers F.Cu B.Cu) (net 86))
   (segment (start 120.84705 81.199251) (end 120.84705 80.38157) (width 0.2) (layer F.Cu) (net 87))
   (segment (start 120.84705 80.38157) (end 120.58806 80.12258) (width 0.2) (layer F.Cu) (net 87))
@@
   (segment (start 120.737 84.612) (end 120.458049 84.333049) (width 0.2) (layer F.Cu) (net 87))
   (segment (start 120.458049 84.333049) (end 120.458049 84.065268) (width 0.2) (layer F.Cu) (net 87))
-  (segment (start 134.353447 100.2646) (end 134.707 100.2646) (width 0.2) (layer B.Cu) (net 88))
-  (segment (start 131.28006 101.17958) (end 132.05156 101.17958) (width 0.2) (layer B.Cu) (net 88))
-  (segment (start 134.707 100.618153) (end 134.707 100.2646) (width 0.2) (layer F.Cu) (net 88))
-  (segment (start 134.707 107.717261) (end 134.707 100.618153) (width 0.2) (layer F.Cu) (net 88))
-  (via (at 134.707 100.2646) (size 0.5) (drill 0.3) (layers F.Cu B.Cu) (net 88))
-  (segment (start 132.96654 100.2646) (end 134.353447 100.2646) (width 0.2) (layer B.Cu) (net 88))
-  (segment (start 130.601328 111.822933) (end 134.707 107.717261) (width 0.2) (layer F.Cu) (net 88))
-  (segment (start 132.05156 101.17958) (end 132.96654 100.2646) (width 0.2) (layer B.Cu) (net 88))
+  (segment (start 134.702999 107.721262) (end 134.702999 101.174999) (width 0.2) (layer F.Cu) (net 88))
+  (segment (start 133.568001 100.539999) (end 133.818 100.29) (width 0.2) (layer B.Cu) (net 88))
+  (segment (start 134.067999 100.539999) (end 133.818 100.29) (width 0.2) (layer F.Cu) (net 88))
+  (segment (start 134.702999 101.174999) (end 134.067999 100.539999) (width 0.2) (layer F.Cu) (net 88))
+  (segment (start 132.92842 101.17958) (end 133.568001 100.539999) (width 0.2) (layer B.Cu) (net 88))
+  (segment (start 130.601328 111.822933) (end 134.702999 107.721262) (width 0.2) (layer F.Cu) (net 88))
+  (segment (start 131.28006 101.17958) (end 132.92842 101.17958) (width 0.2) (layer B.Cu) (net 88))
+  (via (at 133.818 100.29) (size 0.5) (drill 0.3) (layers F.Cu B.Cu) (net 88))
   (segment (start 117.62459 90.679371) (end 117.62459 90.325818) (width 0.2) (layer B.Cu) (net 88))
   (segment (start 117.974945 91.473943) (end 117.62459 91.123588) (width 0.2) (layer B.Cu) (net 88))

Commit message: version1.oo1
Parts:
- moved TH65 28.0 mm to (136.0, 134.7)
- moved TH43 16.4 mm to (132.2, 138.5)
- moved TH76 16.3 mm to (138.5, 141.7)
- moved TH73 5.08 mm to (138.5, 151.9)
- moved TH69 4.02 mm to (152.5, 143.0)
- moved TH19 3.75 mm to (136.0, 129.0)
- moved TH66 3.33 mm to (164.9, 142.3)
- moved TH74 2.54 mm to (133.4, 151.9)
- moved TH70 2.29 mm to (152.5, 146.1)
- moved TH8 2.01 mm to (110.6, 138.5)
- moved TH71 1.91 mm to (148.7, 146.1)
- moved TH42 1.34 mm to (132.3, 141.7)
- moved TH83 1.27 mm to (148.7, 140.4)
- moved TH75 1.27 mm to (127.1, 151.9)
- moved TH14 1.21 mm to (115.7, 138.5)
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Routing:
- net +3V3: track 541.7 -> 583.5 mm, vias 33 -> 32
- net +1V2: track 153.2 -> 183.6 mm
- net GND: track 1239.6 -> 1245.2 mm, vias 53 -> 56
- net (no net): track 2.00 -> 0.00 mm
- net /spartan6/usCD: track 35.6 -> 34.9 mm
- net /spartan6/usMISO: track 34.3 -> 33.7 mm
- net /spartan6/usSCK: track 35.5 -> 34.9 mm
- net /spartan6/usMOSI: track 38.0 -> 37.4 mm
- net /spartan6/usCS: track 38.4 -> 37.8 mm
