File: hard/PCB/HDMIspartan6_Board.sch (KiCad schematic (older format))
At the start: 50 parts

Commit message: Changes in HDMISpartan6_Board
Parts:
- added TH51, TH52, TH53, TH54, TH55, TH56, TH57, TH58, TH59, TH60, TH61, TH62, TH63, TH64, TH65, TH66, TH67, TH68, TH69, TH70, TH71, TH72, TH73, TH74, TH75, TH76, TH77, TH78, TH79, TH80, TH81, TH82, TH83, TH84, TH85, TH86, TH87, TH88, TH89, TH90: CONN_1, Project:1Pin_12mil_VIA, symbol CONN_1
- TH1: footprint Measurement_Points:Measurement_Point_Round-TH_Small -> Project:1Pin_12mil_VIATH_Small
- TH50: footprint Measurement_Points:Measurement_Point_Round-TH_Small -> Project:1Pin_12mil_VIA
Connections:
- net GND: now also TH51.1 (P1), TH52.1 (P1), TH53.1 (P1), TH54.1 (P1), TH55.1 (P1), TH56.1 (P1), TH57.1 (P1), TH58.1 (P1), TH59.1 (P1), TH60.1 (P1), TH61.1 (P1), TH62.1 (P1), TH63.1 (P1), TH64.1 (P1), TH65.1 (P1), TH66.1 (P1), TH67.1 (P1), TH68.1 (P1), TH69.1 (P1), TH70.1 (P1), TH71.1 (P1), TH72.1 (P1), TH73.1 (P1), TH74.1 (P1), TH75.1 (P1), TH76.1 (P1), TH77.1 (P1), TH78.1 (P1), TH79.1 (P1), TH80.1 (P1), TH81.1 (P1), TH82.1 (P1), TH83.1 (P1), TH84.1 (P1), TH85.1 (P1), TH86.1 (P1), TH87.1 (P1), TH88.1 (P1), TH89.1 (P1), TH90.1 (P1)
Other:
- note removed: "PENDIENTES:\n\n>>> IMPLEMENTAR REGLAS DEL FABRICANTE <<<\n\n- Reorganizar PinOut\n- Asignar LEDs indicadores a FPGA\n"

Commit message: versión 1.0
Parts:
- added TH100, TH101, TH102, TH103, TH104, TH105, TH106, TH107, TH108, TH109, TH110, TH91, TH92, TH93, TH94, TH95, TH96, TH97, TH98, TH99: CONN_1, Project:1Pin_12mil_VIA, symbol CONN_1
- TH1: footprint Project:1Pin_12mil_VIATH_Small -> Project:1Pin_12mil_VIA
Connections:
- net GND: now also TH100.1 (P1), TH101.1 (P1), TH102.1 (P1), TH103.1 (P1), TH104.1 (P1), TH105.1 (P1), TH106.1 (P1), TH107.1 (P1), TH108.1 (P1), TH109.1 (P1), TH110.1 (P1), TH91.1 (P1), TH92.1 (P1), TH93.1 (P1), TH94.1 (P1), TH95.1 (P1), TH96.1 (P1), TH97.1 (P1), TH98.1 (P1), TH99.1 (P1)
