File: hard/PCB/atmega32u4.sch (KiCad schematic (older format))
At the start: 21 parts, among them P4 CONN_01X06, P5 CONN_01X08, P6 CONN_01X08, P7 CONN_01X10, U7 ATMEGA32U4-A

Commit message: versión 1.0
Parts:
- removed P4: CONN_01X06, Pin_Headers:Pin_Header_Straight_1x06_Pitch2.54mm, symbol CONN_01X06
- removed P5, P6: CONN_01X08, Pin_Headers:Pin_Header_Straight_1x08_Pitch2.54mm, symbol CONN_01X08
- removed P7: CONN_01X10, Pin_Headers:Pin_Header_Straight_1x10_Pitch2.54mm, symbol CONN_01X10
- added R14, R15: 2k2, Resistors_SMD:R_0603, symbol R
- renumbered PA2 to P5
Connections:
- wire segments 109 -> 111
- no-connect marks 1 -> 2
Changed lines of the file:
@@
 NoConn ~ 1800 3600
 $Comp
-L GND #PWR0137
+L GND #PWR142
 U 1 1 5992199E
 P 2700 2600
-F 0 "#PWR0137" H 2700 2350 50  0001 C CNN
+F 0 "#PWR142" H 2700 2350 50  0001 C CNN
 F 1 "GND" H 2700 2450 50  0000 C CNN
 F 2 "" H 2700 2600 50  0000 C CNN
@@
 $EndComp
 $Comp
-L GND #PWR0138
+L GND #PWR145
 U 1 1 599219A4
 P 2000 3750
-F 0 "#PWR0138" H 2000 3500 50  0001 C CNN
+F 0 "#PWR145" H 2000 3500 50  0001 C CNN
 F 1 "GND" H 2000 3600 50  0000 C CNN
 F 2 "" H 2000 3750 50  0000 C CNN
@@
 $EndComp
 $Comp
-L GND #PWR0139
+L GND #PWR144
 U 1 1 599219AA
 P 650 3750
-F 0 "#PWR0139" H 650 3500 50  0001 C CNN
+F 0 "#PWR144" H 650 3500 50  0001 C CNN
 F 1 "GND" H 650 3600 50  0000 C CNN
 F 2 "" H 650 3750 50  0000 C CNN
@@
 $EndComp
 $Comp
-L GND #PWR0140
+L GND #PWR152
 U 1 1 599488A1
 P 5100 5300
-F 0 "#PWR0140" H 5100 5050 50  0001 C CNN
+F 0 "#PWR152" H 5100 5050 50  0001 C CNN
 F 1 "GND" H 5100 5150 50  0000 C CNN
 F 2 "" H 5100 5300 50  0000 C CNN
@@
 $EndComp
 $Comp
-L +3V3 #PWR0141
+L +3V3 #PWR137
 U 1 1 5994A407
 P 3950 1450
-F 0 "#PWR0141" H 3950 1300 50  0001 C CNN
+F 0 "#PWR137" H 3950 1300 50  0001 C CNN
 F 1 "+3V3" H 3950 1590 50  0000 C CNN
 F 2 "" H 3950 1450 50  0000 C CNN
@@
 $EndComp
 $Comp
-L +3V3 #PWR0142
+L +3V3 #PWR141
 U 1 1 5994A44D
 P 5000 1650
-F 0 "#PWR0142" H 5000 1500 50  0001 C CNN
+F 0 "#PWR141" H 5000 1500 50  0001 C CNN
 F 1 "+3V3" H 5000 1790 50  0000 C CNN
 F 2 "" H 5000 1650 50  0000 C CNN
@@
 $EndComp
 $Comp
-L +3V3 #PWR0143
+L +3V3 #PWR146
 U 1 1 5994A5B2
 P 3750 3750
-F 0 "#PWR0143" H 3750 3600 50  0001 C CNN
+F 0 "#PWR146" H 3750 3600 50  0001 C CNN
 F 1 "+3V3" H 3750 3890 50  0000 C CNN
 F 2 "" H 3750 3750 50  0000 C CNN
@@
 $EndComp
 $Comp
-L +3V3 #PWR0144
+L +3V3 #PWR134
 U 1 1 5994ABA1
 P 700 750
-F 0 "#PWR0144" H 700 600 50  0001 C CNN
+F 0 "#PWR134" H 700 600 50  0001 C CNN
 F 1 "+3V3" H 700 890 50  0000 C CNN
 F 2 "" H 700 750 50  0000 C CNN
@@
 $EndComp
 $Comp
-L GND #PWR0145
+L GND #PWR136
 U 1 1 5994ABA7
 P 700 1050
-F 0 "#PWR0145" H 700 800 50  0001 C CNN
+F 0 "#PWR136" H 700 800 50  0001 C CNN
 F 1 "GND" H 700 900 50  0000 C CNN
 F 2 "" H 700 1050 50  0000 C CNN
@@
 micro\ndecoupling
 $Comp
-L GND #PWR0146
+L GND #PWR147
 U 1 1 5994B368
 P 3750 4050
-F 0 "#PWR0146" H 3750 3800 50  0001 C CNN
+F 0 "#PWR147" H 3750 3800 50  0001 C CNN
 F 1 "GND" H 3750 3900 50  0000 C CNN
 F 2 "" H 3750 4050 50  0000 C CNN
@@
 $EndComp
 $Comp
-L GND #PWR0147
+L GND #PWR138
 U 1 1 5994BB94
 P 4600 1500
-F 0 "#PWR0147" H 4600 1250 50  0001 C CNN
+F 0 "#PWR138" H 4600 1250 50  0001 C CNN
 F 1 "GND" H 4600 1350 50  0000 C CNN
 F 2 "" H 4600 1500 50  0000 C CNN
@@
 $EndComp
 $Comp
-L GND #PWR0148
+L GND #PWR139
 U 1 1 5994BB9D
 P 5400 1500
-F 0 "#PWR0148" H 5400 1250 50  0001 C CNN
+F 0 "#PWR139" H 5400 1250 50  0001 C CNN
 F 1 "GND" H 5400 1350 50  0000 C CNN
 F 2 "" H 5400 1500 50  0000 C CNN
@@
 $EndComp
 $Comp
-L +3V3 #PWR0149
+L +3V3 #PWR135
 U 1 1 5994BCFA
 P 4250 750
-F 0 "#PWR0149" H 4250 600 50  0001 C CNN
+F 0 "#PWR135" H 4250 600 50  0001 C CNN
 F 1 "+3V3" H 4250 890 50  0000 C CNN
 F 2 "" H 4250 750 50  0000 C CNN
@@
 $EndComp
 $Comp
-L GND #PWR0150
+L GND #PWR149
 U 1 1 5994CF65
 P 3800 4950
-F 0 "#PWR0150" H 3800 4700 50  0001 C CNN
+F 0 "#PWR149" H 3800 4700 50  0001 C CNN
 F 1 "GND" H 3800 4800 50  0000 C CNN
 F 2 "" H 3800 4950 50  0000 C CNN
@@
 $EndComp
 $Comp
-L CONN_02X05 PA2
+L CONN_02X05 P5
 U 1 1 5994E51A
 P 9350 5300
-F 0 "PA2" H 9350 5600 50  0000 C CNN
+F 0 "P5" H 9350 5600 50  0000 C CNN
 F 1 "CONN_02X05" H 9350 5000 50  0000 C CNN
 F 2 "Pin_Headers:Pin_Header_Straight_2x05_Pitch2.54mm" H 9350 4100 50  0001 C CNN
@@
 $EndComp
 $Comp
-L +3V3 #PWR0151
+L +3V3 #PWR150
 U 1 1 5994E521
 P 8800 5050
-F 0 "#PWR0151" H 8800 4900 50  0001 C CNN
+F 0 "#PWR150" H 8800 4900 50  0001 C CNN
 F 1 "+3V3" H 8800 5200 50  0000 C CNN
 F 2 "" H 8800 5050 50  0000 C CNN
@@
 $EndComp
 $Comp
-L GND #PWR0152
+L GND #PWR151
 U 1 1 5994E527
 P 9900 5100
-F 0 "#PWR0152" H 9900 4850 50  0001 C CNN
+F 0 "#PWR151" H 9900 4850 50  0001 C CNN
 F 1 "GND" V 9900 4900 50  0000 C CNN
 F 2 "" H 9900 5100 50  0000 C CNN
@@
 Text Label 6350 3450 0    60   ~ 0
 uD2
-Text Label 6300 2750 0    60   ~ 0
+Text Label 3350 2050 0    60   ~ 0
 uD9
 Text Label 6300 2650 0    60   ~ 0
@@
 uD[0..9]
 $Comp
-L GND #PWR0153
+L GND #PWR148
 U 1 1 599E071E
 P 6450 4050
-F 0 "#PWR0153" H 6450 3800 50  0001 C CNN
+F 0 "#PWR148" H 6450 3800 50  0001 C CNN
 F 1 "GND" H 6450 3900 50  0000 C CNN
 F 2 "" H 6450 4050 50  0000 C CNN
@@
 $EndComp
 $Comp
-L GND #PWR0154
+L GND #PWR140
 U 1 1 599E3877
 P 2350 1600
-F 0 "#PWR0154" H 2350 1350 50  0001 C CNN
+F 0 "#PWR140" H 2350 1350 50  0001 C CNN
 F 1 "GND" H 2350 1450 50  0000 C CNN
 F 2 "" H 2350 1600 50  0000 C CNN
@@
 	6600 3450 6250 3450
 Wire Wire Line
-	6600 3350 6250 3350
-Wire Wire Line
-	6250 3250 6600 3250
+	6250 3350 7350 3350
+Wire Wire Line
+	6250 3250 7100 3250
 Wire Wire Line
 	6600 2950 6250 2950
 Wire Wire Line
 	6250 3050 6600 3050
-Wire Wire Line
-	6250 2750 6600 2750
 Wire Wire Line
 	6600 2650 6250 2650
@@
 	3950 1900 3950 2050
 Wire Wire Line
-	3550 2050 4000 2050
+	3350 2050 4000 2050
 Wire Wire Line
 	5100 5200 5100 5300
@@
 Text Label 8000 3900 0    60   ~ 0
 uD9
-$Comp
-L CONN_01X08 P6
-U 1 1 59B6D22D
-P 10050 3400
-F 0 "P6" H 10050 3850 50  0000 C CNN
-F 1 "CONN_01X08" V 10150 3400 50  0000 C CNN
-F 2 "Pin_Headers:Pin_Header_Straight_1x08_Pitch2.54mm" H 10050 3400 50  0001 C CNN
-F 3 "" H 10050 3400 50  0000 C CNN
-	1    10050 3400
-	1    0    0    -1
-$EndComp
-$Comp
-L CONN_01X08 P5
-U 1 1 59B6D2B6
-P 9600 2450
-F 0 "P5" H 9600 2900 50  0000 C CNN
-F 1 "CONN_01X08" V 9700 2450 50  0000 C CNN
-F 2 "Pin_Headers:Pin_Header_Straight_1x08_Pitch2.54mm" H 9600 2450 50  0001 C CNN
-F 3 "" H 9600 2450 50  0000 C CNN
-	1    9600 2450
-	1    0    0    -1
-$EndComp
-$Comp
-L CONN_01X10 P7
-U 1 1 59B6D358
-P 9600 3500
-F 0 "P7" H 9600 4050 50  0000 C CNN
-F 1 "CONN_01X10" V 9700 3500 50  0000 C CNN
-F 2 "Pin_Headers:Pin_Header_Straight_1x10_Pitch2.54mm" H 9600 3500 50  0001 C CNN
-F 3 "" H 9600 3500 50  0000 C CNN
-	1    9600 3500
-	1    0    0    -1
-$EndComp
-$Comp
-L CONN_01X06 P4
-U 1 1 59B6D3D1
-P 10100 2400
-F 0 "P4" H 10100 2750 50  0000 C CNN
-F 1 "CONN_01X06" V 10200 2400 50  0000 C CNN
-F 2 "Pin_Headers:Pin_Header_Straight_1x06_Pitch2.54mm" H 10100 2400 50  0001 C CNN
-F 3 "" H 10100 2400 50  0000 C CNN
-	1    10100 2400
-	1    0    0    -1
-$EndComp
 Connection ~ 5300 1800
+NoConn ~ 6250 2750
+$Comp
+L R R14
+U 1 1 59CA6DB9
+P 7100 3050
+F 0 "R14" V 7180 3050 50  0000 C CNN
+F 1 "2k2" V 7100 3050 50  0000 C CNN
+F 2 "Resistors_SMD:R_0603" H 7100 3050 60  0001 C CNN
+F 3 "" H 7100 3050 60  0001 C CNN
+	1    7100 3050
+	1    0    0    1
+$EndComp
+$Comp
+L R R15
+U 1 1 59CA714F
+P 7350 3050
+F 0 "R15" V 7430 3050 50  0000 C CNN
+F 1 "2k2" V 7350 3050 50  0000 C CNN
+F 2 "Resistors_SMD:R_0603" H 7350 3050 60  0001 C CNN
+F 3 "" H 7350 3050 60  0001 C CNN
+	1    7350 3050
+	1    0    0    -1
+$EndComp
+Wire Wire Line
+	7100 2900 7350 2900
+Wire Wire Line
+	7100 3250 7100 3200
+Wire Wire Line
+	7350 3350 7350 3200
+$Comp
+L +3V3 #PWR143
+U 1 1 59CA74FA
+P 7250 2900
+F 0 "#PWR143" H 7250 2750 50  0001 C CNN
+F 1 "+3V3" H 7250 3040 50  0000 C CNN
+F 2 "" H 7250 2900 50  0000 C CNN
+F 3 "" H 7250 2900 50  0000 C CNN
+	1    7250 2900
+	1    0    0    -1
+$EndComp
+Connection ~ 7250 2900
 $EndSCHEMATC
