File: HW/PCB/spartan6.sch (KiCad schematic (older format))
At the start: 34 parts, among them J1 CONN_02X09, J3 HDMI_A, J4 CONN-MICRO-SD-CARD-PUSH-PULL, P1 CONN_02X20, P3 CONN_01X03, U1 XC6SLX9-2TQG144C, U6 S25FL064LABNFI043

Commit message: change all board files
Parts:
- J4: Description CONN MICRO SD CARD HINGED TYPE -> (none); Digikey ref (none) -> WM9731CT-ND; MF_Name Molex -> (none); MF_PN 5009010801 -> (none); Package UNDEFINED -> (none); S1_Name Digikey -> (none); S1_PN WM9731CT-ND -> (none); Verified Not Verified -> (none); a (none) -> a
Changed lines of the file:
@@
 F 2 "Project:CONN-SD-MICRO-MOLEX" H 10750 7450 50  0001 C CIN
 F 3 "https://www.molex.com/pdm_docs/sd/475710001_sd.pdf" H 10750 7800 10  0001 C CNN
-F 4 "UNDEFINED" H 10750 7450 50  0001 C CIN "Package"
-F 5 "Molex" H 10750 7450 50  0001 C CIN "MF_Name"
-F 6 "5009010801" H 10750 7450 50  0001 C CIN "MF_PN"
-F 7 "Digikey" H 10750 7450 50  0001 C CIN "S1_Name"
-F 8 "WM9731CT-ND " H 10750 7450 50  0001 C CIN "S1_PN"
-F 9 "CONN MICRO SD CARD HINGED TYPE" H 10750 7450 50  0001 C CIN "Description"
-F 10 "Not Verified" H 10750 7450 50  0001 C CIN "Verified"
+F 4 "a" H 10750 7800 60  0000 C CNN "a"
+F 5 "WM9731CT-ND " H 10750 7450 50  0001 C CIN "Digikey ref"
 	1    10750 7800
 	1    0    0    -1
