File: HW/PCB/spartan6.sch (KiCad schematic (older format))
At the start: 34 parts, among them J1 CONN_02X09, J3 HDMI_A, J4 CONN-MICRO-SD-CARD-PUSH-PULL, P1 CONN_02X20, P3 CONN_01X03, U1 XC6SLX9-2TQG144C, U6 S25FL064LABNFI043

Commit message: se cambia la referencia del resonador XF2, queda pendiente actualizar la huella
Parts:
- removed J4: CONN-MICRO-SD-CARD-PUSH-PULL, Project:CONN-SD-MICRO-MOLEX, symbol CONN-MICRO-SD-CARD-PUSH-PULL
- added XS2: uSD CARD, Project:Conn_uSDcard, symbol TFP09-2-12B
- J1: DIGIKEY REF WM18656-ND -> (none); a a -> (none)
- P1: DIGIKEY REF 1528-1783-ND -> (none); a a -> (none)
- U6: value S25FL064LABNFI043 -> S25FL064LABNFI041; Digikey REF 428-4075-1-ND -> (none); Mouser REF (none) -> 727-S25FL064LANFI041
Connections:
- net labels added: usCD
- no-connect marks 34 -> 33
Changed lines of the file:
@@
 F 1 "CONN_02X20" V 2100 6700 50  0000 C CNN
 F 2 "Pin_Headers:Pin_Header_Straight_2x20_Pitch2.54mm" H 2100 5750 50  0001 C CNN
-F 3 "https://media.digikey.com/pdf/Data%20Sheets/Adafruit%20PDFs/1979_Web.pdf" H 2100 5750 50  0000 C CNN
-F 4 "a" H 2100 6700 60  0000 C CNN "a"
-F 5 "1528-1783-ND " H 2100 6700 60  0001 C CNN "DIGIKEY REF"
+F 3 "" H 2100 5750 50  0000 C CNN
 	1    2100 6700
 	1    0    0    -1
@@
 F 1 "CONN_02X09" V 13450 4950 50  0000 C CNN
 F 2 "Project:LVDS_SMD" H 13450 3750 50  0001 C CNN
-F 3 "https://www.mouser.com/ds/2/276/0877591850_PCB_HEADERS-154431.pdf" H 13450 3750 50  0001 C CNN
-F 4 "a" H 13450 4950 60  0000 C CNN "a"
-F 5 "WM18656-ND" H 13450 4950 60  0001 C CNN "DIGIKEY REF"
+F 3 "" H 13450 3750 50  0001 C CNN
 	1    13450 4950
 	1    0    0    -1
@@
 P 10550 9050
 F 0 "U6" H 10250 9300 50  0000 L CNN
-F 1 "S25FL064LABNFI043" H 10600 9300 50  0000 L CNN
+F 1 "S25FL064LABNFI041" H 10600 9300 50  0000 L CNN
 F 2 "Housings_DFN_QFN:DFN-8-1EP_4x4mm_Pitch0.8mm" H 10200 9000 50  0001 C CNN
-F 3 "http://www.cypress.com/file/316661/download" H 10200 9000 50  0001 C CNN
-F 4 "428-4075-1-ND " H 10550 9050 60  0001 C CNN "Digikey REF"
+F 3 "http://www.mouser.com/ds/2/100/002-12878_S25FL064L_64-Mbit_8-Mbyte_3.0_V_FL-L_SPI-1102570.pdf" H 10200 9000 50  0001 C CNN
+F 4 "727-S25FL064LANFI041 " H 10550 9050 60  0001 C CNN "Mouser REF"
 	1    10550 9050
 	-1   0    0    -1
@@
 	4200 5150 4300 5050
 $Comp
+L TFP09-2-12B XS2
+U 1 1 59A8FEBA
+P 8500 9200
+F 0 "XS2" H 8750 8900 50  0000 C CNN
+F 1 "uSD CARD" V 8200 9350 50  0000 C CNN
+F 2 "Project:Conn_uSDcard" H 8500 9200 10  0001 C CNN
+F 3 "https://github.com/PhoenixbornTech/DigiBadgeV2/blob/master/Datasheets/10-TFP09-2-12B.pdf" H 8500 9200 10  0001 C CNN
+F 4 "AliExpress: " H 8500 9200 60  0001 C CNN "DIGIKEY REF"
+	1    8500 9200
+	1    0    0    -1
+$EndComp
+$Comp
 L +3V3 #PWR068
 U 1 1 59A92F13
-P 9850 8000
-F 0 "#PWR068" H 9850 7850 50  0001 C CNN
-F 1 "+3V3" H 9850 8140 50  0000 C CNN
-F 2 "" H 9850 8000 50  0000 C CNN
-F 3 "" H 9850 8000 50  0000 C CNN
-	1    9850 8000
+P 8350 8450
+F 0 "#PWR068" H 8350 8300 50  0001 C CNN
+F 1 "+3V3" H 8350 8590 50  0000 C CNN
+F 2 "" H 8350 8450 50  0000 C CNN
+F 3 "" H 8350 8450 50  0000 C CNN
+	1    8350 8450
 	1    0    0    -1
 $EndComp
@@
 L GND #PWR069
 U 1 1 59A9322C
-P 10000 8400
-F 0 "#PWR069" H 10000 8150 50  0001 C CNN
-F 1 "GND" H 10000 8250 50  0000 C CNN
-F 2 "" H 10000 8400 50  0000 C CNN
-F 3 "" H 10000 8400 50  0000 C CNN
-	1    10000 8400
+P 8350 9600
+F 0 "#PWR069" H 8350 9350 50  0001 C CNN
+F 1 "GND" H 8350 9450 50  0000 C CNN
+F 2 "" H 8350 9600 50  0000 C CNN
+F 3 "" H 8350 9600 50  0000 C CNN
+	1    8350 9600
 	1    0    0    -1
 $EndComp
-Text Label 9700 7450 2    60   ~ 0
+Text Label 9250 9150 2    60   ~ 0
 usMISO
-Text Label 9700 7350 2    60   ~ 0
+Text Label 9250 8950 2    60   ~ 0
 usMOSI
-Text Label 9650 7650 2    60   ~ 0
+Text Label 9250 8850 2    60   ~ 0
 usCS
-Text Label 9700 7550 2    60   ~ 0
+Text Label 9250 9050 2    60   ~ 0
 usSCK
+Text Label 9250 9350 2    60   ~ 0
+usCD
+NoConn ~ 8900 8750
+NoConn ~ 8900 9250
 Text Label 14750 3450 0    60   ~ 0
 RpMISO
@@
 	2750 6650 2350 6650
 Wire Wire Line
+	8350 8450 8350 8550
+Wire Wire Line
+	8350 9500 8350 9600
+Wire Wire Line
+	9250 8850 8900 8850
+Wire Wire Line
+	9250 8950 8900 8950
+Wire Wire Line
+	9250 9050 8900 9050
+Wire Wire Line
+	9250 9150 8900 9150
+Wire Wire Line
+	9250 9350 8900 9350
+Wire Wire Line
 	4650 3550 4850 3550
 Wire Wire Line
@@
 Text Label 7150 1650 3    60   ~ 0
 usSCK
+Text Label 6950 1650 3    60   ~ 0
+usCD
+Wire Wire Line
+	6950 1650 6950 2000
 Wire Wire Line
 	7050 1650 7050 2000
@@
 Text Notes 13350 5500 0    60   ~ 0
 LVDS\n
-$Comp
-L CONN-MICRO-SD-CARD-PUSH-PULL J4
-U 1 1 5AB38E2F
-P 10750 7800
-AR Path="/54B6445D/5AB38E2F" Ref="J4"  Part="1"
-AR Path="/5AB38E2F" Ref="J4"  Part="1"
-F 0 "J4" H 10350 8400 50  0000 L CNN
-F 1 "CONN-MICRO-SD-CARD-PUSH-PULL" H 10350 7200 50  0000 L CNN
-F 2 "Project:CONN-SD-MICRO-MOLEX" H 10750 7450 50  0001 C CIN
-F 3 "https://www.molex.com/pdm_docs/sd/475710001_sd.pdf" H 10750 7800 10  0001 C CNN
-F 4 "UNDEFINED" H 10750 7450 50  0001 C CIN "Package"
-F 5 "Molex" H 10750 7450 50  0001 C CIN "MF_Name"
-F 6 "5009010801" H 10750 7450 50  0001 C CIN "MF_PN"
-F 7 "Digikey" H 10750 7450 50  0001 C CIN "S1_Name"
-F 8 "WM9731CT-ND " H 10750 7450 50  0001 C CIN "S1_PN"
-F 9 "CONN MICRO SD CARD HINGED TYPE" H 10750 7450 50  0001 C CIN "Description"
-F 10 "Not Verified" H 10750 7450 50  0001 C CIN "Verified"
-	1    10750 7800
-	1    0    0    -1
-$EndComp
-Wire Wire Line
-	10150 8250 10000 8250
-Wire Wire Line
-	10000 8250 10000 8400
-Wire Wire Line
-	10150 7650 9650 7650
-Wire Wire Line
-	10150 7350 9700 7350
-Wire Wire Line
-	10150 7450 9700 7450
-Wire Wire Line
-	10150 7550 9700 7550
-Wire Wire Line
-	10150 8150 9850 8150
-Wire Wire Line
-	9850 8150 9850 8000
-NoConn ~ 6950 2000
-NoConn ~ 10150 7950
-NoConn ~ 10150 7850
 $EndSCHEMATC
