File: HW/PCB/atmega32u4.sch (KiCad schematic (older format))
At the start: 19 parts, among them P5 CONN_02X05, U7 ATMEGA32U4-A

Commit message: se cambia la referencia del resonador XF2, queda pendiente actualizar la huella
Parts:
- XF2: value CSTCR8M0G53Z-R0 -> CSTNE8M00G55Z000R0; DIGIKEY REF 490-1218-2-ND -> 490-17960-1-ND
Other:
- note added: "NOTA: CAMBIAR LA HUELLA DEL RESONADOR XF2"
Changed lines of the file:
@@
 P 3350 2500
 F 0 "XF2" H 3350 2400 60  0000 C CNN
-F 1 "CSTCR8M0G53Z-R0" V 3350 3050 60  0000 C CNN
+F 1 "CSTNE8M00G55Z000R0" V 3350 3050 60  0000 C CNN
 F 2 "Project:CSTCE8M00G55-RO" H 3350 2500 60  0001 C CNN
 F 3 "http://www.murata.com/~/media/webrenewal/support/library/catalog/products/timingdevice/ceralock/p16e.ashx" H 3350 2500 60  0001 C CNN
-F 4 "490-1218-2-ND" H 3350 2500 60  0001 C CNN "DIGIKEY REF"
+F 4 "490-17960-1-ND" H 3350 2500 60  0001 C CNN "DIGIKEY REF"
 	1    3350 2500
 	0    1    1    0
@@
 $EndComp
 Connection ~ 7250 2900
+Text Notes 2700 3000 0    60   ~ 0
+NOTA: CAMBIAR LA  HUELLA DEL RESONADOR XF2
 $EndSCHEMATC

Commit message: modificardo cF7 y cF8 a  33 pf
Parts:
- CF7, CF8: value 47pF -> 33pF
Other:
- note removed: "NOTA: CAMBIAR LA HUELLA DEL RESONADOR XF2"
Changed lines of the file:
@@
 P 3000 2200
 F 0 "CF7" H 3050 2300 50  0000 L CNN
-F 1 "47pF" V 3100 1950 50  0000 L CNN
+F 1 "33pF" V 3100 1950 50  0000 L CNN
 F 2 "Capacitors_SMD:C_0603" H 3000 2200 60  0001 C CNN
 F 3 "" H 3000 2200 60  0001 C CNN
@@
 P 3000 2800
 F 0 "CF8" H 3050 2900 50  0000 L CNN
-F 1 "47pF" V 3100 2550 50  0000 L CNN
+F 1 "33pF" V 3100 2550 50  0000 L CNN
 F 2 "Capacitors_SMD:C_0603" H 3000 2800 60  0001 C CNN
 F 3 "" H 3000 2800 60  0001 C CNN
@@
 $EndComp
 Connection ~ 7250 2900
-Text Notes 2700 3000 0    60   ~ 0
-NOTA: CAMBIAR LA  HUELLA DEL RESONADOR XF2
 $EndSCHEMATC
